File: Greenwood18N2/Greenwood18N2.kicad_sch (KiCad schematic)
At the start: 246 parts, among them SW1 Switch w/LED, SW10 Switch w/LED, SW100 Switch w/LED, SW101 Switch w/LED, SW102 Switch w/LED, SW103 Switch w/LED, SW104 Switch w/LED, SW105 Switch w/LED, SW106 Switch w/LED, SW107 Switch w/LED, SW108 Switch w/LED, SW109 Switch w/LED, SW11 Switch w/LED, SW110 Switch w/LED, SW12 Switch w/LED, SW13 Switch w/LED, SW14 Switch w/LED, SW15 Switch w/LED, SW16 Switch w/LED, SW17 Switch w/LED, SW18 RotaryEncoder_Switch, SW19 RotaryEncoder_Switch, SW2 Switch w/LED, SW20 Switch w/LED, SW21 Switch w/LED, SW22 Switch w/LED, SW23 Switch w/LED, SW24 Switch w/LED, SW25 Switch w/LED, SW26 Switch w/LED, SW27 Switch w/LED, SW28 Switch w/LED, SW29 Switch w/LED, SW3 Switch w/LED, SW30 Switch w/LED, SW31 Switch w/LED, SW32 Switch w/LED, SW33 Switch w/LED, SW34 Switch w/LED, SW35 Switch w/LED, SW36 Switch w/LED, SW37 Switch w/LED, SW38 Switch w/LED, SW39 Switch w/LED, SW4 Switch w/LED, SW40 Switch w/LED, SW41 Switch w/LED, SW42 Switch w/LED, SW43 Switch w/LED, SW44 Switch w/LED, SW45 Switch w/LED, SW46 Switch w/LED, SW47 Switch w/LED, SW48 Switch w/LED, SW49 Switch w/LED, SW5 Switch w/LED, SW50 Switch w/LED, SW51 Switch w/LED, SW52 Switch w/LED, SW53 Switch w/LED, SW54 Switch w/LED, SW55 Switch w/LED, SW56 Switch w/LED, SW57 Switch w/LED, SW58 Switch w/LED, SW59 Switch w/LED, SW6 Switch w/LED, SW60 Switch w/LED, SW61 Switch w/LED, SW62 Switch w/LED, SW63 Switch w/LED, SW64 Switch w/LED, SW65 Switch w/LED, SW66 Switch w/LED, SW67 Switch w/LED, SW68 Switch w/LED, SW69 Switch w/LED, SW7 Switch w/LED, SW70 Switch w/LED, SW71 Switch w/LED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

Commit message: Rework of encoders
Remove the dual LED, switch and encoder footprints, it was too complex and I want encoders, I will never be using them as just mx switches.
Changed the encoder under the LCD to an EVQWGD001 since it wont block the screen and be easier to use with just your index finger.
Parts:
- removed C2, C7: 100nF, Capacitor_SMD:C_1206_3216Metric_Pad1.33x1.80mm_HandSolder, symbol Device:C
- removed SW18, SW19, SW75: RotaryEncoder_Switch, Greenwood:ROT_Alps_EC11E-Hotswap_LED, symbol KeebLib:Rotary_MX_w/LED
- added H9: MountingHole, MountingHole:MountingHole_2.2mm_M2_DIN965_Pad, symbol Mechanical:MountingHole
- added R1: 5.1k, Resistor_SMD:R_1206_3216Metric_Pad1.30x1.75mm_HandSolder, symbol Device:R
- added SW1: RotaryEncoder_Switch, Greenwood:RotaryEncoder_Alps_EC11E-Switch_Vertical_H20mm_Centred, symbol Device:RotaryEncoder_Switch
- added SW19: Switch w/LED, Greenwood:Hotswap_MX_Plated_LED_1u, symbol KeebLib:Switch w/LED
- added SW61: RotaryEncoder_Switch, Greenwood:EVQWGD001, symbol Device:RotaryEncoder_Switch
- OLED1: footprint Greenwood:OLED_ST7735_2inch -> KeebLib:OLED_ST7735_2inch
- R2: renamed from R1; value 220k - 5.1M -> 5.1k
- U2: footprint Greenwood:Raspberry_Pi_Pico_Flipped -> ScottoKeebs_MCU:Raspberry_Pi_Pico
- U3: value SN74AHCT1G125DBVR -> 74AHC1G125
- renumbered C4 to C2, C6 to C3, C5 to C4, C3 to C5, H5 to H1, H1 to H2, H2 to H3, H3 to H4, H4 to H5, R2 to R3, SW9 to SW10, SW10 to SW11, SW11 to SW12, SW12 to SW13, SW13 to SW14, SW14 to SW15, SW15 to SW16, SW16 to SW17, SW17 to SW18, SW1 to SW2, SW2 to SW3, SW3 to SW4, SW4 to SW5, SW5 to SW6, SW61 to SW62, SW62 to SW63, SW63 to SW64, SW64 to SW65, SW65 to SW66, SW66 to SW67, SW67 to SW68, SW68 to SW69, SW6 to SW7, SW69 to SW70, SW70 to SW71, SW71 to SW72, SW72 to SW73, SW73 to SW74, SW74 to SW75, SW7 to SW8, SW8 to SW9
Connections:
- net ENC2_B is gone; now on net ROW3: U2.11 (GPIO8)
- net COL0: now also U2.26 (GPIO20), SW1.S2; no longer U2.27 (GPIO21)
- net COL1: now also U2.25 (GPIO19); no longer U2.26 (GPIO20)
- net COL2: now also U2.15 (GPIO11), SW61.S2; no longer U2.17 (GPIO13)
- net COL9: now also SW19.1
- net ENC1_A: now also SW1.A
- net ENC2_A: now also U2.19 (GPIO14), SW61.A; no longer U2.10 (GPIO7)
- net GND: now also R2.1, SW1.C, SW19.6 (GND), SW61.C
- net LED_DAT_3V3: now also U2.32 (GPIO27_ADC1); no longer U2.34 (GPIO28_ADC2)
- net LED_DAT_5V: now also SW2.5 (DIN)
- net LED_PWR: now also SW19.3 (VDD)
- net OLED_MOSI: now also U2.16 (GPIO12); no longer U2.19 (GPIO14)
- net OLED_SCK: now also U2.17 (GPIO13); no longer U2.20 (GPIO15)
- net ROW0: now also U2.27 (GPIO21); no longer U2.29 (GPIO22)
- net ROW1: now also U2.20 (GPIO15); no longer U2.25 (GPIO19)
- net ROW2: now also U2.10 (GPIO7); no longer U2.12 (GPIO9)
- net ROW3: no longer U2.14 (GPIO10)
- net ROW4: now also U2.12 (GPIO9); no longer U2.15 (GPIO11)
- net ROW5: now also U2.14 (GPIO10); no longer U2.16 (GPIO12)
- net VCC: now also R1.2; no longer R2.1
- net at SW60.4 (DOUT): now also SW62.5 (DIN)
- net at SW20.5 (DIN): now also SW19.4 (DOUT)
- net at SW18.4 (DOUT): now also SW19.5 (DIN)
- net at D19.1 (K): now also SW19.2
- net at D1.2 (A): now also SW1.S1
- net LED_EN: now reaches R2.2, U1.3 (EN)
- net LED_EN: now also U2.34 (GPIO28_ADC2)
- net LED_NFAULT: now reaches U1.4 (~{FAULT})
- net LED_NFAULT: now also R1.1
- net at D61.2 (A): now also SW61.S1
- net ENC1_B renamed ENC_B
- net ENC_B: now also U2.29 (GPIO22), SW1.B, SW61.B; no longer U2.32 (GPIO27_ADC1)
- no-connect marks 9 -> 8
Other:
- note added: "NOTE: When USB=500mA, select Rlim = 75k = 74.25k @ 1% = 319mA-401mA range"
- note removed: "NOTE: When USB=500mA, select Rlim = 75k = 74.25k @ 1% = 319mA-401mA range RC circuit to delay EN pin signal when pluggin in USB, t = RC t is for ~62% of input Voltage. 220k gives ~0.2s. 5.1M gives ~0.5s"
- moved on the sheet: C1, C2, C3, C4, D1, D19, D61, H1, H2, H3, H4, H5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

Commit message: Add reset switch
Parts:
- added RESET: SW_Push, KEEBIO:SW_SPST_TL3342, symbol Switch:SW_Push
- renumbered C12 to C10, C5 to C2, C2 to C3, C3 to C4, C4 to C5, C8 to C6, C9 to C7, C10 to C8, C11 to C9
Connections:
- net GND: now also RESET.2
- net RESET: now reaches U2.30 (RUN)
- net RESET: now also RESET.1
- no-connect marks 8 -> 7
Other:
- moved on the sheet: C1, C10, C2, C3, C4, C5, C6, C7, C8, C9, H1, H2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
