File: v1/SP110Duo.kicad_sch (KiCad schematic)
At the start: 307 parts, among them J1 USB_C_Receptacle_USB2.0, Q7 AO3401A, Q8 MMUN2233LT1G, SW1 RotaryEncoder_Switch, SW10 Switch w/LED, SW100 Switch w/LED, SW101 Switch w/LED, SW102 Switch w/LED, SW103 Switch w/LED, SW104 Switch w/LED, SW105 Switch w/LED, SW106 Switch w/LED, SW107 Switch w/LED, SW108 Switch w/LED, SW109 Switch w/LED, SW11 Switch w/LED, SW110 Switch w/LED, SW111 Switch w/LED, SW12 Switch w/LED, SW13 Switch w/LED, SW14 Switch w/LED, SW15 Switch w/LED, SW16 Switch w/LED, SW17 Switch w/LED, SW18 Switch w/LED, SW19 Switch w/LED, SW2 Switch w/LED, SW20 Switch w/LED, SW21 Switch w/LED, SW22 Switch w/LED, SW23 Switch w/LED, SW24 Switch w/LED, SW25 Switch w/LED, SW26 Switch w/LED, SW27 Switch w/LED, SW28 Switch w/LED, SW29 Switch w/LED, SW3 Switch w/LED, SW30 Switch w/LED, SW31 Switch w/LED, SW32 Switch w/LED, SW33 Switch w/LED, SW34 Switch w/LED, SW35 Switch w/LED, SW36 Switch w/LED, SW37 Switch w/LED, SW38 Switch w/LED, SW39 Switch w/LED, SW4 Switch w/LED, SW40 Switch w/LED, SW41 Switch w/LED, SW42 Switch w/LED, SW43 Switch w/LED, SW44 Switch w/LED, SW45 Switch w/LED, SW46 Switch w/LED, SW47 Switch w/LED, SW48 Switch w/LED, SW49 Switch w/LED, SW5 Switch w/LED, SW50 Switch w/LED, SW51 Switch w/LED, SW52 Switch w/LED, SW53 Switch w/LED, SW54 Switch w/LED, SW55 Switch w/LED, SW56 Switch w/LED, SW57 Switch w/LED, SW58 Switch w/LED, SW59 Switch w/LED, SW6 Switch w/LED, SW60 Switch w/LED, SW61 RotaryEncoder_Switch, SW62 Switch w/LED, SW63 Switch w/LED, SW64 Switch w/LED, SW65 Switch w/LED, SW66 Switch w/LED, SW67 Switch w/LED, SW68 Switch w/LED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

Commit message: save
Parts:
- J1: footprint reversible-kicad-footprints:HRO-TYPE-C-31-M-12-HandSoldering-NoSBU -> KeebLib:HRO-TYPE-C-31-M-12-modded
Connections:
- net ENC2_A: now also U4.31 (GPIO20); no longer U4.34 (GPIO22)
- net ENC2_B: now also U4.32 (GPIO21); no longer U4.35 (GPIO23)
- net LCD_BL_PWM: now also U4.30 (GPIO19); no longer U4.32 (GPIO21)
- net LCD_CS: now also U4.29 (GPIO18); no longer U4.31 (GPIO20)
- net LCD_DC: now also U4.28 (GPIO17); no longer U4.30 (GPIO19)
- net LCD_EN: now also U4.35 (GPIO23)
- net LCD_RESET: now also U4.27 (GPIO16); no longer U4.29 (GPIO18)
Changed lines of the file:
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@@
   (junction (at 398.78 506.73) (diameter 0) (color 0 0 0 0)
   )
-  (junction (at 62.23 38.1) (diameter 0) (color 0 0 0 0)
-  )
   (junction (at 182.88 506.73) (diameter 0) (color 0 0 0 0)
   )
@@
     (stroke (width 0) (type default))
   )
-  (wire (pts (xy 62.23 35.56) (xy 62.23 38.1))
-    (stroke (width 0) (type default))
-  )
   (wire (pts (xy 673.735 149.86) (xy 673.735 149.225))
     (stroke (width 0) (type default))
@@
     (stroke (width 0) (type default))
   )
-  (wire (pts (xy 58.42 38.1) (xy 62.23 38.1))
+  (wire (pts (xy 58.42 38.1) (xy 69.85 38.1))
     (stroke (width 0) (type default))
   )
@@
     (stroke (width 0) (type default))
   )
-  (wire (pts (xy 62.23 38.1) (xy 69.85 38.1))
-    (stroke (width 0) (type default))
-  )
   (wire (pts (xy 330.2 353.06) (xy 340.36 353.06))
     (stroke (width 0) (type default))
@@
     )
   )
-  (global_label "LCD_CS" (shape output) (at 435.61 119.38 0) (fields_autoplaced)
+  (global_label "LCD_CS" (shape output) (at 435.61 114.3 0) (fields_autoplaced)
     (effects (font (size 1.27 1.27)) (justify left))
-    (property "Intersheetrefs" "${INTERSHEET_REFS}" (at 445.6104 119.38 0)
+    (property "Intersheetrefs" "${INTERSHEET_REFS}" (at 445.6104 114.3 0)
       (effects (font (size 1.27 1.27)) (justify left) hide)
     )
@@
     )
   )
-  (global_label "LCD_BL_PWM" (shape output) (at 435.61 121.92 0) (fields_autoplaced)
+  (global_label "LCD_BL_PWM" (shape output) (at 435.61 116.84 0) (fields_autoplaced)
     (effects (font (size 1.27 1.27)) (justify left))
-    (property "Intersheetrefs" "${INTERSHEET_REFS}" (at 450.5694 121.92 0)
+    (property "Intersheetrefs" "${INTERSHEET_REFS}" (at 450.5694 116.84 0)
       (effects (font (size 1.27 1.27)) (justify left) hide)
     )
@@
     )
   )
-  (global_label "ENC2_A" (shape input) (at 435.61 124.46 0) (fields_autoplaced)
+  (global_label "ENC2_A" (shape input) (at 435.61 119.38 0) (fields_autoplaced)
     (effects (font (size 1.27 1.27)) (justify left))
-    (property "Intersheetrefs" "${INTERSHEET_REFS}" (at 445.6104 124.46 0)
+    (property "Intersheetrefs" "${INTERSHEET_REFS}" (at 445.6104 119.38 0)
       (effects (font (size 1.27 1.27)) (justify left) hide)
     )
@@
     )
   )
-  (global_label "ENC2_B" (shape input) (at 435.61 127 0) (fields_autoplaced)
+  (global_label "ENC2_B" (shape input) (at 435.61 121.92 0) (fields_autoplaced)
     (effects (font (size 1.27 1.27)) (justify left))
-    (property "Intersheetrefs" "${INTERSHEET_REFS}" (at 445.7918 127 0)
+    (property "Intersheetrefs" "${INTERSHEET_REFS}" (at 445.7918 121.92 0)
       (effects (font (size 1.27 1.27)) (justify left) hide)
     )
@@
     )
   )
-  (global_label "LCD_DC" (shape output) (at 435.61 116.84 0) (fields_autoplaced)
+  (global_label "LCD_DC" (shape output) (at 435.61 111.76 0) (fields_autoplaced)
     (effects (font (size 1.27 1.27)) (justify left))
-    (property "Intersheetrefs" "${INTERSHEET_REFS}" (at 445.6709 116.84 0)
+    (property "Intersheetrefs" "${INTERSHEET_REFS}" (at 445.6709 111.76 0)
       (effects (font (size 1.27 1.27)) (justify left) hide)
     )
@@
     )
   )
-  (global_label "LCD_RESET" (shape output) (at 435.61 114.3 0) (fields_autoplaced)
+  (global_label "LCD_RESET" (shape output) (at 435.61 109.22 0) (fields_autoplaced)
     (effects (font (size 1.27 1.27)) (justify left))
-    (property "Intersheetrefs" "${INTERSHEET_REFS}" (at 448.876 114.3 0)
+    (property "Intersheetrefs" "${INTERSHEET_REFS}" (at 448.876 109.22 0)
       (effects (font (size 1.27 1.27)) (justify left) hide)
     )
@@
     )
   )
-  (global_label "V_USB" (shape passive) (at 62.23 35.56 90) (fields_autoplaced)
+  (global_label "LCD_EN" (shape output) (at 435.61 127 0) (fields_autoplaced)
     (effects (font (size 1.27 1.27)) (justify left))
-    (property "Intersheetrefs" "${INTERSHEET_REFS}" (at 62.23 27.8199 90)
+    (property "Intersheetrefs" "${INTERSHEET_REFS}" (at 445.6104 127 0)
       (effects (font (size 1.27 1.27)) (justify left) hide)
     )
@@
       (effects (font (size 1.27 1.27)))
     )
-    (property "Footprint" "reversible-kicad-footprints:HRO-TYPE-C-31-M-12-HandSoldering-NoSBU" (at 46.99 53.34 0)
+    (property "Footprint" "KeebLib:HRO-TYPE-C-31-M-12-modded" (at 46.99 53.34 0)
       (effects (font (size 1.27 1.27)) hide)
     )
