File: SP110duo/new/SP110Duo.kicad_pcb (KiCad board)
At the start: 2 copper layers, 3.6 x 3.3 mm, 420 parts, among them J1 USB_C_Receptacle_USB2.0, Q1 AO3401A, Q2 MMUN2233LT1G, SW1 RotaryEncoder_Switch, SW2 RotaryEncoder_Switch, U1 AZ1117H-3.3TRE1, U2 TPS2553DBVR, U3 74AHC1G125, U4 W25Q128JVSIQ, U5 PRTR5V0U2X, U6 RP2040, Y1 X322512MSB4SI

Commit message: update for rjk
Parts:
- C14, C15, C16, C17, C18, C19, C20, C26, C27, C28, C29, R10, R11, R12, R14, R15, R16, R8, R9, TP5: moved to B.Cu
- D100: renamed from D116; moved to B.Cu
- D103: renamed from D117; moved to B.Cu
- D104: renamed from D111; moved to B.Cu
- D108: renamed from D115; moved to B.Cu
- D110: renamed from D112; moved to B.Cu
- D62: renamed from D113; moved to B.Cu
- D66: renamed from D114; moved to B.Cu
- LED20, LED21, LED22, LED23, LED24, LED25, LED26, LED27, LED28, LED29, LED30, LED31, LED32, LED33, LED34, LED35, LED36, LED37, LED38: footprint Keyboard:LED_MX_6028R -> Keyboard:LED_MX_6028R-ROT
- MX83: renamed from MX99; footprint Keyboard:SW_MX_HS_2u -> Keyboard:SW_MX_HS_1u
- MX99: renamed from MX98; footprint Keyboard:SW_MX_HS_1u -> Keyboard:SW_MX_HS_2u
- TP1, TP2, TP6, TP7: moved to F.Cu
- moved D66 363.8 mm to (217.2, 87.6), turned to 180 degrees
- moved D100 334.2 mm to (199.5, 133.0), turned to 180 degrees
- moved D103 334.2 mm to (199.5, 136.3), turned to 180 degrees
- moved D108 334.2 mm to (199.5, 129.6), turned to 180 degrees
- moved D104 332.6 mm to (199.5, 121.9), turned to 180 degrees
- moved D110 332.6 mm to (199.5, 125.3), turned to 180 degrees
- moved D62 326.9 mm to (178.6, 87.6), turned to 180 degrees
- moved C14 323.4 mm to (115.6, -106.6), turned to 180 degrees
- moved C15 323.4 mm to (115.6, -101.9), turned to 180 degrees
- moved C16 323.4 mm to (115.6, -97.1), turned to 180 degrees
- moved C17 323.4 mm to (115.6, -92.4), turned to 180 degrees
- moved C18 323.4 mm to (115.6, -87.6), turned to 180 degrees
- moved C19 323.4 mm to (115.6, -82.9), turned to 180 degrees
- moved C20 323.4 mm to (115.6, -78.1), turned to 180 degrees
- moved R10 310.7 mm to (109.2, -77.8), turned to 180 degrees
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- renumbered D97 to D101, D98 to D102, D100 to D105, D101 to D106, D102 to D107, D103 to D109, D104 to D111, D105 to D112, D106 to D113, D107 to D114, D108 to D115, D109 to D116, D110 to D117, D64 to D46, D46 to D47, D47 to D48, D48 to D49, D49 to D50, D50 to D51, D51 to D52, D52 to D53, D53 to D54, D54 to D55, D55 to D56, D56 to D57, D57 to D58, D58 to D59, D59 to D60, D60 to D61, D61 to D63, D62 to D64, D63 to D65, D65 to D67, D66 to D68, D67 to D69, D68 to D70, D69 to D71, D70 to D72, D71 to D73, D72 to D74, D73 to D75, D74 to D76, D75 to D77, D76 to D78, D77 to D79, D78 to D80, D79 to D81, D80 to D82, D81 to D83, D82 to D84, D99 to D85, D83 to D86, D84 to D87, D85 to D88, D86 to D89, D87 to D90, D88 to D91, D89 to D92, D90 to D93, D91 to D94, D92 to D95, D93 to D96, D94 to D97, D95 to D98, D96 to D99, MX64 to MX46, MX46 to MX47, MX47 to MX48, MX48 to MX49, MX49 to MX50, MX50 to MX51, MX51 to MX52, MX52 to MX53, MX53 to MX54, MX54 to MX55, MX55 to MX56, MX56 to MX57, MX57 to MX58, MX58 to MX59, MX59 to MX60, MX60 to MX61, MX61 to MX62, MX62 to MX63, MX63 to MX64, MX83 to MX84, MX84 to MX85, MX85 to MX86, MX86 to MX87, MX87 to MX88, MX88 to MX89, MX89 to MX90, MX90 to MX91, MX91 to MX92, MX92 to MX93, MX93 to MX94, MX94 to MX95, MX95 to MX96, MX96 to MX97, MX97 to MX98
Connections:
- D10 pad 1: Net-(D10-K) -> ROW0
- D10 pad 2: ROW0 -> Net-(D10-A)
- D100 pad 1: RKJ-PUSH -> ROW5
- D100 pad 2: ROW5 -> RKJ-PUSH
- D101 pad 1: ROW5 -> Net-(D101-K)
- D101 pad 2: Net-(D97-A) -> ROW5
- D102 pad 1: Net-(D98-K) -> ROW5
- D102 pad 2: ROW5 -> Net-(D102-A)
- D103 pad 1: ROW5 -> RKJ-A
- D103 pad 2: RKJ-A -> ROW5
- D104 pad 1: ROW2 -> ROW5
- D107 pad 1: Net-(D102-K) -> ROW5
- D107 pad 2: ROW5 -> Net-(D107-A)
- D108 pad 1: ROW4 -> RKJ-B
- D108 pad 2: RKJ-B -> ROW5
- D109 pad 1: Net-(D103-K) -> ROW5
- D109 pad 2: ROW5 -> Net-(D109-A)
- D110 pad 1: ROW3 -> RKJ-C
- D110 pad 2: RKJ-C -> ROW5
- D111 pad 1: Net-(D104-K) -> ROW5
- D111 pad 2: ROW5 -> Net-(D111-A)
- D113 pad 1: Net-(D106-K) -> ROW5
- D113 pad 2: ROW5 -> Net-(D113-A)
- D115 pad 1: Net-(D108-K) -> ROW5
- D115 pad 2: ROW5 -> Net-(D115-A)
- D117 pad 1: Net-(D110-K) -> ROW5
- D117 pad 2: ROW5 -> Net-(D117-A)
- D12 pad 1: Net-(D12-K) -> ROW0
- D12 pad 2: ROW0 -> Net-(D12-A)
- D14 pad 1: Net-(D14-K) -> ROW0
- D14 pad 2: ROW0 -> Net-(D14-A)
- D16 pad 1: Net-(D16-K) -> ROW0
- D16 pad 2: ROW0 -> Net-(D16-A)
- D18 pad 1: Net-(D18-K) -> ROW0
- D18 pad 2: ROW0 -> Net-(D18-A)
- D20 pad 1: Net-(D20-K) -> ROW0
- D20 pad 2: ROW0 -> Net-(D20-A)
- D30 pad 1: Net-(D30-K) -> ROW1
- D30 pad 2: ROW1 -> Net-(D30-A)
- D32 pad 1: Net-(D32-K) -> ROW1
- D32 pad 2: ROW1 -> Net-(D32-A)
- D34 pad 1: Net-(D34-K) -> ROW1
- D34 pad 2: ROW1 -> Net-(D34-A)
- D36 pad 1: Net-(D36-K) -> ROW1
- D36 pad 2: ROW1 -> Net-(D36-A)
- D38 pad 1: Net-(D38-K) -> ROW1
- D38 pad 2: ROW1 -> Net-(D38-A)
- D40 pad 1: Net-(D40-K) -> ROW1
- D40 pad 2: ROW1 -> Net-(D40-A)
- D46 pad 2: ROW3 -> ROW2
- D50 pad 1: Net-(D49-K) (its old number) -> ROW2
- D50 pad 2: ROW2 -> Net-(D50-A)
- D52 pad 1: Net-(D51-K) (its old number) -> ROW2
- D52 pad 2: ROW2 -> Net-(D52-A)
- D54 pad 1: Net-(D53-K) (its old number) -> ROW2
- D54 pad 2: ROW2 -> Net-(D54-A)
- D56 pad 1: Net-(D55-K) (its old number) -> ROW2
- D56 pad 2: ROW2 -> Net-(D56-A)
- D58 pad 1: Net-(D57-K) (its old number) -> ROW2
- D58 pad 2: ROW2 -> Net-(D58-A)
- D60 pad 1: Net-(D59-K) (its old number) -> ROW2
- D60 pad 2: ROW2 -> Net-(D60-A)
- D66 pad 1: ROW3 -> ROT2_D
- D66 pad 2: ROT2_D -> ROW3
- D69 pad 1: Net-(D67-K) (its old number) -> ROW3
- D69 pad 2: ROW3 -> Net-(D69-A)
- D71 pad 1: Net-(D69-K) -> ROW3
- D71 pad 2: ROW3 -> Net-(D71-A)
- D73 pad 1: Net-(D71-K) -> ROW3
- D73 pad 2: ROW3 -> Net-(D73-A)
- D75 pad 1: Net-(D73-K) -> ROW3
- D75 pad 2: ROW3 -> Net-(D75-A)
- D77 pad 1: Net-(D75-K) -> ROW3
- D77 pad 2: ROW3 -> Net-(D77-A)
- D79 pad 1: Net-(D77-K) -> ROW3
- D79 pad 2: ROW3 -> Net-(D79-A)
- D85 pad 1: ROW5 -> ROW4
- D88 pad 1: Net-(D85-K) -> ROW4
- D88 pad 2: ROW4 -> Net-(D88-A)
- D90 pad 1: Net-(D87-K) (its old number) -> ROW4
- D90 pad 2: ROW4 -> Net-(D90-A)
- D92 pad 1: Net-(D89-K) (its old number) -> ROW4
- D92 pad 2: ROW4 -> Net-(D92-A)
- D94 pad 1: Net-(D91-K) (its old number) -> ROW4
- D94 pad 2: ROW4 -> Net-(D94-A)
- D96 pad 1: Net-(D93-K) (its old number) -> ROW4
- D96 pad 2: ROW4 -> Net-(D96-A)
- D98 pad 1: Net-(D95-K) (its old number) -> ROW4
- D98 pad 2: ROW4 -> Net-(D98-A)
- MX10 pad 1: Net-(D10-K) -> Net-(D10-A)
- MX102 pad 1: Net-(D102-K) -> Net-(D107-A)
- MX103 pad 1: Net-(D103-K) -> Net-(D109-A)
- MX104 pad 1: Net-(D104-K) -> Net-(D111-A)
- MX105 pad 2: COL7 -> COL6
- MX106 pad 1: Net-(D106-K) -> Net-(D113-A)
- MX107 pad 2: COL8 -> COL7
- MX108 pad 1: Net-(D108-K) -> Net-(D115-A)
- MX109 pad 2: COL9 -> COL8
- MX110 pad 1: Net-(D110-K) -> Net-(D117-A)
- MX12 pad 1: Net-(D12-K) -> Net-(D12-A)
- MX14 pad 1: Net-(D14-K) -> Net-(D14-A)
- MX16 pad 1: Net-(D16-K) -> Net-(D16-A)
- MX18 pad 1: Net-(D18-K) -> Net-(D18-A)
- MX20 pad 1: Net-(D20-K) -> Net-(D20-A)
- MX30 pad 1: Net-(D30-K) -> Net-(D30-A)
- MX32 pad 1: Net-(D32-K) -> Net-(D32-A)
- MX34 pad 1: Net-(D34-K) -> Net-(D34-A)
- MX36 pad 1: Net-(D36-K) -> Net-(D36-A)
- MX38 pad 1: Net-(D38-K) -> Net-(D38-A)
- MX40 pad 1: Net-(D40-K) -> Net-(D40-A)
- MX50 pad 1: Net-(D49-K) (its old number) -> Net-(D50-A)
- MX52 pad 1: Net-(D51-K) (its old number) -> Net-(D52-A)
- MX54 pad 1: Net-(D53-K) (its old number) -> Net-(D54-A)
- MX56 pad 1: Net-(D55-K) (its old number) -> Net-(D56-A)
- MX58 pad 1: Net-(D57-K) (its old number) -> Net-(D58-A)
- MX60 pad 1: Net-(D59-K) (its old number) -> Net-(D60-A)
- MX62 pad 2: COL0 -> COL1
- MX64 pad 2: COL1 -> COL2
- MX66 pad 2: COL4 -> COL3
- MX67 pad 1: Net-(D67-K) (its old number) -> Net-(D69-A)
- MX68 pad 2: COL5 -> COL4
- MX69 pad 1: Net-(D69-K) -> Net-(D71-A)
- MX70 pad 2: COL6 -> COL5
- MX71 pad 1: Net-(D71-K) -> Net-(D73-A)
- MX72 pad 2: COL7 -> COL6
- MX73 pad 1: Net-(D73-K) -> Net-(D75-A)
- MX74 pad 2: COL8 -> COL7
- MX75 pad 1: Net-(D75-K) -> Net-(D77-A)
- MX76 pad 2: COL9 -> COL8
- MX77 pad 1: Net-(D77-K) -> Net-(D79-A)
- MX83 pad 2: COL1 -> COL2
- MX85 pad 2: COL4 -> COL3
- MX86 pad 1: Net-(D85-K) -> Net-(D88-A)
- MX87 pad 2: COL5 -> COL4
- MX88 pad 1: Net-(D87-K) (its old number) -> Net-(D90-A)
- MX89 pad 2: COL6 -> COL5
- MX90 pad 1: Net-(D89-K) (its old number) -> Net-(D92-A)
- MX91 pad 2: COL7 -> COL6
- MX92 pad 1: Net-(D91-K) (its old number) -> Net-(D94-A)
- MX93 pad 2: COL8 -> COL7
- MX94 pad 1: Net-(D93-K) (its old number) -> Net-(D96-A)
- MX95 pad 2: COL9 -> COL8
- MX96 pad 1: Net-(D95-K) (its old number) -> Net-(D98-A)
- MX98 pad 1: Net-(D97-A) -> Net-(D101-K)
- MX98 pad 2: COL0 -> COL1
- MX99 pad 1: Net-(D98-K) -> Net-(D102-A)
- S1 pad 7: COL2 -> ROW5

Commit message: update new design
Parts:
- removed D117: D, Keyboard:D_SOD-123F
- added LED111: MX_SK6803MINI-E, Keyboard:LED_MX_6028R-ROT, B.Cu at (433.4, 133.0)
- added LED112: MX_SK6803MINI-E, Keyboard:LED_MX_6028R-ROT, B.Cu at (452.4, 133.0)
- added LED113: MX_SK6803MINI-E, Keyboard:LED_MX_6028R-ROT, B.Cu at (471.5, 133.0)
- added MX111: MX_SW_HS, Keyboard:SW_MX_HS_1u, B.Cu at (433.4, 138.1)
- added MX112: MX_SW_HS, Keyboard:SW_MX_HS_1u, B.Cu at (452.4, 138.1)
- added MX113: MX_SW_HS, Keyboard:SW_MX_HS_1u, B.Cu at (471.5, 138.1)
- LED100, LED101, LED102, LED103, LED104, LED105, LED106, LED107, LED108, LED109, LED110, LED39, LED60, LED61, LED62, LED63, LED64, LED65, LED66, LED67, LED68, LED69, LED70, LED71, LED72, LED73, LED74, LED75, LED76, LED77, LED78, LED79: footprint Keyboard:LED_MX_6028R -> Keyboard:LED_MX_6028R-ROT
- MX100, MX101, MX102, MX104: footprint Keyboard:SW_MX_HS_1.25u -> Keyboard:SW_MX_HS_1u
- MX103: footprint Keyboard:SW_MX_HS_2.75u -> Keyboard:SW_MX_HS_1u
- MX105, MX77, MX85: footprint Keyboard:SW_MX_HS_2.25u -> Keyboard:SW_MX_HS_1u
- MX106, MX107, MX48, MX61: footprint Keyboard:SW_MX_HS_1.5u -> Keyboard:SW_MX_HS_1u
- MX40, MX99: footprint Keyboard:SW_MX_HS_2u -> Keyboard:SW_MX_HS_1u
- MX42, MX47, MX79, MX84: footprint Keyboard:SW_MX_HS_2u_Vertical -> Keyboard:SW_MX_HS_1u
- MX65, MX96: footprint Keyboard:SW_MX_HS_1.75u -> Keyboard:SW_MX_HS_1u
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Connections:
- D1 pad 1: Net-(D1-K) -> ROW0
- D1 pad 2: ROW0 -> Net-(D1-A)
- D10 pad 1: ROW0 -> Net-(D10-K)
- D10 pad 2: Net-(D10-A) -> ROW0
- D100 pad 1: ROW5 -> Net-(D100-K)
- D100 pad 2: RKJ-PUSH -> ROW5
- D102 pad 1: ROW5 -> Net-(D102-K)
- D102 pad 2: Net-(D102-A) -> ROW5
- D103 pad 1: RKJ-A -> ROW5
- D103 pad 2: ROW5 -> Net-(D103-A)
- D104 pad 1: ROW5 -> Net-(D104-K)
- D104 pad 2: RKJ-D -> ROW5
- D105 pad 1: Net-(D105-K) -> ROW5
- D105 pad 2: ROW5 -> Net-(D105-A)
- D106 pad 1: ROW5 -> Net-(D106-K)
- D106 pad 2: Net-(D106-A) -> ROW5
- D107 pad 1: ROW5 -> Net-(D107-K)
- D107 pad 2: Net-(D107-A) -> ROW5
- D108 pad 1: RKJ-B -> Net-(D108-K)
- D109 pad 1: ROW5 -> Net-(D109-K)
- D109 pad 2: Net-(D109-A) -> ROW5
- D11 pad 1: Net-(D11-K) -> ROW0
- D11 pad 2: ROW0 -> Net-(D11-A)
- D110 pad 1: RKJ-C -> Net-(D110-K)
- D113 pad 1: ROW5 -> ROT1_D
- D113 pad 2: Net-(D113-A) -> ROW0
- D114 pad 1: Net-(D114-K) -> ROW3
- D114 pad 2: ROW5 -> ROT2_D
- D115 pad 2: Net-(D115-A) -> COM
- D116 pad 1: Net-(D116-K) -> ROW5
- D116 pad 2: ROW5 -> Net-(D116-A)
- D12 pad 1: ROW0 -> Net-(D12-K)
- D12 pad 2: Net-(D12-A) -> ROW0
- D13 pad 1: Net-(D13-K) -> ROW0
- D13 pad 2: ROW0 -> Net-(D13-A)
- D14 pad 1: ROW0 -> Net-(D14-K)
- D14 pad 2: Net-(D14-A) -> ROW0
- D15 pad 1: Net-(D15-K) -> ROW0
- D15 pad 2: ROW0 -> Net-(D15-A)
- D16 pad 1: ROW0 -> Net-(D16-K)
- D16 pad 2: Net-(D16-A) -> ROW0
- D17 pad 1: Net-(D17-K) -> ROW0
- D17 pad 2: ROW0 -> Net-(D17-A)
- D18 pad 1: ROW0 -> Net-(D18-K)
- D18 pad 2: Net-(D18-A) -> ROW0
- D19 pad 1: Net-(D19-K) -> ROW0
- D19 pad 2: ROW0 -> Net-(D19-A)
- D2 pad 1: ROW0 -> Net-(D2-K)
- D2 pad 2: Net-(D2-A) -> ROW0
- D20 pad 1: ROW0 -> Net-(D20-K)
- D20 pad 2: Net-(D20-A) -> ROW1
- D21 pad 1: Net-(D21-K) -> ROW1
- D21 pad 2: ROW1 -> Net-(D21-A)
- D22 pad 1: ROW1 -> Net-(D22-K)
- D22 pad 2: Net-(D22-A) -> ROW1
- D24 pad 1: ROW1 -> Net-(D24-K)
- D24 pad 2: Net-(D24-A) -> ROW1
- D25 pad 1: Net-(D25-K) -> ROW1
- D25 pad 2: ROW1 -> Net-(D25-A)
- D26 pad 1: ROW1 -> Net-(D26-K)
- D26 pad 2: Net-(D26-A) -> ROW1
- D27 pad 1: Net-(D27-K) -> ROW1
- D27 pad 2: ROW1 -> Net-(D27-A)
- D28 pad 1: ROW1 -> Net-(D28-K)
- D28 pad 2: Net-(D28-A) -> ROW1
- D29 pad 1: Net-(D29-K) -> ROW1
- D29 pad 2: ROW1 -> Net-(D29-A)
- D3 pad 1: Net-(D3-K) -> ROW0
- D3 pad 2: ROW0 -> Net-(D3-A)
- D30 pad 1: ROW1 -> Net-(D30-K)
- D30 pad 2: Net-(D30-A) -> ROW1
- D31 pad 1: Net-(D31-K) -> ROW1
- D31 pad 2: ROW1 -> Net-(D31-A)
- D32 pad 1: ROW1 -> Net-(D32-K)
- D32 pad 2: Net-(D32-A) -> ROW1
- D33 pad 1: Net-(D33-K) -> ROW1
- D33 pad 2: ROW1 -> Net-(D33-A)
- D34 pad 1: ROW1 -> Net-(D34-K)
- D34 pad 2: Net-(D34-A) -> ROW1
- D35 pad 1: Net-(D35-K) -> ROW1
- D35 pad 2: ROW1 -> Net-(D35-A)
- D36 pad 1: ROW1 -> Net-(D36-K)
- D36 pad 2: Net-(D36-A) -> ROW1
- D37 pad 1: Net-(D37-K) -> ROW1
- D37 pad 2: ROW1 -> Net-(D37-A)
- D38 pad 1: ROW1 -> Net-(D38-K)
- D38 pad 2: Net-(D38-A) -> ROW1
- D39 pad 1: Net-(D39-K) -> ROW1
- D39 pad 2: ROW1 -> Net-(D39-A)
- D4 pad 1: ROW0 -> Net-(D4-K)
- D4 pad 2: Net-(D4-A) -> ROW0
- D40 pad 1: ROW1 -> Net-(D40-K)
- D40 pad 2: Net-(D40-A) -> ROW2
- D41 pad 1: Net-(D41-K) -> ROW2
- D41 pad 2: ROW2 -> Net-(D41-A)
- D42 pad 1: ROW2 -> Net-(D42-K)
- D42 pad 2: Net-(D42-A) -> ROW2
- D43 pad 1: Net-(D43-K) -> ROW2
- D43 pad 2: ROW2 -> Net-(D43-A)
- D44 pad 1: ROW2 -> Net-(D44-K)
- D44 pad 2: Net-(D44-A) -> ROW2
- D45 pad 1: Net-(D45-K) -> ROW2
- D45 pad 2: ROW2 -> Net-(D45-A)
- D47 pad 1: Net-(D47-K) -> ROW2
- D47 pad 2: ROW2 -> Net-(D47-A)
- D48 pad 1: ROW2 -> Net-(D48-K)
- D48 pad 2: Net-(D48-A) -> ROW2
- D49 pad 1: Net-(D49-K) -> ROW2
- D49 pad 2: ROW2 -> Net-(D49-A)
- D5 pad 1: Net-(D5-K) -> ROW0
- D5 pad 2: ROW0 -> Net-(D5-A)
- D50 pad 1: ROW2 -> Net-(D50-K)
- D50 pad 2: Net-(D50-A) -> ROW2
- D51 pad 1: Net-(D51-K) -> ROW2
- D51 pad 2: ROW2 -> Net-(D51-A)
- D52 pad 1: ROW2 -> Net-(D52-K)
- D52 pad 2: Net-(D52-A) -> ROW2
- D53 pad 1: Net-(D53-K) -> ROW2
- D53 pad 2: ROW2 -> Net-(D53-A)
- D54 pad 1: ROW2 -> Net-(D54-K)
- D54 pad 2: Net-(D54-A) -> ROW2
- D55 pad 1: Net-(D55-K) -> ROW2
- D55 pad 2: ROW2 -> Net-(D55-A)
- D56 pad 1: ROW2 -> Net-(D56-K)
- D56 pad 2: Net-(D56-A) -> ROW2
- D57 pad 1: Net-(D57-K) -> ROW2
- D57 pad 2: ROW2 -> Net-(D57-A)
- D58 pad 1: ROW2 -> Net-(D58-K)
- D58 pad 2: Net-(D58-A) -> ROW2
- D59 pad 1: Net-(D59-K) -> ROW2
- D59 pad 2: ROW2 -> Net-(D59-A)
- D6 pad 1: ROW0 -> Net-(D6-K)
- D6 pad 2: Net-(D6-A) -> ROW0
- D60 pad 1: ROW2 -> Net-(D60-K)
- D60 pad 2: Net-(D60-A) -> ROW3
- D61 pad 1: Net-(D61-K) -> ROW3
- D61 pad 2: ROW3 -> Net-(D61-A)
- D62 pad 1: ROW3 -> Net-(D62-K)
- D62 pad 2: ROT1_D -> ROW3
- D66 pad 1: ROT2_D -> Net-(D66-K)
- D67 pad 1: Net-(D67-K) -> ROW3
- D67 pad 2: ROW3 -> Net-(D67-A)
- D68 pad 1: ROW3 -> Net-(D68-K)
- D68 pad 2: Net-(D68-A) -> ROW3
- D7 pad 1: Net-(D7-K) -> ROW0
- D7 pad 2: ROW0 -> Net-(D7-A)
- D8 pad 1: ROW0 -> Net-(D8-K)
- D8 pad 2: Net-(D8-A) -> ROW0
- D87 pad 1: Net-(D87-K) -> ROW4
- D87 pad 2: ROW4 -> Net-(D87-A)
- D88 pad 1: ROW4 -> Net-(D88-K)
- D88 pad 2: Net-(D88-A) -> ROW4
- D89 pad 1: Net-(D89-K) -> ROW4
- D89 pad 2: ROW4 -> Net-(D89-A)
- D9 pad 1: Net-(D9-K) -> ROW0
- D9 pad 2: ROW0 -> Net-(D9-A)
- D90 pad 1: ROW4 -> Net-(D90-K)
- D90 pad 2: Net-(D90-A) -> ROW4
- D91 pad 1: Net-(D91-K) -> ROW4
- D91 pad 2: ROW4 -> Net-(D91-A)
- D92 pad 1: ROW4 -> Net-(D92-K)
- D92 pad 2: Net-(D92-A) -> ROW4
- D93 pad 1: Net-(D93-K) -> ROW4
- D93 pad 2: ROW4 -> Net-(D93-A)
- D94 pad 1: ROW4 -> Net-(D94-K)
- D94 pad 2: Net-(D94-A) -> ROW4
- D95 pad 1: Net-(D95-K) -> ROW4
- D95 pad 2: ROW4 -> Net-(D95-A)
- D96 pad 1: ROW4 -> Net-(D96-K)
- D96 pad 2: Net-(D96-A) -> ROW4
- D97 pad 1: Net-(D97-K) -> ROW4
- D97 pad 2: ROW4 -> Net-(D97-A)
- D98 pad 1: ROW4 -> Net-(D98-K)
- D98 pad 2: Net-(D98-A) -> ROW4
- D99 pad 1: Net-(D99-K) -> ROW4
- D99 pad 2: ROW5 -> Net-(D99-A)
- LED10 pad 2: unconnected-(LED10-DOUT-Pad2) -> Net-(LED10-DOUT)
- LED10 pad 3: unconnected-(LED10-DIN-Pad3) -> Net-(LED10-DIN)
- LED100 pad 2: Net-(LED100-DOUT) -> unconnected-(LED100-DOUT-Pad2)
- LED11 pad 2: unconnected-(LED11-DOUT-Pad2) -> Net-(LED11-DOUT)
- LED11 pad 3: unconnected-(LED11-DIN-Pad3) -> Net-(LED10-DOUT)
- LED12 pad 2: unconnected-(LED12-DOUT-Pad2) -> Net-(LED12-DOUT)
- LED12 pad 3: unconnected-(LED12-DIN-Pad3) -> Net-(LED11-DOUT)
- LED13 pad 2: unconnected-(LED13-DOUT-Pad2) -> Net-(LED13-DOUT)
- LED13 pad 3: unconnected-(LED13-DIN-Pad3) -> Net-(LED12-DOUT)
- LED14 pad 2: unconnected-(LED14-DOUT-Pad2) -> Net-(LED14-DOUT)
- LED14 pad 3: unconnected-(LED14-DIN-Pad3) -> Net-(LED13-DOUT)
- LED15 pad 2: unconnected-(LED15-DOUT-Pad2) -> Net-(LED15-DOUT)
- LED15 pad 3: unconnected-(LED15-DIN-Pad3) -> Net-(LED14-DOUT)
- LED16 pad 2: unconnected-(LED16-DOUT-Pad2) -> Net-(LED16-DOUT)
- LED16 pad 3: unconnected-(LED16-DIN-Pad3) -> Net-(LED15-DOUT)
- LED17 pad 2: unconnected-(LED17-DOUT-Pad2) -> Net-(LED17-DOUT)
- LED17 pad 3: unconnected-(LED17-DIN-Pad3) -> Net-(LED16-DOUT)
- LED18 pad 2: unconnected-(LED18-DOUT-Pad2) -> Net-(LED18-DOUT)
- LED18 pad 3: unconnected-(LED18-DIN-Pad3) -> Net-(LED17-DOUT)
- LED19 pad 3: unconnected-(LED19-DIN-Pad3) -> Net-(LED18-DOUT)
- LED38 pad 3: Net-(LED19-DOUT) -> Net-(LED38-DIN)
- LED39 pad 1: LED_PWR -> GND
- LED39 pad 2: Net-(LED39-DOUT) -> Net-(LED38-DIN)
- LED39 pad 3: Net-(LED20-DOUT) -> Net-(LED19-DOUT)
- LED39 pad 4: GND -> LED_PWR
- LED40 pad 3: Net-(LED39-DOUT) -> Net-(LED20-DOUT)
- LED45 pad 2: unconnected-(LED45-DOUT-Pad2) -> Net-(LED45-DOUT)
- LED46 pad 3: unconnected-(LED46-DIN-Pad3) -> Net-(LED45-DOUT)
- LED57 pad 2: Net-(LED57-DOUT) -> unconnected-(LED57-DOUT-Pad2)
- LED58 pad 1: GND -> LED_PWR
- LED58 pad 2: Net-(LED58-DOUT) -> unconnected-(LED58-DOUT-Pad2)
- LED58 pad 3: Net-(LED58-DIN) -> unconnected-(LED58-DIN-Pad3)
- LED58 pad 4: LED_PWR -> GND
- LED59 pad 1: GND -> LED_PWR
- LED59 pad 2: Net-(LED58-DIN) -> Net-(LED59-DOUT)
- LED59 pad 3: Net-(LED59-DIN) -> unconnected-(LED59-DIN-Pad3)
- LED59 pad 4: LED_PWR -> GND
- LED60 pad 2: Net-(LED59-DIN) -> Net-(LED60-DOUT)
- LED7 pad 2: unconnected-(LED7-DOUT-Pad2) -> Net-(LED7-DOUT)
- LED75 pad 3: Net-(LED57-DOUT) -> Net-(LED75-DIN)
- LED76 pad 1: LED_PWR -> GND
- LED76 pad 2: Net-(LED76-DOUT) -> Net-(LED75-DIN)
- LED76 pad 3: Net-(LED58-DOUT) -> Net-(LED76-DIN)
- LED76 pad 4: GND -> LED_PWR
- LED77 pad 1: LED_PWR -> GND
- LED77 pad 2: Net-(LED77-DOUT) -> Net-(LED76-DIN)
- LED77 pad 3: Net-(LED76-DOUT) -> Net-(LED77-DIN)
- LED77 pad 4: GND -> LED_PWR
- LED78 pad 1: LED_PWR -> GND
- LED78 pad 2: Net-(LED78-DOUT) -> Net-(LED77-DIN)
- LED78 pad 3: Net-(LED77-DOUT) -> unconnected-(LED78-DIN-Pad3)
- LED78 pad 4: GND -> LED_PWR
- LED79 pad 1: LED_PWR -> unconnected-(LED79-VDD-Pad1)
- LED79 pad 2: Net-(LED79-DOUT) -> unconnected-(LED79-DOUT-Pad2)
- LED79 pad 3: Net-(LED78-DOUT) -> Net-(LED59-DOUT)
- LED79 pad 4: GND -> unconnected-(LED79-VSS-Pad4)
- LED8 pad 2: unconnected-(LED8-DOUT-Pad2) -> Net-(LED8-DOUT)
- LED8 pad 3: unconnected-(LED8-DIN-Pad3) -> Net-(LED7-DOUT)
- LED80 pad 3: Net-(LED79-DOUT) -> Net-(LED60-DOUT)
- LED82 pad 2: unconnected-(LED82-DOUT-Pad2) -> Net-(LED82-DOUT)
- LED83 pad 2: unconnected-(LED83-DOUT-Pad2) -> Net-(LED83-DOUT)
- LED83 pad 3: unconnected-(LED83-DIN-Pad3) -> Net-(LED82-DOUT)
- LED84 pad 2: unconnected-(LED84-DOUT-Pad2) -> Net-(LED84-DOUT)
- LED84 pad 3: unconnected-(LED84-DIN-Pad3) -> Net-(LED83-DOUT)
- LED85 pad 2: unconnected-(LED85-DOUT-Pad2) -> Net-(LED85-DOUT)
- LED85 pad 3: unconnected-(LED85-DIN-Pad3) -> Net-(LED84-DOUT)
- LED86 pad 2: unconnected-(LED86-DOUT-Pad2) -> Net-(LED86-DOUT)
- LED86 pad 3: unconnected-(LED86-DIN-Pad3) -> Net-(LED85-DOUT)
- LED87 pad 3: unconnected-(LED87-DIN-Pad3) -> Net-(LED86-DOUT)
- LED9 pad 2: unconnected-(LED9-DOUT-Pad2) -> Net-(LED10-DIN)
- LED9 pad 3: unconnected-(LED9-DIN-Pad3) -> Net-(LED8-DOUT)
- LED93 pad 2: Net-(LED110-DIN) -> unconnected-(LED93-DOUT-Pad2)
- LED94 pad 1: GND -> LED_PWR
- LED94 pad 3: Net-(LED94-DIN) -> unconnected-(LED94-DIN-Pad3)
- LED94 pad 4: LED_PWR -> GND
- LED95 pad 1: GND -> LED_PWR
- LED95 pad 2: Net-(LED94-DIN) -> unconnected-(LED95-DOUT-Pad2)
- LED95 pad 3: Net-(LED95-DIN) -> unconnected-(LED95-DIN-Pad3)
- LED95 pad 4: LED_PWR -> GND
- LED96 pad 1: GND -> LED_PWR
- LED96 pad 2: Net-(LED95-DIN) -> unconnected-(LED96-DOUT-Pad2)
- LED96 pad 3: Net-(LED96-DIN) -> unconnected-(LED96-DIN-Pad3)
- LED96 pad 4: LED_PWR -> GND
- LED97 pad 1: GND -> LED_PWR
- LED97 pad 2: Net-(LED96-DIN) -> unconnected-(LED97-DOUT-Pad2)
- LED97 pad 3: Net-(LED97-DIN) -> unconnected-(LED97-DIN-Pad3)
- LED97 pad 4: LED_PWR -> GND
- LED98 pad 1: GND -> LED_PWR
- LED98 pad 2: Net-(LED97-DIN) -> Net-(LED98-DOUT)
- LED98 pad 3: Net-(LED98-DIN) -> unconnected-(LED98-DIN-Pad3)
- LED98 pad 4: LED_PWR -> GND
- LED99 pad 1: GND -> LED_PWR
- LED99 pad 2: Net-(LED98-DIN) -> Net-(LED113-DIN)
- LED99 pad 3: Net-(LED100-DOUT) -> Net-(LED98-DOUT)
- LED99 pad 4: LED_PWR -> GND
- MX1 pad 1: Net-(D1-K) -> COL0
- MX1 pad 2: COL0 -> Net-(D1-A)
- MX10 pad 1: Net-(D10-A) -> COL5
- MX10 pad 2: COL4 -> Net-(D10-K)
- MX100 pad 1: Net-(D105-K) -> COL0
- MX100 pad 2: COL3 -> Net-(D100-K)
- MX101 pad 1: Net-(D106-A) -> COL1
- MX101 pad 2: COL3 -> Net-(D101-K)
- MX102 pad 1: Net-(D107-A) -> COL2
- MX102 pad 2: COL4 -> Net-(D102-K)
- MX103 pad 1: Net-(D109-A) -> COL2
- MX103 pad 2: COL5 -> Net-(D103-A)
- MX104 pad 1: Net-(D111-A) -> COL3
- MX104 pad 2: COL6 -> Net-(D104-K)
- MX105 pad 1: Net-(D112-K) -> COL3
- MX105 pad 2: COL6 -> Net-(D105-A)
- MX106 pad 1: Net-(D113-A) -> COL4
- MX106 pad 2: COL7 -> Net-(D106-K)
- MX107 pad 1: Net-(D114-K) -> COL5
- MX107 pad 2: COL7 -> Net-(D107-K)
- MX108 pad 1: Net-(D115-A) -> COL6
- MX108 pad 2: COL8 -> Net-(D108-K)
- MX109 pad 1: Net-(D116-K) -> COL7
- MX109 pad 2: COL8 -> Net-(D109-K)
- MX11 pad 1: Net-(D11-K) -> COL5
- MX11 pad 2: COL5 -> Net-(D11-A)
- MX110 pad 1: Net-(D117-A) -> COL8
- MX110 pad 2: COL9 -> Net-(D110-K)
- MX12 pad 1: Net-(D12-A) -> COL6
- MX12 pad 2: COL5 -> Net-(D12-K)
- MX13 pad 1: Net-(D13-K) -> COL6
- MX13 pad 2: COL6 -> Net-(D13-A)
- MX14 pad 1: Net-(D14-A) -> COL7
- MX14 pad 2: COL6 -> Net-(D14-K)
- MX15 pad 1: Net-(D15-K) -> COL7
- MX15 pad 2: COL7 -> Net-(D15-A)
- MX16 pad 1: Net-(D16-A) -> COL8
- MX16 pad 2: COL7 -> Net-(D16-K)
- MX17 pad 1: Net-(D17-K) -> COL8
- MX17 pad 2: COL8 -> Net-(D17-A)
- MX18 pad 1: Net-(D18-A) -> COL9
- MX18 pad 2: COL8 -> Net-(D18-K)
- MX19 pad 1: Net-(D19-K) -> COL9
- MX19 pad 2: COL9 -> Net-(D19-A)
- MX2 pad 1: Net-(D2-A) -> COL1
- MX2 pad 2: COL0 -> Net-(D2-K)
- MX20 pad 1: Net-(D20-A) -> COL0
- MX20 pad 2: COL9 -> Net-(D20-K)
- MX21 pad 1: Net-(D21-K) -> COL0
- MX21 pad 2: COL0 -> Net-(D21-A)
- MX22 pad 1: Net-(D22-A) -> COL1
- MX22 pad 2: COL0 -> Net-(D22-K)
- MX23 pad 1: Net-(D23-K) -> COL1
- MX23 pad 2: COL1 -> Net-(D23-K)
- MX24 pad 1: Net-(D24-A) -> COL2
- MX24 pad 2: COL1 -> Net-(D24-K)
- MX25 pad 1: Net-(D25-K) -> COL2
- MX25 pad 2: COL2 -> Net-(D25-A)
- MX26 pad 1: Net-(D26-A) -> COL3
- MX26 pad 2: COL2 -> Net-(D26-K)
- MX27 pad 1: Net-(D27-K) -> COL3
- MX27 pad 2: COL3 -> Net-(D27-A)
- MX28 pad 1: Net-(D28-A) -> COL4
- MX28 pad 2: COL3 -> Net-(D28-K)
- MX29 pad 1: Net-(D29-K) -> COL4
- MX29 pad 2: COL4 -> Net-(D29-A)
- MX3 pad 1: Net-(D3-K) -> COL1
- MX3 pad 2: COL1 -> Net-(D3-A)
- MX30 pad 1: Net-(D30-A) -> COL5
- MX30 pad 2: COL4 -> Net-(D30-K)
- MX31 pad 1: Net-(D31-K) -> COL5
- MX31 pad 2: COL5 -> Net-(D31-A)
- MX32 pad 1: Net-(D32-A) -> COL6
- MX32 pad 2: COL5 -> Net-(D32-K)
- MX33 pad 1: Net-(D33-K) -> COL6
- MX33 pad 2: COL6 -> Net-(D33-A)
- MX34 pad 1: Net-(D34-A) -> COL7
- MX34 pad 2: COL6 -> Net-(D34-K)
- MX35 pad 1: Net-(D35-K) -> COL7
- MX35 pad 2: COL7 -> Net-(D35-A)
- MX36 pad 1: Net-(D36-A) -> COL8
- MX36 pad 2: COL7 -> Net-(D36-K)
- MX37 pad 1: Net-(D37-K) -> COL8
- MX37 pad 2: COL8 -> Net-(D37-A)
- MX38 pad 1: Net-(D38-A) -> COL9
- MX38 pad 2: COL8 -> Net-(D38-K)
- MX39 pad 1: Net-(D39-K) -> COL9
- MX39 pad 2: COL9 -> Net-(D39-A)
- MX4 pad 1: Net-(D4-A) -> COL2
- MX4 pad 2: COL1 -> Net-(D4-K)
- MX40 pad 1: Net-(D40-A) -> COL0
- MX40 pad 2: COL9 -> Net-(D40-K)
- MX41 pad 1: Net-(D41-K) -> COL0
- MX41 pad 2: COL0 -> Net-(D41-A)
- MX42 pad 1: Net-(D42-A) -> COL1
- MX42 pad 2: COL0 -> Net-(D42-K)
- MX43 pad 1: Net-(D43-K) -> COL1
- MX43 pad 2: COL1 -> Net-(D43-A)
- MX44 pad 1: Net-(D44-A) -> COL2
- MX44 pad 2: COL1 -> Net-(D44-K)
- MX45 pad 1: Net-(D45-K) -> COL2
- MX45 pad 2: COL2 -> Net-(D45-A)
- MX46 pad 1: Net-(D46-K) -> COL3
- MX46 pad 2: COL2 -> Net-(D46-K)
- MX47 pad 1: Net-(D47-K) -> COL3
- MX47 pad 2: COL3 -> Net-(D47-A)
- MX48 pad 1: Net-(D48-A) -> COL4
- MX48 pad 2: COL3 -> Net-(D48-K)
- MX49 pad 1: Net-(D49-K) -> COL4
- MX49 pad 2: COL4 -> Net-(D49-A)
- MX5 pad 1: Net-(D5-K) -> COL2
- MX5 pad 2: COL2 -> Net-(D5-A)
- MX50 pad 1: Net-(D50-A) -> COL5
- MX50 pad 2: COL4 -> Net-(D50-K)
- MX51 pad 1: Net-(D51-K) -> COL5
- MX51 pad 2: COL5 -> Net-(D51-A)
- MX52 pad 1: Net-(D52-A) -> COL6
- MX52 pad 2: COL5 -> Net-(D52-K)
- MX53 pad 1: Net-(D53-K) -> COL6
- MX53 pad 2: COL6 -> Net-(D53-A)
- MX54 pad 1: Net-(D54-A) -> COL7
- MX54 pad 2: COL6 -> Net-(D54-K)
- MX55 pad 1: Net-(D55-K) -> COL7
- MX55 pad 2: COL7 -> Net-(D55-A)
- MX56 pad 1: Net-(D56-A) -> COL8
- MX56 pad 2: COL7 -> Net-(D56-K)
- MX57 pad 1: Net-(D57-K) -> COL8
- MX57 pad 2: COL8 -> Net-(D57-A)
- MX58 pad 1: Net-(D58-A) -> COL9
- MX58 pad 2: COL8 -> Net-(D58-K)
- MX59 pad 1: Net-(D59-K) -> COL9
- MX59 pad 2: COL9 -> Net-(D59-A)
- MX6 pad 1: Net-(D6-A) -> COL3
- MX6 pad 2: COL2 -> Net-(D6-K)
- MX60 pad 1: Net-(D60-A) -> COL0
- MX60 pad 2: COL9 -> Net-(D60-K)
- MX61 pad 1: Net-(D61-K) -> COL0
- MX61 pad 2: COL0 -> Net-(D61-A)
- MX62 pad 1: Net-(D63-A) -> COL1
- MX62 pad 2: COL1 -> Net-(D62-K)
- MX63 pad 1: Net-(D64-K) -> COL1
- MX63 pad 2: COL1 -> Net-(D63-A)
- MX64 pad 1: Net-(D65-A) -> COL2
- MX64 pad 2: COL2 -> Net-(D64-K)
- MX65 pad 1: Net-(D67-K) -> COL2
- MX65 pad 2: COL3 -> Net-(D65-A)
- MX66 pad 1: Net-(D68-A) -> COL3
- MX66 pad 2: COL3 -> Net-(D66-K)
- MX67 pad 1: Net-(D69-A) -> COL3
- MX67 pad 2: COL4 -> Net-(D67-A)
- MX68 pad 1: Net-(D70-K) -> COL4
- MX68 pad 2: COL4 -> Net-(D68-K)
- MX69 pad 1: Net-(D71-A) -> COL4
- MX69 pad 2: COL5 -> Net-(D69-A)
- MX7 pad 1: Net-(D7-K) -> COL3
- MX7 pad 2: COL3 -> Net-(D7-A)
- MX70 pad 1: Net-(D72-K) -> COL5
- MX70 pad 2: COL5 -> Net-(D70-K)
- MX71 pad 1: Net-(D73-A) -> COL5
- MX71 pad 2: COL6 -> Net-(D71-A)
- MX72 pad 1: Net-(D74-K) -> COL6
- MX72 pad 2: COL6 -> Net-(D72-K)
- MX73 pad 1: Net-(D75-A) -> COL6
- MX73 pad 2: COL7 -> Net-(D73-A)
- MX74 pad 1: Net-(D76-K) -> COL7
- MX74 pad 2: COL7 -> Net-(D74-K)
- MX75 pad 1: Net-(D77-A) -> COL7
- MX75 pad 2: COL8 -> Net-(D75-A)
- MX76 pad 1: Net-(D78-K) -> COL8
- MX76 pad 2: COL8 -> Net-(D76-K)
- MX77 pad 1: Net-(D79-A) -> COL8
- MX77 pad 2: COL9 -> Net-(D77-A)
- MX78 pad 1: Net-(D80-K) -> COL9
- MX78 pad 2: COL0 -> Net-(D78-K)
- MX79 pad 1: Net-(D81-A) -> COL9
- MX79 pad 2: COL0 -> Net-(D79-A)
- MX8 pad 1: Net-(D8-A) -> COL4
- MX8 pad 2: COL3 -> Net-(D8-K)
- MX80 pad 1: Net-(D82-K) -> COL0
- MX80 pad 2: COL1 -> Net-(D80-K)
- MX81 pad 1: Net-(D83-A) -> COL0
- MX81 pad 2: COL1 -> Net-(D81-A)
- MX82 pad 1: Net-(D84-K) -> COL1
- MX82 pad 2: COL2 -> Net-(D82-K)
- MX83 pad 1: Net-(D85-A) -> COL1
- MX83 pad 2: COL2 -> Net-(D83-A)
- MX84 pad 1: Net-(D86-K) -> COL2
- MX84 pad 2: COL3 -> Net-(D84-K)
- MX85 pad 1: Net-(D87-K) -> COL2
- MX85 pad 2: COL3 -> Net-(D85-A)
- MX86 pad 1: Net-(D88-A) -> COL3
- MX86 pad 2: COL4 -> Net-(D86-K)
- MX87 pad 1: Net-(D89-K) -> COL3
- MX87 pad 2: COL4 -> Net-(D87-A)
- MX88 pad 1: Net-(D90-A) -> COL4
- MX88 pad 2: COL5 -> Net-(D88-K)
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Routing:
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Other:
- board text removed: "JLCJLCJLCJLC"

Commit message: check ing
Parts:
- removed D116: D, Keyboard:D_SOD-123F
- removed LED112, LED113: MX_SK6803MINI-E, Keyboard:LED_MX_6028R-ROT
- removed MX112, MX113: MX_SW_HS, Keyboard:SW_MX_HS_1u
- removed S1: RKJXT1F42001, Keyboard:RKJXT1F42001
- added C30: 100nF, Capacitor_SMD:C_0805_2012Metric, B.Cu at (-35.2, 49.5)
- added C31: 100nF, Capacitor_SMD:C_0805_2012Metric, B.Cu at (-35.2, 52.5)
- added C32: 100nF, Capacitor_SMD:C_0805_2012Metric, B.Cu at (-35.2, 55.5)
- added C33: 100nF, Capacitor_SMD:C_0805_2012Metric, B.Cu at (2.38, 42.9)
- added R21: 5.1k, Resistor_SMD:R_0805_2012Metric, B.Cu at (-30.8, 49.5)
- added R22: 5.1k, Resistor_SMD:R_0805_2012Metric, B.Cu at (-30.8, 52.5)
- added R23: 5.1k, Resistor_SMD:R_0805_2012Metric, B.Cu at (-30.8, 55.4)
- added R24: 5.1k, Resistor_SMD:R_0805_2012Metric, B.Cu at (-30.8, 58.4)
- added R25: 5.1k, Resistor_SMD:R_0805_2012Metric, B.Cu at (-30.8, 61.3)
- added R26: 5.1k, Resistor_SMD:R_0805_2012Metric, B.Cu at (-30.8, 64.2)
- added R27: 5.1k, Resistor_SMD:R_0805_2012Metric, B.Cu at (-30.8, 67.2)
- added R28: 5.1k, Resistor_SMD:R_0805_2012Metric, B.Cu at (-30.8, 70.2)
- added SW3: RotaryEncoder_Switch, Keyboard:RotaryEncoder_Alps_EC11E-Switch_Vertical_H20mm_Centred, F.Cu at (158.8, 38.1)
- added SW4: RKJXT1F42001, Keyboard:RKJXT1F42001, F.Cu at (147.4, 133.4)
- LED79: footprint Keyboard:LED_MX_6028R-ROT -> Keyboard:LED_MX_6028R
- LED98, LED99: footprint Keyboard:LED_MX_6028R -> Keyboard:LED_MX_6028R-ROT
- MX100, MX18, MX38: footprint Keyboard:SW_MX_HS_1u -> Keyboard:SW_MX_HS_2u
- MX101, MX102, MX103, MX105: footprint Keyboard:SW_MX_HS_1u -> Keyboard:SW_MX_HS_1.25u
- MX104: footprint Keyboard:SW_MX_HS_1u -> Keyboard:SW_MX_HS_2.75u
- MX106, MX77, MX84: footprint Keyboard:SW_MX_HS_1u -> Keyboard:SW_MX_HS_2.25u
- MX107, MX108, MX45, MX58: footprint Keyboard:SW_MX_HS_1u -> Keyboard:SW_MX_HS_1.5u
- MX65, MX95: footprint Keyboard:SW_MX_HS_1u -> Keyboard:SW_MX_HS_1.75u
- MX80: footprint Keyboard:SW_MX_HS_1u -> Keyboard:SW_MX_HS_2u_Vertical
- Q1: footprint Package_TO_SOT_SMD:SOT-23-3 -> Package_TO_SOT_SMD:SOT-23
- U1: footprint Package_TO_SOT_SMD:SOT-223-3_TabPin2 -> Package_TO_SOT_SMD:SOT-23-3
- U4: footprint Package_SO:SOIC-8_5.275x5.275mm_P1.27mm -> Package_SO:SOIC-8_5.23x5.23mm_P1.27mm
- U5: footprint Package_TO_SOT_SMD:SOT-143_Handsoldering -> Package_TO_SOT_SMD:SOT-143
- moved LED79 438.6 mm to (33.3, 114.0)
- moved MX79 438.6 mm to (33.3, 119.1)
- moved D79 438.5 mm to (28.7, 127.8)
- moved D112 431.0 mm to (28.7, 46.8)
- moved LED98 419.5 mm to (33.3, 133.0)
- moved MX98 419.5 mm to (33.3, 138.1)
- moved D98 419.5 mm to (28.7, 146.8)
- moved LED99 395.7 mm to (76.2, 133.0)
- moved MX99 395.7 mm to (76.2, 138.1)
- moved D99 395.7 mm to (71.5, 146.8)
- moved D114 235.3 mm to (129.0, 158.1)
- moved C27 159.8 mm to (46.8, 39.7), turned to 0 degrees
- moved C26 154.1 mm to (46.8, 36.5), turned to 0 degrees
- moved R14 151.0 mm to (46.8, 42.1)
- moved R8 142.5 mm to (46.8, 44.4), turned to 0 degrees
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Connections:
- D101 pad 1: Net-(D101-K) -> ROW5
- D101 pad 2: ROW5 -> Net-(D101-A)
- D105 pad 1: ROW5 -> Net-(D105-K)
- D105 pad 2: Net-(D105-A) -> ROW5
- D109 pad 1: Net-(D109-K) -> ROW5
- D109 pad 2: ROW5 -> Net-(D109-A)
- D112 pad 2: ROW5 -> ROW0
- D113 pad 1: ROT1_D -> ROW3
- D113 pad 2: ROW0 -> Net-(D113-A)
- D114 pad 2: ROT2_D -> Net-(D114-A)
- D65 pad 1: ROW3 -> Net-(D65-K)
- D65 pad 2: Net-(D65-A) -> ROW3
- D66 pad 1: Net-(D66-K) -> ROW3
- D66 pad 2: ROW3 -> Net-(D66-A)
- D67 pad 1: ROW3 -> Net-(D67-K)
- D67 pad 2: Net-(D67-A) -> ROW3
- D68 pad 1: Net-(D68-K) -> ROW3
- D68 pad 2: ROW3 -> Net-(D68-A)
- D69 pad 1: ROW3 -> Net-(D69-K)
- D69 pad 2: Net-(D69-A) -> ROW3
- D70 pad 1: Net-(D70-K) -> ROW3
- D70 pad 2: ROW3 -> Net-(D70-A)
- D71 pad 1: ROW3 -> Net-(D71-K)
- D71 pad 2: Net-(D71-A) -> ROW3
- D72 pad 1: Net-(D72-K) -> ROW3
- D72 pad 2: ROW3 -> Net-(D72-A)
- D73 pad 1: ROW3 -> Net-(D73-K)
- D73 pad 2: Net-(D73-A) -> ROW3
- D74 pad 1: Net-(D74-K) -> ROW3
- D74 pad 2: ROW3 -> Net-(D74-A)
- D75 pad 1: ROW3 -> Net-(D75-K)
- D75 pad 2: Net-(D75-A) -> ROW3
- D76 pad 1: Net-(D76-K) -> ROW3
- D76 pad 2: ROW3 -> Net-(D76-A)
- D77 pad 1: ROW3 -> Net-(D77-K)
- D77 pad 2: Net-(D77-A) -> ROW3
- D78 pad 1: Net-(D78-K) -> ROW3
- D78 pad 2: ROW3 -> Net-(D78-A)
- D79 pad 1: ROW3 -> Net-(D79-K)
- D79 pad 2: Net-(D79-A) -> ROW4
- D80 pad 1: Net-(D80-K) -> ROW4
- D80 pad 2: ROW4 -> Net-(D80-A)
- D81 pad 1: ROW4 -> Net-(D81-K)
- D81 pad 2: Net-(D81-A) -> ROW4
- D82 pad 1: Net-(D82-K) -> ROW4
- D82 pad 2: ROW4 -> Net-(D82-A)
- D83 pad 1: ROW4 -> Net-(D83-K)
- D83 pad 2: Net-(D83-A) -> ROW4
- D98 pad 2: ROW4 -> ROW5
- D99 pad 1: ROW4 -> Net-(D99-K)
- D99 pad 2: Net-(D99-A) -> ROW5
- LED100 pad 1: GND -> LED_PWR
- LED100 pad 4: LED_PWR -> GND
- LED101 pad 1: GND -> LED_PWR
- LED101 pad 4: LED_PWR -> GND
- LED102 pad 1: GND -> LED_PWR
- LED102 pad 4: LED_PWR -> GND
- LED103 pad 1: GND -> LED_PWR
- LED103 pad 4: LED_PWR -> GND
- LED104 pad 1: GND -> LED_PWR
- LED104 pad 4: LED_PWR -> GND
- LED105 pad 1: GND -> LED_PWR
- LED105 pad 4: LED_PWR -> GND
- LED106 pad 1: GND -> LED_PWR
- LED106 pad 4: LED_PWR -> GND
- LED107 pad 1: GND -> LED_PWR
- LED107 pad 4: LED_PWR -> GND
- LED108 pad 1: GND -> LED_PWR
- LED108 pad 4: LED_PWR -> GND
- LED109 pad 1: GND -> LED_PWR
- LED109 pad 4: LED_PWR -> GND
- LED110 pad 1: GND -> LED_PWR
- LED110 pad 4: LED_PWR -> GND
- LED111 pad 1: GND -> LED_PWR
- LED111 pad 4: LED_PWR -> GND
- LED20 pad 1: GND -> LED_PWR
- LED20 pad 4: LED_PWR -> GND
- LED21 pad 1: GND -> LED_PWR
- LED21 pad 4: LED_PWR -> GND
- LED22 pad 1: GND -> LED_PWR
- LED22 pad 4: LED_PWR -> GND
- LED23 pad 1: GND -> LED_PWR
- LED23 pad 4: LED_PWR -> GND
- LED24 pad 1: GND -> LED_PWR
- LED24 pad 4: LED_PWR -> GND
- LED25 pad 1: GND -> LED_PWR
- LED25 pad 4: LED_PWR -> GND
- LED26 pad 1: GND -> LED_PWR
- LED26 pad 4: LED_PWR -> GND
- LED27 pad 1: GND -> LED_PWR
- LED27 pad 4: LED_PWR -> GND
- LED28 pad 1: GND -> LED_PWR
- LED28 pad 4: LED_PWR -> GND
- LED29 pad 1: GND -> LED_PWR
- LED29 pad 4: LED_PWR -> GND
- LED30 pad 1: GND -> LED_PWR
- LED30 pad 4: LED_PWR -> GND
- LED31 pad 1: GND -> LED_PWR
- LED31 pad 4: LED_PWR -> GND
- LED32 pad 1: GND -> LED_PWR
- LED32 pad 4: LED_PWR -> GND
- LED33 pad 1: GND -> LED_PWR
- LED33 pad 4: LED_PWR -> GND
- LED34 pad 1: GND -> LED_PWR
- LED34 pad 4: LED_PWR -> GND
- LED35 pad 1: GND -> LED_PWR
- LED35 pad 4: LED_PWR -> GND
- LED36 pad 1: GND -> LED_PWR
- LED36 pad 4: LED_PWR -> GND
- LED37 pad 1: GND -> LED_PWR
- LED37 pad 4: LED_PWR -> GND
- LED38 pad 1: GND -> LED_PWR
- LED38 pad 4: LED_PWR -> GND
- LED39 pad 1: GND -> LED_PWR
- LED39 pad 4: LED_PWR -> GND
- LED40 pad 1: LED_PWR -> GND
- LED40 pad 4: GND -> LED_PWR
- LED41 pad 1: LED_PWR -> GND
- LED41 pad 4: GND -> LED_PWR
- LED42 pad 1: LED_PWR -> GND
- LED42 pad 4: GND -> LED_PWR
- LED43 pad 1: LED_PWR -> GND
- LED43 pad 4: GND -> LED_PWR
- LED44 pad 1: LED_PWR -> GND
- LED44 pad 4: GND -> LED_PWR
- LED45 pad 1: LED_PWR -> GND
- LED45 pad 4: GND -> LED_PWR
- LED46 pad 1: LED_PWR -> GND
- LED46 pad 4: GND -> LED_PWR
- LED47 pad 1: LED_PWR -> GND
- LED47 pad 4: GND -> LED_PWR
- LED48 pad 1: LED_PWR -> GND
- LED48 pad 4: GND -> LED_PWR
- LED49 pad 1: LED_PWR -> GND
- LED49 pad 4: GND -> LED_PWR
- LED50 pad 1: LED_PWR -> GND
- LED50 pad 4: GND -> LED_PWR
- LED51 pad 1: LED_PWR -> GND
- LED51 pad 4: GND -> LED_PWR
- LED52 pad 1: LED_PWR -> GND
- LED52 pad 4: GND -> LED_PWR
- LED53 pad 1: LED_PWR -> GND
- LED53 pad 4: GND -> LED_PWR
- LED54 pad 1: LED_PWR -> GND
- LED54 pad 4: GND -> LED_PWR
- LED55 pad 1: LED_PWR -> GND
- LED55 pad 4: GND -> LED_PWR
- LED56 pad 1: LED_PWR -> GND
- LED56 pad 4: GND -> LED_PWR
- LED57 pad 1: LED_PWR -> GND
- LED57 pad 4: GND -> LED_PWR
- LED58 pad 1: LED_PWR -> GND
- LED58 pad 4: GND -> LED_PWR
- LED59 pad 1: LED_PWR -> GND
- LED59 pad 4: GND -> LED_PWR
- LED78 pad 3: unconnected-(LED78-DIN-Pad3) -> Net-(LED59-DOUT)
- LED79 pad 1: unconnected-(LED79-VDD-Pad1) -> GND
- LED79 pad 2: unconnected-(LED79-DOUT-Pad2) -> Net-(LED79-DOUT)
- LED79 pad 3: Net-(LED59-DOUT) -> Net-(LED60-DOUT)
- LED79 pad 4: unconnected-(LED79-VSS-Pad4) -> LED_PWR
- LED80 pad 1: LED_PWR -> GND
- LED80 pad 3: Net-(LED60-DOUT) -> Net-(LED79-DOUT)
- LED80 pad 4: GND -> LED_PWR
- LED81 pad 1: LED_PWR -> GND
- LED81 pad 4: GND -> LED_PWR
- LED82 pad 1: LED_PWR -> GND
- LED82 pad 4: GND -> LED_PWR
- LED83 pad 1: LED_PWR -> GND
- LED83 pad 4: GND -> LED_PWR
- LED84 pad 1: LED_PWR -> GND
- LED84 pad 4: GND -> LED_PWR
- LED85 pad 1: LED_PWR -> GND
- LED85 pad 4: GND -> LED_PWR
- LED86 pad 1: LED_PWR -> GND
- LED86 pad 4: GND -> LED_PWR
- LED87 pad 1: LED_PWR -> GND
- LED87 pad 4: GND -> LED_PWR
- LED88 pad 1: LED_PWR -> GND
- LED88 pad 2: unconnected-(LED88-DOUT-Pad2) -> Net-(LED88-DOUT)
- LED88 pad 4: GND -> LED_PWR
- LED89 pad 1: LED_PWR -> GND
- LED89 pad 2: unconnected-(LED89-DOUT-Pad2) -> Net-(LED89-DOUT)
- LED89 pad 3: unconnected-(LED89-DIN-Pad3) -> Net-(LED88-DOUT)
- LED89 pad 4: GND -> LED_PWR
- LED90 pad 1: LED_PWR -> GND
- LED90 pad 2: unconnected-(LED90-DOUT-Pad2) -> Net-(LED90-DOUT)
- LED90 pad 3: unconnected-(LED90-DIN-Pad3) -> Net-(LED89-DOUT)
- LED90 pad 4: GND -> LED_PWR
- LED91 pad 1: LED_PWR -> GND
- LED91 pad 2: unconnected-(LED91-DOUT-Pad2) -> Net-(LED91-DOUT)
- LED91 pad 3: unconnected-(LED91-DIN-Pad3) -> Net-(LED90-DOUT)
- LED91 pad 4: GND -> LED_PWR
- LED92 pad 1: LED_PWR -> GND
- LED92 pad 3: unconnected-(LED92-DIN-Pad3) -> Net-(LED91-DOUT)
- LED92 pad 4: GND -> LED_PWR
- LED93 pad 1: LED_PWR -> GND
- LED93 pad 2: unconnected-(LED93-DOUT-Pad2) -> Net-(LED93-DOUT)
- LED93 pad 4: GND -> LED_PWR
- LED94 pad 1: LED_PWR -> GND
- LED94 pad 2: unconnected-(LED94-DOUT-Pad2) -> Net-(LED94-DOUT)
- LED94 pad 3: unconnected-(LED94-DIN-Pad3) -> Net-(LED93-DOUT)
- LED94 pad 4: GND -> LED_PWR
- LED95 pad 1: LED_PWR -> GND
- LED95 pad 2: unconnected-(LED95-DOUT-Pad2) -> Net-(LED95-DOUT)
- LED95 pad 3: unconnected-(LED95-DIN-Pad3) -> Net-(LED94-DOUT)
- LED95 pad 4: GND -> LED_PWR
- LED96 pad 1: LED_PWR -> GND
- LED96 pad 2: unconnected-(LED96-DOUT-Pad2) -> Net-(LED96-DOUT)
- LED96 pad 3: unconnected-(LED96-DIN-Pad3) -> Net-(LED95-DOUT)
- LED96 pad 4: GND -> LED_PWR
- LED97 pad 1: LED_PWR -> GND
- LED97 pad 2: unconnected-(LED97-DOUT-Pad2) -> Net-(LED111-DIN)
- LED97 pad 3: unconnected-(LED97-DIN-Pad3) -> Net-(LED96-DOUT)
- LED97 pad 4: GND -> LED_PWR
- LED98 pad 2: Net-(LED98-DOUT) -> unconnected-(LED98-DOUT-Pad2)
- LED98 pad 3: unconnected-(LED98-DIN-Pad3) -> Net-(LED98-DIN)
- LED99 pad 2: Net-(LED113-DIN) -> unconnected-(LED99-DOUT-Pad2)
- LED99 pad 3: Net-(LED98-DOUT) -> Net-(LED98-DIN)
- MX100 pad 1: COL0 -> COL2
- MX101 pad 1: COL1 -> COL2
- MX101 pad 2: Net-(D101-K) -> Net-(D101-A)
- MX102 pad 1: COL2 -> COL3
- MX103 pad 1: COL2 -> COL3
- MX104 pad 1: COL3 -> COL4
- MX105 pad 1: COL3 -> COL5
- MX105 pad 2: Net-(D105-A) -> Net-(D105-K)
- MX106 pad 1: COL4 -> COL6
- MX107 pad 1: COL5 -> COL7
- MX108 pad 1: COL6 -> COL8
- MX109 pad 1: COL7 -> COL8
- MX109 pad 2: Net-(D109-K) -> Net-(D109-A)
- MX110 pad 1: COL8 -> COL9
- MX111 pad 1: COL8 -> COL9
- MX65 pad 1: COL2 -> COL3
- MX65 pad 2: Net-(D65-A) -> Net-(D65-K)
- MX66 pad 2: Net-(D66-K) -> Net-(D66-A)
- MX67 pad 1: COL3 -> COL4
- MX67 pad 2: Net-(D67-A) -> Net-(D67-K)
- MX68 pad 2: Net-(D68-K) -> Net-(D68-A)
- MX69 pad 1: COL4 -> COL5
- MX69 pad 2: Net-(D69-A) -> Net-(D69-K)
- MX70 pad 2: Net-(D70-K) -> Net-(D70-A)
- MX71 pad 1: COL5 -> COL6
- MX71 pad 2: Net-(D71-A) -> Net-(D71-K)
- MX72 pad 2: Net-(D72-K) -> Net-(D72-A)
- MX73 pad 1: COL6 -> COL7
- MX73 pad 2: Net-(D73-A) -> Net-(D73-K)
- MX74 pad 2: Net-(D74-K) -> Net-(D74-A)
- MX75 pad 1: COL7 -> COL8
- MX75 pad 2: Net-(D75-A) -> Net-(D75-K)
- MX76 pad 2: Net-(D76-K) -> Net-(D76-A)
- MX77 pad 1: COL8 -> COL9
- MX77 pad 2: Net-(D77-A) -> Net-(D77-K)
- MX78 pad 2: Net-(D78-K) -> Net-(D78-A)
- MX79 pad 1: COL9 -> COL0
- MX79 pad 2: Net-(D79-A) -> Net-(D79-K)
- MX80 pad 2: Net-(D80-K) -> Net-(D80-A)
- MX81 pad 1: COL0 -> COL1
- MX81 pad 2: Net-(D81-A) -> Net-(D81-K)
- MX82 pad 2: Net-(D82-K) -> Net-(D82-A)
- MX83 pad 1: COL1 -> COL2
- MX83 pad 2: Net-(D83-A) -> Net-(D83-K)
- MX84 pad 1: COL2 -> COL3
- MX85 pad 1: COL2 -> COL3
- MX86 pad 1: COL3 -> COL4
- MX87 pad 1: COL3 -> COL4
- MX88 pad 1: COL4 -> COL5
- MX89 pad 1: COL4 -> COL5
- MX90 pad 1: COL5 -> COL6
- MX91 pad 1: COL5 -> COL6
- MX92 pad 1: COL6 -> COL7
- MX93 pad 1: COL6 -> COL7
- MX94 pad 1: COL7 -> COL8
- MX95 pad 1: COL7 -> COL8
- MX96 pad 1: COL8 -> COL9
- MX97 pad 1: COL8 -> COL9
- MX98 pad 1: COL9 -> COL0
- MX99 pad 1: COL9 -> COL1
- MX99 pad 2: Net-(D99-A) -> Net-(D99-K)
- SW1 pad S2: ROT1_D -> Net-(D112-K)
- SW2 pad S2: ROT2_D -> Net-(D113-A)
- U6 pad 31: ENC2_A -> ENC1_A
- U6 pad 32: ENC2_B -> ENC1_B
- U6 pad 34: unconnected-(U6-GPIO22-Pad34) -> ENC4_A
- U6 pad 35: LCD_EN -> ENC2_A
- U6 pad 38: ENC1_A -> ENC2_B
- U6 pad 39: ENC1_B -> ENC3_A
Routing:
- net COL2: track 262.7 -> 0.00 mm
- net COL3: track 251.8 -> 0.00 mm
- net COL8: track 242.5 -> 0.00 mm
- net COL5: track 211.7 -> 0.00 mm
- net COL4: track 211.7 -> 0.00 mm
- net COL6: track 209.8 -> 0.00 mm
- net COL7: track 208.9 -> 0.00 mm
- net COL0: track 201.0 -> 0.00 mm
- net COL1: track 181.1 -> 0.00 mm
- net COL9: track 143.1 -> 0.00 mm
- net ENC1_A: track 0.00 -> 2.40 mm
- net ROT1_A: track 0.00 -> 2.38 mm
