File: SP110duo/new/SP110Duo.kicad_sch (KiCad schematic)
At the start: 420 parts, among them J1 USB_C_Receptacle_USB2.0, Q7 AO3401A, Q8 MMUN2233LT1G, SW1 RotaryEncoder_Switch, SW2 RotaryEncoder_Switch, U1 AZ1117H-3.3TRE1, U2 TPS2553DBVR, U3 74AHC1G125, U4 W25Q128JVSIQ, U5 PRTR5V0U2X, U6 RP2040, Y1 X322512MSB4SI

Commit message: update for rjk
Parts:
- LED20, LED21, LED22, LED23, LED24, LED25, LED26, LED27, LED28, LED29, LED30, LED31, LED32, LED33, LED34, LED35, LED36, LED37, LED38: footprint Keyboard:LED_MX_6028R -> Keyboard:LED_MX_6028R-ROT
- MX103: footprint Keyboard:SW_MX_HS_1.25u -> Keyboard:SW_MX_HS_2.75u
- MX104: footprint Keyboard:SW_MX_HS_1u -> Keyboard:SW_MX_HS_1.25u
- MX105, MX77: footprint Keyboard:SW_MX_HS_1u -> Keyboard:SW_MX_HS_2.25u
- MX106, MX107: footprint Keyboard:SW_MX_HS_1u -> Keyboard:SW_MX_HS_1.5u
- MX40: footprint Keyboard:SW_MX_HS_2.25u -> Keyboard:SW_MX_HS_2u
- MX47: renamed from MX46; footprint Keyboard:SW_MX_HS_1u -> Keyboard:SW_MX_HS_1.5u
- MX48: renamed from MX47; footprint Keyboard:SW_MX_HS_1u -> Keyboard:SW_MX_HS_1.5u
- MX61: renamed from MX60; footprint Keyboard:SW_MX_HS_1u -> Keyboard:SW_MX_HS_1.5u
- MX65: footprint Keyboard:SW_MX_HS_1u -> Keyboard:SW_MX_HS_1.75u
- MX96: renamed from MX95; footprint Keyboard:SW_MX_HS_1u -> Keyboard:SW_MX_HS_1.75u
- renumbered D113 to D111, D114 to D112, D116 to D113, D117 to D114, D111 to D115, D115 to D116, D112 to D117, D64 to D46, D46 to D47, D47 to D48, D48 to D49, D49 to D50, D50 to D51, D51 to D52, D52 to D53, D53 to D54, D54 to D55, D55 to D56, D56 to D57, D57 to D58, D58 to D59, D59 to D60, D60 to D61, D61 to D62, D62 to D63, D63 to D64, D99 to D83, D83 to D84, D84 to D85, D85 to D86, D86 to D87, D87 to D88, D88 to D89, D89 to D90, D90 to D91, D91 to D92, D92 to D93, D93 to D94, D94 to D95, D95 to D96, D96 to D97, D97 to D98, D98 to D99, MX64 to MX46, MX48 to MX49, MX49 to MX50, MX50 to MX51, MX51 to MX52, MX52 to MX53, MX53 to MX54, MX54 to MX55, MX55 to MX56, MX56 to MX57, MX57 to MX58, MX58 to MX59, MX59 to MX60, MX61 to MX62, MX62 to MX63, MX63 to MX64, MX99 to MX83, MX83 to MX84, MX84 to MX85, MX85 to MX86, MX86 to MX87, MX87 to MX88, MX88 to MX89, MX89 to MX90, MX90 to MX91, MX91 to MX92, MX92 to MX93, MX93 to MX94, MX94 to MX95, MX96 to MX97, MX97 to MX98, MX98 to MX99
Connections:
- net COL0: no longer MX62.2, MX98.2
- net COL1: now also MX62.2, MX98.2; no longer MX64.2, MX83.2
- net COL2: now also MX64.2, MX83.2; no longer S1.7 (COM)
- net COL3: now also MX66.2, MX85.2
- net COL4: now also MX68.2, MX87.2; no longer MX66.2, MX85.2
- net COL5: now also MX70.2, MX89.2; no longer MX68.2, MX87.2
- net COL6: now also MX105.2, MX72.2, MX91.2; no longer MX70.2, MX89.2
- net COL7: now also MX107.2, MX74.2, MX93.2; no longer MX105.2, MX72.2, MX91.2
- net COL8: now also MX109.2, MX76.2, MX95.2; no longer MX107.2, MX74.2, MX93.2
- net COL9: no longer MX109.2, MX76.2, MX95.2
- net RKJ-A: now also D114.1 (K); no longer D114.2 (A)
- net RKJ-B: now also D116.1 (K); no longer D116.2 (A)
- net RKJ-C: now also D117.1 (K); no longer D117.2 (A)
- net RKJ-PUSH: now also D113.2 (A); no longer D113.1 (K)
- net ROT2_D: now also D112.1 (K); no longer D112.2 (A)
- net ROW0: now also D10.1 (K), D12.1 (K), D14.1 (K), D16.1 (K), D18.1 (K), D20.1 (K); no longer D10.2 (A), D12.2 (A), D14.2 (A), D16.2 (A), D18.2 (A), D20.2 (A)
- net ROW1: now also D30.1 (K), D32.1 (K), D34.1 (K), D36.1 (K), D38.1 (K), D40.1 (K); no longer D30.2 (A), D32.2 (A), D34.2 (A), D36.2 (A), D38.2 (A), D40.2 (A)
- net ROW2: now also D46.2 (A), D50.1 (K), D52.1 (K), D54.1 (K), D56.1 (K), D58.1 (K), D60.1 (K); no longer D115.1 (K), D50.2 (A), D52.2 (A), D54.2 (A), D56.2 (A), D58.2 (A), D60.2 (A)
- net ROW3: now also D67.1 (K), D69.1 (K), D71.1 (K), D73.1 (K), D75.1 (K), D77.1 (K); no longer D111.1 (K), D112.1 (K), D117.1 (K), D46.2 (A), D67.2 (A), D69.2 (A), D71.2 (A), D73.2 (A), D75.2 (A), D77.2 (A)
- net ROW4: now also D83.1 (K), D86.1 (K), D88.1 (K), D90.1 (K), D92.1 (K), D94.1 (K), D96.1 (K); no longer D116.1 (K), D86.2 (A), D88.2 (A), D90.2 (A), D92.2 (A), D94.2 (A), D96.2 (A)
- net at MX52.1: now also D52.2 (A); no longer D52.1 (K)
- net at MX50.1: now also D50.2 (A); no longer D50.1 (K)
- net at MX96.1: now also D96.2 (A); no longer D96.1 (K)
- net at MX77.1: now also D77.2 (A); no longer D77.1 (K)
- net at MX58.1: now also D58.2 (A); no longer D58.1 (K)
- net at MX67.1: now also D67.2 (A); no longer D67.1 (K)
- net at MX106.1: now also D106.2 (A); no longer D106.1 (K)
- net at MX16.1: now also D16.2 (A); no longer D16.1 (K)
- net at MX69.1: now also D69.2 (A); no longer D69.1 (K)
- net at MX54.1: now also D54.2 (A); no longer D54.1 (K)
- net at MX90.1: now also D90.2 (A); no longer D90.1 (K)
- net at MX103.1: now also D103.2 (A); no longer D103.1 (K)
- net at MX32.1: now also D32.2 (A); no longer D32.1 (K)
- net at MX98.1: now also D98.1 (K); no longer D98.2 (A)
- net at MX34.1: now also D34.2 (A); no longer D34.1 (K)
- net at MX60.1: now also D60.2 (A); no longer D60.1 (K)
- net at MX40.1: now also D40.2 (A); no longer D40.1 (K)
- net at MX108.1: now also D108.2 (A); no longer D108.1 (K)
- net at MX38.1: now also D38.2 (A); no longer D38.1 (K)
- net at MX56.1: now also D56.2 (A); no longer D56.1 (K)
- net at MX86.1: now also D86.2 (A); no longer D86.1 (K)
- net at MX10.1: now also D10.2 (A); no longer D10.1 (K)
- net at MX71.1: now also D71.2 (A); no longer D71.1 (K)
- net at MX94.1: now also D94.2 (A); no longer D94.1 (K)
- net at MX18.1: now also D18.2 (A); no longer D18.1 (K)
- net at MX30.1: now also D30.2 (A); no longer D30.1 (K)
- net at MX36.1: now also D36.2 (A); no longer D36.1 (K)
- net at MX75.1: now also D75.2 (A); no longer D75.1 (K)
- net at MX102.1: now also D102.2 (A); no longer D102.1 (K)
- net at MX104.1: now also D104.2 (A); no longer D104.1 (K)
- net at MX20.1: now also D20.2 (A); no longer D20.1 (K)
- net at MX88.1: now also D88.2 (A); no longer D88.1 (K)
- net at MX73.1: now also D73.2 (A); no longer D73.1 (K)
- net at MX92.1: now also D92.2 (A); no longer D92.1 (K)
- net at MX12.1: now also D12.2 (A); no longer D12.1 (K)
- net at MX14.1: now also D14.2 (A); no longer D14.1 (K)
- net at MX110.1: now also D110.2 (A); no longer D110.1 (K)
- net at MX99.1: now also D99.2 (A); no longer D99.1 (K)
- removed net ROW5: D100.2 (A), D101.1 (K), D102.2 (A), D103.2 (A), D104.2 (A), D105.2 (A), D106.2 (A), D107.2 (A), D108.2 (A), D109.2 (A), D110.2 (A), D113.2 (A), D114.1 (K), D83.1 (K), D97.2 (A), D98.1 (K), D99.2 (A), U6.16 (GPIO13)
- new net COM: D100.2 (A), D101.1 (K), D102.1 (K), D103.1 (K), D104.1 (K), D105.2 (A), D106.1 (K), D107.2 (A), D108.1 (K), D109.2 (A), D110.1 (K), D113.1 (K), D97.2 (A), D98.2 (A), D99.1 (K), S1.7 (COM), U6.16 (GPIO13)
Other:
- moved on the sheet: D10, D102, D103, D104, D105, D106, D107, D108, D110, D111, D112, D113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

Commit message: update new design
Parts:
- removed D114, D115, D117: D, Keyboard:D_SOD-123F, symbol Device:D
- removed LED1, LED109, LED110, LED95: MX_SK6803MINI-E, Keyboard:LED_MX_6028R, symbol Keyboard:MX_SK6803MINI-E
- added D111, D112: D, Keyboard:D_SOD-123F, symbol Device:D
- added LED19, LED86, LED99: MX_SK6803MINI-E, Keyboard:LED_MX_6028R, symbol Keyboard:MX_SK6803MINI-E
- added LED39, LED61, LED66, LED79: MX_SK6803MINI-E, Keyboard:LED_MX_6028R-ROT, symbol Keyboard:MX_SK6803MINI-E
- added MX111, MX112, MX113: MX_SW_HS, Keyboard:SW_MX_HS_1u, symbol PCM_marbastlib-mx:MX_SW_HS_CPG151101S11
- LED100: renamed from LED94; footprint Keyboard:LED_MX_6028R -> Keyboard:LED_MX_6028R-ROT
- LED101: renamed from LED96; footprint Keyboard:LED_MX_6028R -> Keyboard:LED_MX_6028R-ROT
- LED102: renamed from LED97; footprint Keyboard:LED_MX_6028R -> Keyboard:LED_MX_6028R-ROT
- LED103: renamed from LED98; footprint Keyboard:LED_MX_6028R -> Keyboard:LED_MX_6028R-ROT
- LED104: renamed from LED99; footprint Keyboard:LED_MX_6028R -> Keyboard:LED_MX_6028R-ROT
- LED105: renamed from LED100; footprint Keyboard:LED_MX_6028R -> Keyboard:LED_MX_6028R-ROT
- LED106: renamed from LED101; footprint Keyboard:LED_MX_6028R -> Keyboard:LED_MX_6028R-ROT
- LED107: renamed from LED102; footprint Keyboard:LED_MX_6028R -> Keyboard:LED_MX_6028R-ROT
- LED108: renamed from LED103; footprint Keyboard:LED_MX_6028R -> Keyboard:LED_MX_6028R-ROT
- LED109: renamed from LED104; footprint Keyboard:LED_MX_6028R -> Keyboard:LED_MX_6028R-ROT
- LED110: renamed from LED105; footprint Keyboard:LED_MX_6028R -> Keyboard:LED_MX_6028R-ROT
- LED111: renamed from LED106; footprint Keyboard:LED_MX_6028R -> Keyboard:LED_MX_6028R-ROT
- LED112: renamed from LED107; footprint Keyboard:LED_MX_6028R -> Keyboard:LED_MX_6028R-ROT
- LED113: renamed from LED108; footprint Keyboard:LED_MX_6028R -> Keyboard:LED_MX_6028R-ROT
- LED60: renamed from LED58; footprint Keyboard:LED_MX_6028R -> Keyboard:LED_MX_6028R-ROT
- LED62: renamed from LED60; footprint Keyboard:LED_MX_6028R -> Keyboard:LED_MX_6028R-ROT
- LED63: renamed from LED61; footprint Keyboard:LED_MX_6028R -> Keyboard:LED_MX_6028R-ROT
- LED64: renamed from LED62; footprint Keyboard:LED_MX_6028R -> Keyboard:LED_MX_6028R-ROT
- LED65: renamed from LED63; footprint Keyboard:LED_MX_6028R -> Keyboard:LED_MX_6028R-ROT
- LED67: renamed from LED64; footprint Keyboard:LED_MX_6028R -> Keyboard:LED_MX_6028R-ROT
- LED68: renamed from LED65; footprint Keyboard:LED_MX_6028R -> Keyboard:LED_MX_6028R-ROT
- LED69: renamed from LED66; footprint Keyboard:LED_MX_6028R -> Keyboard:LED_MX_6028R-ROT
- LED70: renamed from LED67; footprint Keyboard:LED_MX_6028R -> Keyboard:LED_MX_6028R-ROT
- LED71: renamed from LED68; footprint Keyboard:LED_MX_6028R -> Keyboard:LED_MX_6028R-ROT
- LED72: renamed from LED69; footprint Keyboard:LED_MX_6028R -> Keyboard:LED_MX_6028R-ROT
- LED73: renamed from LED70; footprint Keyboard:LED_MX_6028R -> Keyboard:LED_MX_6028R-ROT
- LED74: renamed from LED71; footprint Keyboard:LED_MX_6028R -> Keyboard:LED_MX_6028R-ROT
- LED75: renamed from LED72; footprint Keyboard:LED_MX_6028R -> Keyboard:LED_MX_6028R-ROT
- LED76: renamed from LED73; footprint Keyboard:LED_MX_6028R -> Keyboard:LED_MX_6028R-ROT
- LED77: renamed from LED74; footprint Keyboard:LED_MX_6028R -> Keyboard:LED_MX_6028R-ROT
- LED78: renamed from LED75; footprint Keyboard:LED_MX_6028R -> Keyboard:LED_MX_6028R-ROT
- MX100, MX101, MX102, MX104: footprint Keyboard:SW_MX_HS_1.25u -> Keyboard:SW_MX_HS_1u
- MX103: footprint Keyboard:SW_MX_HS_2.75u -> Keyboard:SW_MX_HS_1u
- MX105, MX77, MX85: footprint Keyboard:SW_MX_HS_2.25u -> Keyboard:SW_MX_HS_1u
- MX106, MX107, MX47, MX48, MX61: footprint Keyboard:SW_MX_HS_1.5u -> Keyboard:SW_MX_HS_1u
- MX40: footprint Keyboard:SW_MX_HS_2u -> Keyboard:SW_MX_HS_1u
- MX65, MX96: footprint Keyboard:SW_MX_HS_1.75u -> Keyboard:SW_MX_HS_1u
- renumbered D111 to D113, D112 to D114, D113 to D115, LED2 to LED1, LED11 to LED10, LED12 to LED11, LED13 to LED12, LED14 to LED13, LED15 to LED14, LED16 to LED15, LED17 to LED16, LED18 to LED17, LED19 to LED18, LED3 to LED2, LED4 to LED3, LED5 to LED4, LED39 to LED40, LED40 to LED41, LED41 to LED42, LED42 to LED43, LED43 to LED44, LED44 to LED45, LED45 to LED46, LED46 to LED47, LED47 to LED48, LED48 to LED49, LED6 to LED5, LED49 to LED50, LED50 to LED51, LED51 to LED52, LED52 to LED53, LED53 to LED54, LED54 to LED55, LED55 to LED56, LED56 to LED57, LED57 to LED58, LED7 to LED6, LED8 to LED7, LED9 to LED8, LED76 to LED80, LED77 to LED81, LED78 to LED82, LED79 to LED83, LED80 to LED84, LED81 to LED85, LED82 to LED87, LED83 to LED88, LED84 to LED89, LED10 to LED9, LED85 to LED90, LED86 to LED91, LED87 to LED92, LED88 to LED93, LED89 to LED94, LED90 to LED95, LED91 to LED96, LED92 to LED97, LED93 to LED98
Connections:
- net RKJ-A is gone; now on net COL5: S1.1 (A)
- net RKJ-C is gone; now on net COL0: S1.6 (C)
- net RKJ-D is gone; now on net COL4: S1.9 (D_1)
- net COL0: now also MX1.1, MX100.1, MX20.1, MX21.1, MX40.1, MX41.1, MX60.1, MX61.1, MX80.1, MX81.1, SW1.S1; no longer MX1.2, MX2.2, MX21.2, MX22.2, MX41.2, MX42.2, MX61.2, MX78.2, MX79.2, MX97.2
- net COL1: now also MX101.1, MX2.1, MX22.1, MX23.1, MX3.1, MX42.1, MX43.1, MX62.1, MX63.1, MX82.1, MX83.1, S1.4 (B); no longer MX23.2, MX24.2, MX3.2, MX4.2, MX43.2, MX44.2, MX62.2, MX63.2, MX80.2, MX81.2, MX98.2, MX99.2
- net COL2: now also MX102.1, MX103.1, MX24.1, MX25.1, MX4.1, MX44.1, MX45.1, MX5.1, MX64.1, MX65.1, MX84.1, MX85.1; no longer MX25.2, MX26.2, MX45.2, MX46.2, MX5.2, MX6.2, MX64.2, MX82.2, MX83.2
- net COL3: now also MX104.1, MX105.1, MX26.1, MX27.1, MX46.1, MX47.1, MX6.1, MX66.1, MX67.1, MX7.1, MX86.1, MX87.1; no longer MX100.2, MX101.2, MX27.2, MX28.2, MX47.2, MX48.2, MX65.2, MX66.2, MX7.2, MX8.2, MX84.2, MX85.2, SW1.S1, SW2.S1
- net COL4: now also MX106.1, MX28.1, MX29.1, MX48.1, MX49.1, MX68.1, MX69.1, MX8.1, MX88.1, MX89.1, MX9.1; no longer MX10.2, MX102.2, MX29.2, MX30.2, MX49.2, MX50.2, MX67.2, MX68.2, MX86.2, MX87.2, MX9.2
- net COL5: now also MX10.1, MX107.1, MX11.1, MX30.1, MX31.1, MX50.1, MX51.1, MX70.1, MX71.1, MX90.1, MX91.1; no longer MX103.2, MX11.2, MX12.2, MX31.2, MX32.2, MX51.2, MX52.2, MX69.2, MX70.2, MX88.2, MX89.2
- net COL6: now also MX108.1, MX12.1, MX13.1, MX32.1, MX33.1, MX52.1, MX53.1, MX72.1, MX73.1, MX92.1, MX93.1, S1.2 (PUSH); no longer MX104.2, MX105.2, MX13.2, MX14.2, MX33.2, MX34.2, MX53.2, MX54.2, MX71.2, MX72.2, MX90.2, MX91.2
- net COL7: now also MX109.1, MX14.1, MX15.1, MX34.1, MX35.1, MX54.1, MX55.1, MX74.1, MX75.1, MX94.1, MX95.1; no longer MX106.2, MX107.2, MX15.2, MX16.2, MX35.2, MX36.2, MX55.2, MX56.2, MX73.2, MX74.2, MX92.2, MX93.2
- net COL8: now also MX110.1, MX16.1, MX17.1, MX36.1, MX37.1, MX56.1, MX57.1, MX76.1, MX77.1, MX96.1, MX97.1, MX111.1; no longer MX108.2, MX109.2, MX17.2, MX18.2, MX37.2, MX38.2, MX57.2, MX58.2, MX75.2, MX76.2, MX94.2, MX95.2
- net COL9: now also MX18.1, MX19.1, MX38.1, MX39.1, MX58.1, MX59.1, MX78.1, MX79.1, MX98.1, MX99.1, MX112.1, MX113.1; no longer MX110.2, MX19.2, MX20.2, MX39.2, MX40.2, MX59.2, MX60.2, MX77.2, MX96.2
- net COM: now also D115.2 (A); no longer D100.2 (A), D101.1 (K), D102.1 (K), D103.1 (K), D104.1 (K), D105.2 (A), D106.1 (K), D107.2 (A), D108.1 (K), D109.2 (A), D110.1 (K), D115.1 (K), D97.2 (A), D98.2 (A), D99.1 (K), U6.16 (GPIO13)
- net GND: now also LED59.4 (VSS), LED19.4 (VSS), LED39.1 (VDD), LED61.1 (VDD), LED66.1 (VDD), LED86.4 (VSS), LED99.4 (VSS); no longer LED59.1 (VDD)
- net LED_DAT_5V: now also LED1.3 (DIN)
- net LED_PWR: now also LED59.1 (VDD), LED19.1 (VDD), LED39.4 (VSS), LED61.4 (VSS), LED66.4 (VSS), LED86.1 (VDD), LED99.1 (VDD); no longer LED59.4 (VSS)
- net ROT1_D: now also D113.1 (K); no longer D113.2 (A)
- net ROT2_D: now also D114.2 (A); no longer D114.1 (K)
- net ROW0: now also D1.1 (K), D10.2 (A), D11.1 (K), D113.2 (A), D12.2 (A), D13.1 (K), D14.2 (A), D15.1 (K), D16.2 (A), D17.1 (K), D18.2 (A), D19.1 (K), D2.2 (A), D3.1 (K), D4.2 (A), D5.1 (K), D6.2 (A), D7.1 (K), D8.2 (A), D9.1 (K); no longer D1.2 (A), D10.1 (K), D11.2 (A), D12.1 (K), D13.2 (A), D14.1 (K), D15.2 (A), D16.1 (K), D17.2 (A), D18.1 (K), D19.2 (A), D2.1 (K), D20.1 (K), D3.2 (A), D4.1 (K), D5.2 (A), D6.1 (K), D7.2 (A), D8.1 (K), D9.2 (A)
- net ROW1: now also D20.2 (A), D21.1 (K), D22.2 (A), D24.2 (A), D25.1 (K), D26.2 (A), D27.1 (K), D28.2 (A), D29.1 (K), D30.2 (A), D31.1 (K), D32.2 (A), D33.1 (K), D34.2 (A), D35.1 (K), D36.2 (A), D37.1 (K), D38.2 (A), D39.1 (K); no longer D21.2 (A), D22.1 (K), D24.1 (K), D25.2 (A), D26.1 (K), D27.2 (A), D28.1 (K), D29.2 (A), D30.1 (K), D31.2 (A), D32.1 (K), D33.2 (A), D34.1 (K), D35.2 (A), D36.1 (K), D37.2 (A), D38.1 (K), D39.2 (A), D40.1 (K)
- net ROW2: now also D40.2 (A), D41.1 (K), D42.2 (A), D43.1 (K), D44.2 (A), D45.1 (K), D47.1 (K), D48.2 (A), D49.1 (K), D50.2 (A), D51.1 (K), D52.2 (A), D53.1 (K), D54.2 (A), D55.1 (K), D56.2 (A), D57.1 (K), D58.2 (A), D59.1 (K); no longer D41.2 (A), D42.1 (K), D43.2 (A), D44.1 (K), D45.2 (A), D47.2 (A), D48.1 (K), D49.2 (A), D50.1 (K), D51.2 (A), D52.1 (K), D53.2 (A), D54.1 (K), D55.2 (A), D56.1 (K), D57.2 (A), D58.1 (K), D59.2 (A), D60.1 (K)
- net ROW3: now also D114.1 (K), D60.2 (A), D61.1 (K), D62.2 (A), D63.1 (K), D64.2 (A), D65.1 (K), D66.2 (A), D78.2 (A), D79.1 (K); no longer D61.2 (A), D62.1 (K), D63.2 (A), D64.1 (K), D65.2 (A), D66.1 (K)
- net ROW4: now also D85.1 (K), D86.2 (A), D87.1 (K), D88.2 (A), D89.1 (K), D90.2 (A), D91.1 (K), D92.2 (A), D93.1 (K), D94.2 (A), D95.1 (K), D96.2 (A), D97.1 (K), D98.2 (A), D99.1 (K); no longer D78.2 (A), D79.1 (K), D85.2 (A), D86.1 (K), D87.2 (A), D88.1 (K), D89.2 (A), D90.1 (K), D91.2 (A), D92.1 (K), D93.2 (A), D94.1 (K), D95.2 (A), D96.1 (K)
- net at LED98.2 (DOUT): now also LED99.3 (DIN)
- net at LED58.2 (DOUT): no longer LED78.3 (DIN)
- net at D77.2 (A): now also MX77.2; no longer MX77.1
- net at LED65.3 (DIN): now also LED66.2 (DOUT); no longer LED67.2 (DOUT)
- net at D81.2 (A): now also MX81.2; no longer MX81.1
- net at D67.2 (A): now also MX67.2; no longer MX67.1
- net at D80.1 (K): now also MX80.2; no longer MX80.1
- net ROW5: now reaches D106.2 (A)
- net ROW5: now also D100.2 (A), D101.2 (A), D102.2 (A), D103.1 (K), D104.2 (A), D105.1 (K), D107.2 (A), D108.2 (A), D109.2 (A), D110.2 (A), D115.1 (K), D116.1 (K), U6.16 (GPIO13), D111.1 (K), D112.2 (A); no longer MX106.1
- net at D69.2 (A): now also MX69.2; no longer MX69.1
- net at LED6.2 (DOUT): now also LED7.3 (DIN)
- net at D103.2 (A): now also MX103.2; no longer MX103.1
- net at D116.2 (A): now also MX113.2
- net at D98.1 (K): now also MX98.2; no longer MX98.1
- net at LED8.2 (DOUT): now also LED9.3 (DIN)
- net at LED8.3 (DIN): now also LED7.2 (DOUT)
- net at LED100.3 (DIN): now also LED101.2 (DOUT)
- net at D46.1 (K): now also MX46.2; no longer MX46.1
- net at LED87.3 (DIN): now also LED86.2 (DOUT); no longer LED85.2 (DOUT)
- net at D79.2 (A): now also MX79.2; no longer MX79.1
- net at LED11.2 (DOUT): now also LED12.3 (DIN)
- net at LED11.3 (DIN): now also LED10.2 (DOUT)
- net at D83.2 (A): now also MX83.2; no longer MX83.1
- net at LED18.2 (DOUT): now also LED19.3 (DIN); no longer LED38.3 (DIN)
- net at LED18.3 (DIN): now also LED17.2 (DOUT)
- net at LED113.3 (DIN): now also LED99.2 (DOUT)
- net at LED15.2 (DOUT): now also LED16.3 (DIN)
- net at LED15.3 (DIN): now also LED14.2 (DOUT)
- net at D76.1 (K): now also MX76.2; no longer MX76.1
- net at D84.1 (K): now also MX84.2; no longer MX84.1
- net at LED9.2 (DOUT): now also LED10.3 (DIN)
- net at D109.1 (K): now also MX109.2; no longer MX109.1
- net at LED59.2 (DOUT): now also LED79.3 (DIN); no longer LED60.3 (DIN)
- net at LED62.2 (DOUT): now also LED61.3 (DIN); no longer LED59.3 (DIN)
- net at D78.1 (K): now also MX78.2; no longer MX78.1
- net at D82.1 (K): now also MX82.2; no longer MX82.1
- net at D74.1 (K): now also MX74.2; no longer MX74.1
- net at D71.2 (A): now also MX71.2; no longer MX71.1
- net at D23.1 (K): now also MX23.2; no longer MX23.1
- net at LED17.3 (DIN): now also LED16.2 (DOUT)
- net at D107.1 (K): now also MX107.2; no longer MX107.1
- net at D70.1 (K): now also MX70.2; no longer MX70.1
- net at LED12.2 (DOUT): now also LED13.3 (DIN)
- net at D75.2 (A): now also MX75.2; no longer MX75.1
- net at D72.1 (K): now also MX72.2; no longer MX72.1
- net at D73.2 (A): now also MX73.2; no longer MX73.1
- net at D68.1 (K): now also MX68.2; no longer MX68.1
- net at D99.2 (A): now also MX99.2; no longer MX99.1
- net at LED13.2 (DOUT): now also LED14.3 (DIN)
- net at D100.1 (K): now also MX100.2; no longer MX100.1
- removed net RKJ-B: D116.1 (K), S1.4 (B)
- removed net RKJ-PUSH: D115.2 (A), S1.2 (PUSH)
- new net: D101.1 (K), MX101.2
- new net: D6.1 (K), MX6.2
- new net: D54.1 (K), MX54.2
- new net: D38.1 (K), MX38.2
- new net: D24.1 (K), MX24.2
- new net: D32.1 (K), MX32.2
- new net: D53.2 (A), MX53.2
- new net: D102.1 (K), MX102.2
- new net: D59.2 (A), MX59.2
- new net: D16.1 (K), MX16.2
- new net: D14.1 (K), MX14.2
- new net: D112.1 (K), MX112.2
- new net: D85.2 (A), MX85.2
- new net: D104.1 (K), MX104.2
- new net: D106.1 (K), MX106.2
- new net: D62.1 (K), MX62.2
- new net: D47.2 (A), MX47.2
- new net: D111.2 (A), MX111.2
- new net: D64.1 (K), MX64.2
- new net: D33.2 (A), MX33.2
- new net: D35.2 (A), MX35.2
- new net: D12.1 (K), MX12.2
- new net: D18.1 (K), MX18.2
- new net: D66.1 (K), MX66.2
- new net: D55.2 (A), MX55.2
- new net: D17.2 (A), MX17.2
- new net: LED19.2 (DOUT), LED39.3 (DIN)
- new net: D8.1 (K), MX8.2
- new net: LED38.3 (DIN), LED39.2 (DOUT)
- new net: D26.1 (K), MX26.2
- new net: D58.1 (K), MX58.2
- new net: D11.2 (A), MX11.2
- new net: LED66.3 (DIN), LED67.2 (DOUT)
- new net: D93.2 (A), MX93.2
- new net: D15.2 (A), MX15.2
- new net: D86.1 (K), MX86.2
- new net: D9.2 (A), MX9.2
- new net: D27.2 (A), MX27.2
- new net: D29.2 (A), MX29.2
- new net: D43.2 (A), MX43.2
- new net: D56.1 (K), MX56.2
- new net: D65.2 (A), MX65.2
- new net: D19.2 (A), MX19.2
- new net: D51.2 (A), MX51.2
- new net: D41.2 (A), MX41.2
- new net: D96.1 (K), MX96.2
- new net: D97.2 (A), MX97.2
- new net: D60.1 (K), MX60.2
- new net: D21.2 (A), MX21.2
- new net: D48.1 (K), MX48.2
- new net: D22.1 (K), MX22.2
- new net: D108.1 (K), MX108.2
- new net: D5.2 (A), MX5.2
- new net: D40.1 (K), MX40.2
- new net: D94.1 (K), MX94.2
- new net: D28.1 (K), MX28.2
- new net: D10.1 (K), MX10.2
- new net: D30.1 (K), MX30.2
- new net: LED85.2 (DOUT), LED86.3 (DIN)
- new net: D52.1 (K), MX52.2
- new net: D87.2 (A), MX87.2
- new net: D105.2 (A), MX105.2
- new net: D45.2 (A), MX45.2
- new net: D61.2 (A), MX61.2
- new net: D25.2 (A), MX25.2
- new net: D110.1 (K), MX110.2
- new net: D63.2 (A), MX63.2
- new net: D49.2 (A), MX49.2
- new net: D37.2 (A), MX37.2
- new net: D91.2 (A), MX91.2
- new net: D88.1 (K), MX88.2
- new net: D39.2 (A), MX39.2
- new net: D20.1 (K), MX20.2
- new net: D34.1 (K), MX34.2
- new net: D92.1 (K), MX92.2
- new net: D7.2 (A), MX7.2
- new net: D31.2 (A), MX31.2
- new net: D13.2 (A), MX13.2
- new net: D1.2 (A), MX1.2
- new net: D36.1 (K), MX36.2
- new net: D44.1 (K), MX44.2
- new net: D50.1 (K), MX50.2
- new net: D89.2 (A), MX89.2
- new net: D57.2 (A), MX57.2
- new net: D90.1 (K), MX90.2
- new net: D42.1 (K), MX42.2
- new net: D3.2 (A), MX3.2
- new net: D2.1 (K), MX2.2
- new net: D95.2 (A), MX95.2
- new net: LED60.3 (DIN), LED61.2 (DOUT)
- new net: D4.1 (K), MX4.2
Other:
- moved on the sheet: D113, D114, D115, LED1, LED10, LED100, LED101, LED102, LED103, LED104, LED105, LED106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

Commit message: check ing
Parts:
- removed D65, D85: D, Keyboard:D_SOD-123F, symbol Device:D
- removed LED112, LED113: MX_SK6803MINI-E, Keyboard:LED_MX_6028R-ROT, symbol Keyboard:MX_SK6803MINI-E
- removed MX65, MX85: MX_SW_HS, Keyboard:SW_MX_HS_1u, symbol PCM_marbastlib-mx:MX_SW_HS_CPG151101S11
- added C30, C31, C32, C33: 100nF, Capacitor_SMD:C_0805_2012Metric, symbol Device:C
- added D114: D, Keyboard:D_SOD-123F, symbol Device:D
- added R21, R22, R23, R24, R25, R26, R27, R28: 5.1k, Resistor_SMD:R_0805_2012Metric, symbol Device:R
- added SW4: RotaryEncoder_Switch, Keyboard:RotaryEncoder_Alps_EC11E-Switch_Vertical_H20mm_Centred, symbol Device:RotaryEncoder_Switch
- LED79: footprint Keyboard:LED_MX_6028R-ROT -> Keyboard:LED_MX_6028R
- LED98, LED99: footprint Keyboard:LED_MX_6028R -> Keyboard:LED_MX_6028R-ROT
- MX100: renamed from MX102; footprint Keyboard:SW_MX_HS_1u -> Keyboard:SW_MX_HS_2u
- MX101: renamed from MX103; footprint Keyboard:SW_MX_HS_1u -> Keyboard:SW_MX_HS_1.25u
- MX102: renamed from MX104; footprint Keyboard:SW_MX_HS_1u -> Keyboard:SW_MX_HS_1.25u
- MX103: renamed from MX105; footprint Keyboard:SW_MX_HS_1u -> Keyboard:SW_MX_HS_1.25u
- MX104: renamed from MX106; footprint Keyboard:SW_MX_HS_1u -> Keyboard:SW_MX_HS_2.75u
- MX105: renamed from MX107; footprint Keyboard:SW_MX_HS_1u -> Keyboard:SW_MX_HS_1.25u
- MX106: renamed from MX108; footprint Keyboard:SW_MX_HS_1u -> Keyboard:SW_MX_HS_2.25u
- MX107: renamed from MX109; footprint Keyboard:SW_MX_HS_1u -> Keyboard:SW_MX_HS_1.5u
- MX108: renamed from MX110; footprint Keyboard:SW_MX_HS_1u -> Keyboard:SW_MX_HS_1.5u
- MX18, MX38: footprint Keyboard:SW_MX_HS_1u -> Keyboard:SW_MX_HS_2u
- MX45, MX58: footprint Keyboard:SW_MX_HS_1u -> Keyboard:SW_MX_HS_1.5u
- MX65: renamed from MX66; footprint Keyboard:SW_MX_HS_1u -> Keyboard:SW_MX_HS_1.75u
- MX77: renamed from MX78; footprint Keyboard:SW_MX_HS_1u -> Keyboard:SW_MX_HS_2.25u
- MX80: renamed from MX81; footprint Keyboard:SW_MX_HS_1u -> Keyboard:SW_MX_HS_2u_Vertical
- MX84: renamed from MX86; footprint Keyboard:SW_MX_HS_1u -> Keyboard:SW_MX_HS_2.25u
- MX95: renamed from MX97; footprint Keyboard:SW_MX_HS_1u -> Keyboard:SW_MX_HS_1.75u
- Q7: footprint Package_TO_SOT_SMD:SOT-23-3 -> Package_TO_SOT_SMD:SOT-23
- U1: footprint Package_TO_SOT_SMD:SOT-223-3_TabPin2 -> Package_TO_SOT_SMD:SOT-23-3
- U4: footprint Package_SO:SOIC-8_5.275x5.275mm_P1.27mm -> Package_SO:SOIC-8_5.23x5.23mm_P1.27mm
- U5: footprint Package_TO_SOT_SMD:SOT-143_Handsoldering -> Package_TO_SOT_SMD:SOT-143
- renumbered D102 to D100, D103 to D101, D104 to D102, D105 to D103, D106 to D104, D107 to D105, D108 to D106, D109 to D107, D110 to D108, D111 to D109, D112 to D110, D116 to D111, D113 to D112, D114 to D113, D66 to D65, D67 to D66, D68 to D67, D69 to D68, D70 to D69, D71 to D70, D72 to D71, D73 to D72, D74 to D73, D75 to D74, D76 to D75, D77 to D76, D78 to D77, D79 to D78, D80 to D79, D81 to D80, D82 to D81, D83 to D82, D84 to D83, D86 to D84, D87 to D85, D88 to D86, D89 to D87, D90 to D88, D91 to D89, D92 to D90, D93 to D91, D94 to D92, D95 to D93, D96 to D94, D97 to D95, D98 to D96, D99 to D97, D100 to D98, D101 to D99, MX111 to MX109, MX112 to MX110, MX113 to MX111, MX67 to MX66, MX68 to MX67, MX69 to MX68, MX70 to MX69, MX71 to MX70, MX72 to MX71, MX73 to MX72, MX74 to MX73, MX75 to MX74, MX76 to MX75, MX77 to MX76, MX79 to MX78, MX80 to MX79, MX82 to MX81, MX83 to MX82, MX84 to MX83, MX87 to MX85, MX88 to MX86, MX89 to MX87, MX90 to MX88, MX91 to MX89, MX92 to MX90, MX93 to MX91, MX94 to MX92, MX95 to MX93, MX96 to MX94, MX98 to MX96, MX99 to MX97, MX100 to MX98, MX101 to MX99, S1 to SW3
Connections:
- net +3V3: now also R21.2, R22.2, R25.2, R26.2
- net ENC1_A: now also U6.31 (GPIO20); no longer U6.38 (GPIO26_ADC0)
- net ENC1_B: now also U6.32 (GPIO21), C33.2, R28.2; no longer U6.39 (GPIO27_ADC1)
- net ENC2_A: now also U6.35 (GPIO23); no longer U6.31 (GPIO20)
- net ENC2_B: now also U6.38 (GPIO26_ADC0), C31.2, R24.2; no longer U6.32 (GPIO21)
- net GND: now also LED100.4 (VSS), LED101.4 (VSS), LED102.4 (VSS), LED103.4 (VSS), LED104.4 (VSS), LED105.4 (VSS), LED106.4 (VSS), LED107.4 (VSS), LED108.4 (VSS), LED109.4 (VSS), LED110.4 (VSS), LED111.4 (VSS), LED20.4 (VSS), LED21.4 (VSS), LED22.4 (VSS), LED23.4 (VSS), LED24.4 (VSS), LED25.4 (VSS), LED26.4 (VSS), LED27.4 (VSS), LED28.4 (VSS), LED29.4 (VSS), LED30.4 (VSS), LED31.4 (VSS), LED32.4 (VSS), LED33.4 (VSS), LED34.4 (VSS), LED35.4 (VSS), LED36.4 (VSS), LED37.4 (VSS), LED38.4 (VSS), LED39.4 (VSS), LED40.1 (VDD), LED41.1 (VDD), LED42.1 (VDD), LED43.1 (VDD), LED44.1 (VDD), LED45.1 (VDD), LED46.1 (VDD), LED47.1 (VDD), LED48.1 (VDD), LED49.1 (VDD), LED50.1 (VDD), LED51.1 (VDD), LED52.1 (VDD), LED53.1 (VDD), LED54.1 (VDD), LED55.1 (VDD), LED56.1 (VDD), LED57.1 (VDD), LED58.1 (VDD), LED59.1 (VDD), LED79.1 (VDD), LED80.1 (VDD), LED81.1 (VDD), LED82.1 (VDD), LED83.1 (VDD), LED84.1 (VDD), LED85.1 (VDD), LED86.1 (VDD), LED87.1 (VDD), LED88.1 (VDD), LED89.1 (VDD), LED90.1 (VDD), LED91.1 (VDD), LED92.1 (VDD), LED93.1 (VDD), LED94.1 (VDD), LED95.1 (VDD), LED96.1 (VDD), LED97.1 (VDD), C30.1, C31.1, C32.1, C33.1, SW4.C; no longer LED100.1 (VDD), LED101.1 (VDD), LED102.1 (VDD), LED103.1 (VDD), LED104.1 (VDD), LED105.1 (VDD), LED106.1 (VDD), LED107.1 (VDD), LED108.1 (VDD), LED109.1 (VDD), LED110.1 (VDD), LED111.1 (VDD), LED20.1 (VDD), LED21.1 (VDD), LED22.1 (VDD), LED23.1 (VDD), LED24.1 (VDD), LED25.1 (VDD), LED26.1 (VDD), LED27.1 (VDD), LED28.1 (VDD), LED29.1 (VDD), LED30.1 (VDD), LED31.1 (VDD), LED32.1 (VDD), LED33.1 (VDD), LED34.1 (VDD), LED35.1 (VDD), LED36.1 (VDD), LED37.1 (VDD), LED38.1 (VDD), LED39.1 (VDD), LED40.4 (VSS), LED41.4 (VSS), LED42.4 (VSS), LED43.4 (VSS), LED44.4 (VSS), LED45.4 (VSS), LED46.4 (VSS), LED47.4 (VSS), LED48.4 (VSS), LED49.4 (VSS), LED50.4 (VSS), LED51.4 (VSS), LED52.4 (VSS), LED53.4 (VSS), LED54.4 (VSS), LED55.4 (VSS), LED56.4 (VSS), LED57.4 (VSS), LED58.4 (VSS), LED59.4 (VSS), LED80.4 (VSS), LED81.4 (VSS), LED82.4 (VSS), LED83.4 (VSS), LED84.4 (VSS), LED85.4 (VSS), LED86.4 (VSS), LED87.4 (VSS), LED88.4 (VSS), LED89.4 (VSS), LED90.4 (VSS), LED91.4 (VSS), LED92.4 (VSS), LED93.4 (VSS), LED94.4 (VSS), LED95.4 (VSS), LED96.4 (VSS), LED97.4 (VSS)
- net LCD_EN: no longer U6.35 (GPIO23)
- net LED_PWR: now also LED100.1 (VDD), LED101.1 (VDD), LED102.1 (VDD), LED103.1 (VDD), LED104.1 (VDD), LED105.1 (VDD), LED106.1 (VDD), LED107.1 (VDD), LED108.1 (VDD), LED109.1 (VDD), LED110.1 (VDD), LED111.1 (VDD), LED20.1 (VDD), LED21.1 (VDD), LED22.1 (VDD), LED23.1 (VDD), LED24.1 (VDD), LED25.1 (VDD), LED26.1 (VDD), LED27.1 (VDD), LED28.1 (VDD), LED29.1 (VDD), LED30.1 (VDD), LED31.1 (VDD), LED32.1 (VDD), LED33.1 (VDD), LED34.1 (VDD), LED35.1 (VDD), LED36.1 (VDD), LED37.1 (VDD), LED38.1 (VDD), LED39.1 (VDD), LED40.4 (VSS), LED41.4 (VSS), LED42.4 (VSS), LED43.4 (VSS), LED44.4 (VSS), LED45.4 (VSS), LED46.4 (VSS), LED47.4 (VSS), LED48.4 (VSS), LED49.4 (VSS), LED50.4 (VSS), LED51.4 (VSS), LED52.4 (VSS), LED53.4 (VSS), LED54.4 (VSS), LED55.4 (VSS), LED56.4 (VSS), LED57.4 (VSS), LED58.4 (VSS), LED59.4 (VSS), LED79.4 (VSS), LED80.4 (VSS), LED81.4 (VSS), LED82.4 (VSS), LED83.4 (VSS), LED84.4 (VSS), LED85.4 (VSS), LED86.4 (VSS), LED87.4 (VSS), LED88.4 (VSS), LED89.4 (VSS), LED90.4 (VSS), LED91.4 (VSS), LED92.4 (VSS), LED93.4 (VSS), LED94.4 (VSS), LED95.4 (VSS), LED96.4 (VSS), LED97.4 (VSS); no longer LED100.4 (VSS), LED101.4 (VSS), LED102.4 (VSS), LED103.4 (VSS), LED104.4 (VSS), LED105.4 (VSS), LED106.4 (VSS), LED107.4 (VSS), LED108.4 (VSS), LED109.4 (VSS), LED110.4 (VSS), LED111.4 (VSS), LED20.4 (VSS), LED21.4 (VSS), LED22.4 (VSS), LED23.4 (VSS), LED24.4 (VSS), LED25.4 (VSS), LED26.4 (VSS), LED27.4 (VSS), LED28.4 (VSS), LED29.4 (VSS), LED30.4 (VSS), LED31.4 (VSS), LED32.4 (VSS), LED33.4 (VSS), LED34.4 (VSS), LED35.4 (VSS), LED36.4 (VSS), LED37.4 (VSS), LED38.4 (VSS), LED39.4 (VSS), LED40.1 (VDD), LED41.1 (VDD), LED42.1 (VDD), LED43.1 (VDD), LED44.1 (VDD), LED45.1 (VDD), LED46.1 (VDD), LED47.1 (VDD), LED48.1 (VDD), LED49.1 (VDD), LED50.1 (VDD), LED51.1 (VDD), LED52.1 (VDD), LED53.1 (VDD), LED54.1 (VDD), LED55.1 (VDD), LED56.1 (VDD), LED57.1 (VDD), LED58.1 (VDD), LED59.1 (VDD), LED80.1 (VDD), LED81.1 (VDD), LED82.1 (VDD), LED83.1 (VDD), LED84.1 (VDD), LED85.1 (VDD), LED86.1 (VDD), LED87.1 (VDD), LED88.1 (VDD), LED89.1 (VDD), LED90.1 (VDD), LED91.1 (VDD), LED92.1 (VDD), LED93.1 (VDD), LED94.1 (VDD), LED95.1 (VDD), LED96.1 (VDD), LED97.1 (VDD)
- net ROT2_A: no longer SW3.10 (ENCODER_A)
- net ROT2_B: no longer SW3.5 (ENCODER_B)
- net ROW3: now also D114.1 (K)
- net at LED99.3 (DIN): now also LED98.3 (DIN); no longer LED98.2 (DOUT)
- net at LED96.2 (DOUT): now also LED97.3 (DIN)
- net at LED96.3 (DIN): now also LED95.2 (DOUT)
- net at LED90.2 (DOUT): now also LED91.3 (DIN)
- net at LED90.3 (DIN): now also LED89.2 (DOUT)
- net at LED91.2 (DOUT): now also LED92.3 (DIN)
- net at LED111.3 (DIN): now also LED97.2 (DOUT)
- net at LED78.3 (DIN): now also LED59.2 (DOUT)
- net ENC4_A: now reaches U6.34 (GPIO22)
- net ENC4_A: now also C32.2, R27.1
- net at LED95.3 (DIN): now also LED94.2 (DOUT)
- net at LED80.3 (DIN): now also LED79.2 (DOUT); no longer LED60.2 (DOUT)
- net at LED93.2 (DOUT): now also LED94.3 (DIN)
- net at LED79.3 (DIN): now also LED60.2 (DOUT); no longer LED59.2 (DOUT)
- net at LED88.2 (DOUT): now also LED89.3 (DIN)
- net ROT1_D: no longer names the net of D112.1 (K), SW1.S2
- net ROT2_D: no longer names the net of D113.2 (A), SW2.S2
- new net: D114.2 (A), SW4.S2
- new net ENC3_A: C30.2, R23.1, U6.39 (GPIO27_ADC1)
- new net ROT3_A: R21.1, R23.2, SW4.A
- new net ROT3_B: R22.1, R24.1, SW4.B
- new net ROT4_A: R25.1, R27.2, SW3.10 (ENCODER_A)
- new net ROT4_B: R26.1, R28.1, SW3.5 (ENCODER_B)
Other:
- moved on the sheet: C26, C27, C28, C29, D112, D113, LED100, LED101, LED102, LED103, LED104, LED105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
