File: Overkill/STM32/STM32.kicad_pcb (KiCad board)
At the start: 2 copper layers, 3.6 x 3.3 mm, 460 parts, among them J1 USB_C_Receptacle_USB2.0, Q1 MMUN2133LT1G, Q2 AO3401A, Q3 AO3401A, Q4 AO3401A, Q5 MMUN2233LT1G, Q6 2N7002, Q7 2N7002, SW1 RotaryEncoder_Switch, SW2 RotaryEncoder_Switch, SW3 RKJXT1F42001, SW4 RotaryEncoder_Switch, U10 W25Q32JVSSIQ, U2 TPS2553DBVR, U3 74AHC1G125, U4 AZ1117H-3.3TRE1, U5 TPS2553DBVR-1, U6 LMV321, U7 AZC199-04S, U8 MB85RS64, U9 TPS2553DBVR-1

Commit message: daily
Parts:
- removed BOOT1, RST1: SW_Push, Button_Switch_SMD:SW_SPST_TL3342
- removed C25, C34, C35, C36: 100n, Capacitor_SMD:C_0805_2012Metric
- removed R19, R42, R7: 68k, Resistor_SMD:R_0805_2012Metric
- removed R41, R43, R6: 9.1k, Resistor_SMD:R_0805_2012Metric
- removed R5: 120, Resistor_SMD:R_0805_2012Metric
- removed U10: W25Q32JVSSIQ, Package_SO:SOIC-8_5.23x5.23mm_P1.27mm
- removed U9: TPS2553DBVR-1, Package_TO_SOT_SMD:SOT-23-6_Handsoldering
- added C10: 100n, Capacitor_SMD:C_0603_1608Metric_Pad1.08x0.95mm_HandSolder, B.Cu at (136.6, 88.9)
- added C4: 100n, Capacitor_SMD:C_0603_1608Metric_Pad1.08x0.95mm_HandSolder, B.Cu at (193.5, 179.6)
- added U1: AZC199-04S, Package_TO_SOT_SMD:SOT-23-6, B.Cu at (147.7, 54.8)
- C1: value 100nF -> 1u; footprint Capacitor_SMD:C_0402_1005Metric -> Capacitor_SMD:C_0603_1608Metric_Pad1.08x0.95mm_HandSolder
- C11, C28, C9: footprint Capacitor_SMD:C_0805_2012Metric -> Capacitor_SMD:C_0603_1608Metric_Pad1.08x0.95mm_HandSolder; moved to B.Cu
- C12: value 4.7u -> 100n; footprint Capacitor_SMD:C_0805_2012Metric -> Capacitor_SMD:C_0603_1608Metric_Pad1.08x0.95mm_HandSolder; moved to B.Cu
- C13: value 100nF -> 100n; footprint Capacitor_SMD:C_0402_1005Metric -> Capacitor_SMD:C_0603_1608Metric_Pad1.08x0.95mm_HandSolder; moved to B.Cu
- C14, C15, C16: value 100u -> 100n; footprint Capacitor_Tantalum_SMD:CP_EIA-6032-15_Kemet-U -> Capacitor_SMD:C_0603_1608Metric_Pad1.08x0.95mm_HandSolder; moved to B.Cu
- C17: value 100u -> 4.7u; footprint Capacitor_Tantalum_SMD:CP_EIA-6032-15_Kemet-U -> Capacitor_SMD:C_0603_1608Metric_Pad1.08x0.95mm_HandSolder; moved to B.Cu
- C18, C19: footprint Capacitor_Tantalum_SMD:CP_EIA-6032-15_Kemet-U -> Capacitor_Tantalum_SMD:CP_EIA-6032-15_Kemet-U_Pad2.25x2.35mm_HandSolder; moved to B.Cu
- C2: footprint Capacitor_SMD:C_0402_1005Metric -> Capacitor_SMD:C_0603_1608Metric_Pad1.08x0.95mm_HandSolder
- C20: footprint Capacitor_Tantalum_SMD:CP_EIA-6032-15_Kemet-U -> Capacitor_Tantalum_SMD:CP_EIA-6032-15_Kemet-U_Pad2.25x2.35mm_HandSolder
- C21, C22, C23, C24: value 100n -> 100u; footprint Capacitor_SMD:C_0805_2012Metric -> Capacitor_Tantalum_SMD:CP_EIA-6032-15_Kemet-U_Pad2.25x2.35mm_HandSolder
- C26, C27: value 100nF -> 100n; footprint Capacitor_SMD:C_0805_2012Metric -> Capacitor_SMD:C_0603_1608Metric_Pad1.08x0.95mm_HandSolder
- C29, C30, C31, C32, C33: value 100nF -> 100n; footprint Capacitor_SMD:C_0805_2012Metric -> Capacitor_SMD:C_0603_1608Metric_Pad1.08x0.95mm_HandSolder; moved to B.Cu
- C3: value 1u -> 100n; footprint Capacitor_SMD:C_0402_1005Metric -> Capacitor_SMD:C_0603_1608Metric_Pad1.08x0.95mm_HandSolder; moved to B.Cu
- C5, C6: footprint Capacitor_SMD:C_0805_2012Metric -> Capacitor_SMD:C_0603_1608Metric_Pad1.08x0.95mm_HandSolder
- C7: value 4.7u -> 100n; footprint Capacitor_SMD:C_0805_2012Metric -> Capacitor_SMD:C_0603_1608Metric_Pad1.08x0.95mm_HandSolder
- C8: value 100n -> 4.7u; footprint Capacitor_SMD:C_0805_2012Metric -> Capacitor_SMD:C_0603_1608Metric_Pad1.08x0.95mm_HandSolder; moved to B.Cu
- D116: value 1N4148 -> SMF5.0CA; moved to B.Cu
- D117: value SMF5.0CA -> 1N4148
- F1: footprint Fuse:Fuse_1206_3216Metric -> Fuse:Fuse_1206_3216Metric_Pad1.42x1.75mm_HandSolder; moved to B.Cu
- FB1: footprint Capacitor_SMD:C_0805_2012Metric -> Fuse:Fuse_0805_2012Metric_Pad1.15x1.40mm_HandSolder; moved to B.Cu
- J1: footprint Keyboard:HRO-TYPE-C-31-M-12-modded -> Keyboard:HRO-TYPE-C-31-M-12-HandSoldering-NoSBU; moved to F.Cu
- Q1: value MMUN2133LT1G -> AO3401A; moved to B.Cu
- Q2, Q6, Q7: moved to B.Cu
- Q3: value AO3401A -> MMUN2133LT1G
- R1: value 5.1k -> 9.1k; footprint Resistor_SMD:R_0402_1005Metric -> Resistor_SMD:R_0603_1608Metric_Pad0.98x0.95mm_HandSolder; moved to B.Cu
- R10, R11, R15, R16, R21, R22, R23, R24, R25, R27, R28: value 5.1k -> 9.1k; footprint Resistor_SMD:R_0805_2012Metric -> Resistor_SMD:R_0603_1608Metric_Pad0.98x0.95mm_HandSolder; moved to B.Cu
- R12, R14, R8, R9: value 5.1k -> 9.1k; footprint Resistor_SMD:R_0805_2012Metric -> Resistor_SMD:R_0603_1608Metric_Pad0.98x0.95mm_HandSolder
- R13: value 9.1k -> 120; footprint Resistor_SMD:R_0805_2012Metric -> Resistor_SMD:R_0603_1608Metric_Pad0.98x0.95mm_HandSolder
- R17, R18: footprint Resistor_SMD:R_0805_2012Metric -> Resistor_SMD:R_0603_1608Metric_Pad0.98x0.95mm_HandSolder
- R2: value 75k -> 68k; footprint Resistor_SMD:R_0402_1005Metric -> Resistor_SMD:R_0603_1608Metric_Pad0.98x0.95mm_HandSolder; moved to B.Cu
- R20, R31: value 68k -> 9.1k; footprint Resistor_SMD:R_0805_2012Metric -> Resistor_SMD:R_0603_1608Metric_Pad0.98x0.95mm_HandSolder; moved to B.Cu
- R26, R29, R30, R33, R34, R38, R39: footprint Resistor_SMD:R_0805_2012Metric -> Resistor_SMD:R_0603_1608Metric_Pad0.98x0.95mm_HandSolder; moved to B.Cu
- R3: value 5.1k -> 68k; footprint Resistor_SMD:R_0402_1005Metric -> Resistor_SMD:R_0603_1608Metric_Pad0.98x0.95mm_HandSolder; moved to B.Cu
- R32: value 68k -> 9.1k; footprint Resistor_SMD:R_0805_2012Metric -> Resistor_SMD:R_0603_1608Metric_Pad0.98x0.95mm_HandSolder
- R35, R36, R37: value 5.1K -> 68k; footprint Resistor_SMD:R_0402_1005Metric -> Resistor_SMD:R_0603_1608Metric_Pad0.98x0.95mm_HandSolder; moved to B.Cu
- R4: value 9.1k -> 68k; footprint Resistor_SMD:R_0805_2012Metric -> Resistor_SMD:R_0603_1608Metric_Pad0.98x0.95mm_HandSolder; moved to B.Cu
- R40: value 1k -> 9.1k; footprint Resistor_SMD:R_0402_1005Metric -> Resistor_SMD:R_0603_1608Metric_Pad0.98x0.95mm_HandSolder; moved to B.Cu
- SW3: value RKJXT1F42001 -> RotaryEncoder_Switch; footprint Keyboard:RKJXT1F42001 -> Keyboard:RotaryEncoder_Alps_EC11E-Switch_Vertical_H20mm_Centred
- SW4: value RotaryEncoder_Switch -> RKJXT1F42001; footprint Keyboard:RotaryEncoder_Alps_EC11E-Switch_Vertical_H20mm_Centred -> Keyboard:RKJXT1F42001
- U2: value TPS2553DBVR -> LMV321; footprint Package_TO_SOT_SMD:SOT-23-6 -> Package_TO_SOT_SMD:SOT-23-5; moved to B.Cu
- U3: value 74AHC1G125 -> W25Q32JVSSIQ; footprint Package_TO_SOT_SMD:SOT-23-5 -> Package_SO:SOIC-8_5.23x5.23mm_P1.27mm; moved to B.Cu
- U4: value AZ1117H-3.3TRE1 -> MB85RS64; footprint Package_TO_SOT_SMD:SOT-23-3 -> Package_SO:SOIC-8_3.9x4.9mm_P1.27mm; moved to B.Cu
- U5: value TPS2553DBVR-1 -> AZ1117H-3.3TRE1; footprint Package_TO_SOT_SMD:SOT-23-6_Handsoldering -> Package_TO_SOT_SMD:SOT-23-3
- U6: value LMV321 -> STM32G474RETx; footprint Package_TO_SOT_SMD:SOT-23-5 -> Package_QFP:LQFP-64_10x10mm_P0.5mm; moved to B.Cu
- U7: value AZC199-04S -> TPS2553DBVR-1; footprint Package_TO_SOT_SMD:SOT-23-6 -> Package_TO_SOT_SMD:SOT-23-6_Handsoldering; moved to B.Cu
- U8: value MB85RS64 -> TPS2553DBVR-1; footprint Package_SO:SOIC-8_3.9x4.9mm_P1.27mm -> Package_TO_SOT_SMD:SOT-23-6_Handsoldering; moved to B.Cu
- moved C18 359.4 mm to (209.0, -173.1), turned to 180 degrees
- moved C17 354.6 mm to (201.9, -180.7), turned to -90 degrees
- moved C3 339.3 mm to (193.5, 187.9), turned to 90 degrees
- moved R20 338.1 mm to (204.2, -184.3)
- moved U4 333.7 mm to (197.7, 191.5), turned to -90 degrees
- moved U3 323.8 mm to (197.6, 182.5), turned to -90 degrees
- moved R31 323.5 mm to (191.2, -175.8), turned to 180 degrees
- moved U7 317.1 mm to (206.7, -180.7)
- moved C16 303.7 mm to (143.2, 163.3), turned to 180 degrees
- moved C19 302.6 mm to (145.3, 172.5), turned to 180 degrees
- moved Q7 293.0 mm to (164.9, 165.6), turned to 180 degrees
- moved Q6 292.8 mm to (164.9, 160.6), turned to 180 degrees
- moved R39 291.3 mm to (159.4, 163.0), turned to 90 degrees
- moved R38 289.6 mm to (155.1, 163.0), turned to 90 degrees
- moved R33 288.0 mm to (143.2, 169.5), turned to 180 degrees
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Connections:
- C13 pad 1: LED_PWR -> +3V3
- C14 pad 1: LED_PWR -> +3V3
- C15 pad 1: LED_PWR -> +3V3
- C16 pad 1: LED_PWR -> VDD
- C17 pad 1: LED_PWR -> VBUS
- C18 pad 1: LED_PWR -> VDD
- C2 pad 2: +5V -> +3V3
- C21 pad 1: VDD -> LED_PWR
- C22 pad 1: +3V3 -> LED_PWR
- C23 pad 1: +3V3 -> LED_PWR
- C24 pad 1: +3V3 -> LED_PWR
- C3 pad 1: GND -> +3V3
- C3 pad 2: +3V3 -> GND
- C5 pad 2: BOOT0 -> NRST
- C7 pad 1: VBUS -> GND
- C7 pad 2: GND -> BOOT0
- C9 pad 1: GND -> +3V3
- C9 pad 2: NRST -> GND
- D116 pad 1: Net-(D116-K) -> /VBUS_FUSED
- D116 pad 2: BOOT0_CHRG -> GND
- D117 pad 1: /VBUS_FUSED -> Net-(D117-K)
- D117 pad 2: GND -> BOOT0_CHRG
- D118 pad 1: Net-(D116-K) -> Net-(D117-K)
- D23 pad 1: Net-(D23-K) -> ROW1
- D23 pad 2: ROW1 -> Net-(D23-A)
- LED1 pad 3: LED_DAT_5V -> LED_MTRX_IN
- MX23 pad 2: Net-(D23-K) -> Net-(D23-A)
- Q1 pad 1: BOOT0_CHRG -> GND
- Q1 pad 2: +3V3 -> /VBUS_BLOCKED
- Q1 pad 3: Net-(Q1-C) -> /VBUS_FUSED
- Q2 pad 1: GND -> Net-(Q2-G)
- Q2 pad 2: /VBUS_BLOCKED -> VBUS
- Q2 pad 3: /VBUS_FUSED -> /VBUS_BLOCKED
- Q3 pad 1: Net-(Q3-G) -> BOOT0_CHRG
- Q3 pad 2: VBUS -> +3V3
- Q3 pad 3: /VBUS_BLOCKED -> Net-(Q3-C)
- R1 pad 1: LED_NFAULT -> LED_PWR
- R1 pad 2: +5V -> LED_MTRX_IN
- R13 pad 1: Net-(R13-Pad1) -> Net-(Q3-C)
- R13 pad 2: GND -> BOOT0
- R17 pad 1: /VBUS_BLOCKED -> Net-(R17-Pad1)
- R17 pad 2: PLUG_DETECT -> BOOT0
- R18 pad 1: Net-(R18-Pad1) -> Net-(R17-Pad1)
- R2 pad 1: C_ILIM -> /VBUS_BLOCKED
- R2 pad 2: GND -> PLUG_DETECT
- R20 pad 1: Net-(R19-Pad2) -> VBUS
- R20 pad 2: GND -> BOARD_NFAULT
- R29 pad 2: SK6812_NFAULT -> LED_NFAULT
- R3 pad 1: GND -> PLUG_DETECT
- R3 pad 2: LED_EN -> Net-(R3-Pad2)
- R30 pad 1: SK6812_EN -> LED_EN
- R31 pad 1: CURR_LIM -> Net-(U7-ILIM)
- R32 pad 1: CURR_LIM -> Net-(R31-Pad2)
- R32 pad 2: Net-(Q6-D) -> GND
- R33 pad 2: Net-(Q7-D) -> Net-(R33-Pad2)
- R34 pad 1: CURR_LIM -> Net-(R34-Pad1)
- R34 pad 2: Net-(Q7-D) -> Net-(R33-Pad2)
- R35 pad 1: Net-(R35-Pad1) -> Net-(R34-Pad1)
- R35 pad 2: +3V3 -> GND
- R36 pad 1: RESET -> CURR_LIM
- R36 pad 2: +3V3 -> Net-(Q6-D)
- R37 pad 1: QSPI_SS -> CURR_LIM
- R37 pad 2: Net-(R35-Pad1) -> Net-(Q7-D)
- R38 pad 1: Net-(R38-Pad1) -> CURR_LIM
- R38 pad 2: Net-(R31-Pad2) -> Net-(Q7-D)
- R39 pad 1: SK6812_PWR -> CURR_1500mA_OK
- R39 pad 2: SK6812_PWM -> GND
- R4 pad 1: VBUS -> Net-(R3-Pad2)
- R4 pad 2: BOARD_NFAULT -> GND
- R40 pad 1: Net-(BOOT1-Pad1) -> CURR_3000mA_OK
- R40 pad 2: QSPI_SS -> GND
- U2 pad 1: +5V -> VBUS
- U2 pad 3: LED_EN -> /VBUS_BLOCKED
- U2 pad 4: LED_NFAULT -> Net-(Q2-G)
- U2 pad 5: C_ILIM -> VBUS
- U3 pad 1: GND -> FLASH_CS
- U3 pad 2: LED_DAT_3V3 -> MISO
- U3 pad 3: GND -> unconnected-(U3-IO2-Pad3)
- U3 pad 4: LED_DAT_5V -> GND
- U3 pad 5: LED_PWR -> MOSI
- U4 pad 1: GND -> EEP_CS
- U4 pad 2: +3V3 -> MISO
- U4 pad 3: +5V -> +3V3
- U5 pad 1: VBUS -> GND
- U5 pad 2: GND -> +3V3
- U5 pad 3: VBUS -> +5V
- U6 pad 1: VBUS -> +3V3
- U6 pad 2: GND -> unconnected-(U6-PC13-Pad2)
- U6 pad 3: /VBUS_BLOCKED -> ENC_A
- U6 pad 4: Net-(Q3-G) -> ENC_B
- U6 pad 5: VBUS -> unconnected-(U6-PF0-Pad5)
- U7 pad 1: CC2 -> VBUS
- U7 pad 3: CC1 -> VBUS
- U7 pad 4: D- -> BOARD_NFAULT
- U7 pad 5: /VBUS_BLOCKED -> Net-(U7-ILIM)
- U7 pad 6: D+ -> VDD
- U8 pad 1: EEP_CS -> VDD
- U8 pad 2: MISO -> GND
- U8 pad 3: +3V3 -> LED_EN
- U8 pad 4: GND -> LED_NFAULT
- U8 pad 5: MOSI -> CURR_LIM
- U8 pad 6: SCK -> LED_PWR
Routing:
- net ROW5: track 0.00 -> 433.4 mm
- net ROW0: track 0.00 -> 368.3 mm
- net ROW1: track 0.00 -> 366.7 mm
- net ROW2: track 0.00 -> 361.9 mm
- net ROW3: track 0.00 -> 359.4 mm
- net ROW4: track 0.00 -> 311.9 mm
- net COL3: track 0.00 -> 250.2 mm
- net COL8: track 0.00 -> 243.8 mm
- net COL9: track 0.00 -> 215.4 mm
- net COL5: track 0.00 -> 211.6 mm
- net COL4: track 0.00 -> 211.6 mm
- net COL6: track 0.00 -> 209.6 mm
- net COL7: track 0.00 -> 208.6 mm
- net COL1: track 0.00 -> 181.0 mm
- net COL0: track 0.00 -> 166.7 mm
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