File: Overkill/STM32/STM32.kicad_pcb (KiCad board)
At the start: 2 copper layers, 3.6 x 3.3 mm, 443 parts, among them J1 USB_C_Receptacle_USB2.0, Q1 AO3401A, Q2 AO3401A, Q3 MMUN2133LT1G, Q4 2N7002, Q5 AO3401A, Q6 2N7002, Q7 MMUN2233LT1G, SW1 RKJXT1F42001, SW2 RotaryEncoder_Switch, U1 AZC199-04S, U2 W25Q32JVSSIQ, U3 LMV321, U4 MB85RS64, U5 AZ1117H-3.3TRE1, U6 STM32G474RETx, U7 TPS2553DBVR-1, U8 TPS2553DBVR-1

Commit message: Rotate mcu & wire nets
Parts:
- moved C28 43.1 mm to (171.4, 77.7)
- moved C30 42.9 mm to (166.7, 34.8)
- moved C5 27.3 mm to (127.8, 69.1), turned to -90 degrees
- moved R7 24.1 mm to (157.0, 124.3), turned to 0 degrees
- moved R8 23.6 mm to (157.0, 122.6), turned to 180 degrees
- moved C19 23.5 mm to (157.0, 121.0), turned to 0 degrees
- moved RESET1 18.9 mm to (132.8, 99.2)
- moved C9 18.4 mm to (132.4, 93.8)
- moved D119 18.4 mm to (136.0, 91.9)
- moved D120 18.4 mm to (136.0, 94.6)
- moved C8 15.3 mm to (134.9, 76.5), turned to 180 degrees
- moved D113 13.6 mm to (130.5, 105.7)
- moved D114 13.6 mm to (130.5, 108.3)
- moved D116 13.6 mm to (130.5, 113.5)
- moved D117 13.6 mm to (130.5, 116.1)
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Connections:
- U6 pad 10: LCD_BL_PWM -> unconnected-(U6-PC2-Pad10)
- U6 pad 17: unconnected-(U6-PA3-Pad17) -> COL2
- U6 pad 18: unconnected-(U6-PA4-Pad18) -> ROW0
- U6 pad 19: unconnected-(U6-PA5-Pad19) -> COL1
- U6 pad 2: LCD_RST -> LCD_BL_PWM
- U6 pad 20: ROW5 -> COL0
- U6 pad 21: ROW4 -> ENC2_A
- U6 pad 22: ROW3 -> ENC2_B
- U6 pad 23: ROW2 -> LED_MTRX_IN
- U6 pad 24: ROW1 -> CURR_3000mA_OK
- U6 pad 25: COL2 -> CURR_1500mA_OK
- U6 pad 26: COL1 -> LED_NFAULT
- U6 pad 3: ENC1_B -> unconnected-(U6-PC14-Pad3)
- U6 pad 30: COL0 -> BOARD_NFAULT
- U6 pad 33: ROW0 -> LED_EN
- U6 pad 35: ENC2_A -> COL9
- U6 pad 36: ENC2_B -> COL8
- U6 pad 37: LED_MTRX_IN -> COL7
- U6 pad 38: CURR_3000mA_OK -> COL6
- U6 pad 39: CURR_1500mA_OK -> COL5
- U6 pad 4: ENC1_A -> unconnected-(U6-PC15-Pad4)
- U6 pad 40: LED_NFAULT -> COL4
- U6 pad 41: LED_EN -> COL3
- U6 pad 51: unconnected-(U6-PA15-Pad51) -> LCD_EN
- U6 pad 55: unconnected-(U6-PD2-Pad55) -> LCD_RST
- U6 pad 56: unconnected-(U6-PB3-Pad56) -> LCD_DC
- U6 pad 62: LCD_EN -> LCD_CS
- U6 pad 8: LCD_DC -> unconnected-(U6-PC0-Pad8)
- U6 pad 9: LCD_CS -> unconnected-(U6-PC1-Pad9)
Routing:
- net +3V3: track 59.5 -> 332.4 mm, vias 2 -> 12
- net LED_PWR: track 2576.1 -> 2833.5 mm, vias 0 -> 13
- net COL9: track 531.5 -> 289.6 mm, vias 0 -> 5
- net COL8: track 505.0 -> 309.0 mm, vias 0 -> 5
- net COL0: track 227.8 -> 323.6 mm, vias 0 -> 1
- net COL2: track 270.0 -> 338.3 mm, vias 0 -> 3
- net COL1: track 232.6 -> 280.8 mm, vias 0 -> 1
- net COL3: track 263.4 -> 310.5 mm, vias 0 -> 5
- net COL4: track 297.4 -> 343.3 mm, vias 0 -> 5
- net COL5: track 347.4 -> 385.9 mm, vias 0 -> 5
- net RKJ-B: track 36.4 -> 0.00 mm
- net LED_MTRX_IN: track 3.77 -> 39.4 mm
- net COL6: track 385.1 -> 420.7 mm, vias 0 -> 5
- net VDD: track 30.6 -> 64.8 mm
- net RKJ-P: track 33.4 -> 0.00 mm
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