File: Overkill/STM32/STM32.kicad_sch (KiCad schematic)
At the start: 464 parts, among them J1 USB_C_Receptacle_USB2.0, Q1 MMUN2133LT1G, Q2 AO3401A, Q3 AO3401A, Q6 2N7002, Q7 2N7002, Q7 AO3401A, Q8 MMUN2233LT1G, SW1 RotaryEncoder_Switch, SW2 RotaryEncoder_Switch, SW3 RKJXT1F42001, SW4 RotaryEncoder_Switch, U1 STM32G474RETx, U10 W25Q32JVSSIQ, U2 TPS2553DBVR, U3 74AHC1G125, U4 AZ1117H-3.3TRE1, U5 TPS2553DBVR-1, U6 LMV321, U7 AZC199-04S, U8 MB85RS64, U9 TPS2553DBVR-1

Commit message: daily
Parts:
- removed BOOT1, RST1: SW_Push, Button_Switch_SMD:SW_SPST_TL3342, symbol Switch:SW_Push
- removed C1, C13: 100nF, Capacitor_SMD:C_0402_1005Metric, symbol Device:C
- removed C14, C15, C16, C17, C18, C19, C20: 100u, Capacitor_Tantalum_SMD:CP_EIA-6032-15_Kemet-U, symbol Device:C_Polarized
- removed R1, R3: 5.1k, Resistor_SMD:R_0402_1005Metric, symbol Device:R
- removed R2: 75k, Resistor_SMD:R_0402_1005Metric, symbol Device:R
- removed R35, R36, R37: 5.1K, Resistor_SMD:R_0402_1005Metric, symbol Device:R_Small
- removed R40: 1k, Resistor_SMD:R_0402_1005Metric, symbol Device:R_Small
- removed U2: TPS2553DBVR, Package_TO_SOT_SMD:SOT-23-6, symbol KeebLib:TPS2553DBVR
- removed U3: 74AHC1G125, Package_TO_SOT_SMD:SOT-23-5, symbol 74xGxx:74AHC1G125
- added C20, C21, C22, C23, C24: 100u, Capacitor_Tantalum_SMD:CP_EIA-6032-15_Kemet-U_Pad2.25x2.35mm_HandSolder, symbol Djinn-rescue:CP-Device
- added D119, D120, D121, D122: D, Keyboard:D_SOD-123F, symbol Device:D
- C1: renamed from C2; footprint Capacitor_SMD:C_0402_1005Metric -> Capacitor_SMD:C_0603_1608Metric_Pad1.08x0.95mm_HandSolder
- C10: renamed from C23; footprint Capacitor_SMD:C_0805_2012Metric -> Capacitor_SMD:C_0603_1608Metric_Pad1.08x0.95mm_HandSolder
- C11: renamed from C24; footprint Capacitor_SMD:C_0805_2012Metric -> Capacitor_SMD:C_0603_1608Metric_Pad1.08x0.95mm_HandSolder
- C12: renamed from C25; footprint Capacitor_SMD:C_0805_2012Metric -> Capacitor_SMD:C_0603_1608Metric_Pad1.08x0.95mm_HandSolder
- C13: renamed from C34; footprint Capacitor_SMD:C_0805_2012Metric -> Capacitor_SMD:C_0603_1608Metric_Pad1.08x0.95mm_HandSolder
- C14: renamed from C35; footprint Capacitor_SMD:C_0805_2012Metric -> Capacitor_SMD:C_0603_1608Metric_Pad1.08x0.95mm_HandSolder
- C15: renamed from C36; footprint Capacitor_SMD:C_0805_2012Metric -> Capacitor_SMD:C_0603_1608Metric_Pad1.08x0.95mm_HandSolder
- C16: renamed from C21; footprint Capacitor_SMD:C_0805_2012Metric -> Capacitor_SMD:C_0603_1608Metric_Pad1.08x0.95mm_HandSolder
- C17: renamed from C7; footprint Capacitor_SMD:C_0805_2012Metric -> Capacitor_SMD:C_0603_1608Metric_Pad1.08x0.95mm_HandSolder
- C18: renamed from C4; footprint reversible-kicad-footprints:CP_6032 -> Capacitor_Tantalum_SMD:CP_EIA-6032-15_Kemet-U_Pad2.25x2.35mm_HandSolder
- C19: renamed from C10; footprint reversible-kicad-footprints:CP_6032 -> Capacitor_Tantalum_SMD:CP_EIA-6032-15_Kemet-U_Pad2.25x2.35mm_HandSolder
- C2: renamed from C3; footprint Capacitor_SMD:C_0402_1005Metric -> Capacitor_SMD:C_0603_1608Metric_Pad1.08x0.95mm_HandSolder
- C26, C27, C29, C30, C31, C32, C33: value 100nF -> 100n; footprint Capacitor_SMD:C_0805_2012Metric -> Capacitor_SMD:C_0603_1608Metric_Pad1.08x0.95mm_HandSolder
- C28: footprint Capacitor_SMD:C_0805_2012Metric -> Capacitor_SMD:C_0603_1608Metric_Pad1.08x0.95mm_HandSolder
- C3: renamed from C8; footprint Capacitor_SMD:C_0805_2012Metric -> Capacitor_SMD:C_0603_1608Metric_Pad1.08x0.95mm_HandSolder
- C4: renamed from C11; footprint Capacitor_SMD:C_0805_2012Metric -> Capacitor_SMD:C_0603_1608Metric_Pad1.08x0.95mm_HandSolder
- C5: renamed from C9; footprint Capacitor_SMD:C_0805_2012Metric -> Capacitor_SMD:C_0603_1608Metric_Pad1.08x0.95mm_HandSolder
- C6: renamed from C5; footprint Capacitor_SMD:C_0805_2012Metric -> Capacitor_SMD:C_0603_1608Metric_Pad1.08x0.95mm_HandSolder
- C7: renamed from C6; footprint Capacitor_SMD:C_0805_2012Metric -> Capacitor_SMD:C_0603_1608Metric_Pad1.08x0.95mm_HandSolder
- C8: renamed from C12; footprint Capacitor_SMD:C_0805_2012Metric -> Capacitor_SMD:C_0603_1608Metric_Pad1.08x0.95mm_HandSolder
- C9: renamed from C22; footprint Capacitor_SMD:C_0805_2012Metric -> Capacitor_SMD:C_0603_1608Metric_Pad1.08x0.95mm_HandSolder
- F1: footprint Fuse:Fuse_1206_3216Metric -> Fuse:Fuse_1206_3216Metric_Pad1.42x1.75mm_HandSolder
- FB1: footprint Capacitor_SMD:C_0805_2012Metric -> Fuse:Fuse_0805_2012Metric_Pad1.15x1.40mm_HandSolder
- J1: footprint Keyboard:HRO-TYPE-C-31-M-12-modded -> Keyboard:HRO-TYPE-C-31-M-12-HandSoldering-NoSBU
- R1: renamed from R39; footprint Resistor_SMD:R_0805_2012Metric -> Resistor_SMD:R_0603_1608Metric_Pad0.98x0.95mm_HandSolder
- R10, R11, R12, R14, R15, R16, R21, R22, R23, R24, R25, R27, R28, R8, R9: value 5.1k -> 9.1k; footprint Resistor_SMD:R_0805_2012Metric -> Resistor_SMD:R_0603_1608Metric_Pad0.98x0.95mm_HandSolder
- R13: renamed from R5; footprint Resistor_SMD:R_0805_2012Metric -> Resistor_SMD:R_0603_1608Metric_Pad0.98x0.95mm_HandSolder
- R17: renamed from R7; footprint Resistor_SMD:R_0805_2012Metric -> Resistor_SMD:R_0603_1608Metric_Pad0.98x0.95mm_HandSolder
- R18, R26, R29, R30: footprint Resistor_SMD:R_0805_2012Metric -> Resistor_SMD:R_0603_1608Metric_Pad0.98x0.95mm_HandSolder
- R2: renamed from R17; footprint Resistor_SMD:R_0805_2012Metric -> Resistor_SMD:R_0603_1608Metric_Pad0.98x0.95mm_HandSolder
- R20: renamed from R4; footprint Resistor_SMD:R_0805_2012Metric -> Resistor_SMD:R_0603_1608Metric_Pad0.98x0.95mm_HandSolder
- R3: renamed from R19; footprint Resistor_SMD:R_0805_2012Metric -> Resistor_SMD:R_0603_1608Metric_Pad0.98x0.95mm_HandSolder
- R31: renamed from R6; footprint Resistor_SMD:R_0805_2012Metric -> Resistor_SMD:R_0603_1608Metric_Pad0.98x0.95mm_HandSolder
- R32: renamed from R13; footprint Resistor_SMD:R_0805_2012Metric -> Resistor_SMD:R_0603_1608Metric_Pad0.98x0.95mm_HandSolder
- R33: renamed from R31; footprint Resistor_SMD:R_0805_2012Metric -> Resistor_SMD:R_0603_1608Metric_Pad0.98x0.95mm_HandSolder
- R34: renamed from R38; footprint Resistor_SMD:R_0805_2012Metric -> Resistor_SMD:R_0603_1608Metric_Pad0.98x0.95mm_HandSolder
- R35: renamed from R42; footprint Resistor_SMD:R_0805_2012Metric -> Resistor_SMD:R_0603_1608Metric_Pad0.98x0.95mm_HandSolder
- R36: renamed from R32; footprint Resistor_SMD:R_0805_2012Metric -> Resistor_SMD:R_0603_1608Metric_Pad0.98x0.95mm_HandSolder
- R37: renamed from R33; footprint Resistor_SMD:R_0805_2012Metric -> Resistor_SMD:R_0603_1608Metric_Pad0.98x0.95mm_HandSolder
- R38: renamed from R34; footprint Resistor_SMD:R_0805_2012Metric -> Resistor_SMD:R_0603_1608Metric_Pad0.98x0.95mm_HandSolder
- R39: renamed from R41; footprint Resistor_SMD:R_0805_2012Metric -> Resistor_SMD:R_0603_1608Metric_Pad0.98x0.95mm_HandSolder
- R4: renamed from R20; footprint Resistor_SMD:R_0805_2012Metric -> Resistor_SMD:R_0603_1608Metric_Pad0.98x0.95mm_HandSolder
- R40: renamed from R43; footprint Resistor_SMD:R_0805_2012Metric -> Resistor_SMD:R_0603_1608Metric_Pad0.98x0.95mm_HandSolder
- U6: renamed from U1; footprint DjinnFootprints:STM32G474RETx -> Package_QFP:LQFP-64_10x10mm_P0.5mm; symbol DjinnSymbols:STM32G474RETx -> MCU_ST_STM32G4:STM32G474RETx
- renumbered D117 to D116, D116 to D117, Q2 to Q1, Q3 to Q2, Q1 to Q3, SW4 to SW3, SW3 to SW4, U7 to U1, U6 to U2, U10 to U3, U8 to U4, U4 to U5, U5 to U7, U9 to U8
Connections:
- net LCD_MOSI/SDA is gone; now on net MOSI: LCD1.4 (Pin_4)
- net LCD_RESET is gone; now on net LCD_RST: LCD1.5 (Pin_5)
- net LCD_SCK/SCL is gone; now on net SCK: LCD1.3 (Pin_3)
- net SK6812_EN is gone; now on net LED_EN: R30.1, U6.24 (PB0), U8.3 (EN)
- net SK6812_NFAULT is gone; now on net LED_NFAULT: R29.2, U6.25 (PB1), U8.4 (~{FAULT})
- net SK6812_PWM is gone; now on net LED_MTRX_IN: R1.2, U6.26 (PB2)
- net SK6812_PWR is gone; now on net LED_PWR: C19.1, R1.1, U8.6 (OUT)
- net +3V3: now also U6.1 (VBAT), U6.16 (VDD), U6.28 (VREF+), U6.29 (VDDA), U6.32 (VDD), U6.48 (VDD), U6.64 (VDD)
- net COL0: no longer SW4.6 (C)
- net COL1: no longer SW4.4 (B)
- net COL2: now also SW2.S1, SW4.7 (COM); no longer MX101.1, MX25.1, MX45.1, MX5.1
- net COL3: now also SW3.S1; no longer MX102.1, MX103.1, MX26.1, MX27.1, MX46.1, MX47.1, MX6.1, MX65.1, MX66.1, MX7.1, MX84.1, MX85.1
- net COL4: now also MX102.1, MX103.1, MX27.1, MX47.1, MX6.1, MX66.1, MX7.1, MX85.1; no longer MX104.1, MX28.1, MX29.1, MX48.1, MX49.1, MX67.1, MX68.1, MX8.1, MX86.1, MX87.1, MX9.1, SW4.9 (D_1)
- net COL5: now also MX104.1, MX28.1, MX29.1, MX48.1, MX49.1, MX67.1, MX68.1, MX8.1, MX86.1, MX87.1, MX9.1; no longer MX10.1, MX105.1, MX11.1, MX30.1, MX31.1, MX50.1, MX51.1, MX69.1, MX70.1, MX88.1, MX89.1, SW4.1 (A)
- net COL6: now also MX10.1, MX105.1, MX11.1, MX30.1, MX31.1, MX50.1, MX51.1, MX69.1, MX70.1, MX88.1, MX89.1; no longer MX106.1, MX12.1, MX13.1, MX32.1, MX33.1, MX52.1, MX53.1, MX71.1, MX72.1, MX90.1, MX91.1, SW4.2 (PUSH)
- net COL7: now also MX106.1, MX12.1, MX13.1, MX32.1, MX33.1, MX52.1, MX53.1, MX71.1, MX72.1, MX90.1, MX91.1; no longer MX107.1, MX14.1, MX15.1, MX34.1, MX35.1, MX54.1, MX55.1, MX73.1, MX74.1, MX92.1, MX93.1
- net COL8: now also MX107.1, MX14.1, MX15.1, MX34.1, MX35.1, MX54.1, MX55.1, MX73.1, MX74.1, MX92.1, MX93.1; no longer MX108.1, MX109.1, MX16.1, MX17.1, MX36.1, MX37.1, MX56.1, MX57.1, MX75.1, MX76.1, MX94.1, MX95.1
- net COL9: now also MX108.1, MX109.1, MX16.1, MX17.1, MX36.1, MX37.1, MX56.1, MX57.1, MX75.1, MX76.1, MX94.1, MX95.1; no longer MX110.1, MX111.1, MX18.1, MX19.1, MX38.1, MX39.1, MX58.1, MX59.1, MX77.1, MX78.1, MX96.1, MX97.1
- net GND: now also U6.15 (VSS), U6.27 (VSSA), U6.31 (VSS), U6.47 (VSS), U6.63 (VSS), C20.2, C21.2, C22.2, C23.2, C24.2
- net LED_PWR: now also C20.1, C21.1, C22.1, C23.1, C24.1
- net ROW0: now also D113.1 (K), D114.2 (A)
- net ROW1: now also D115.1 (K), D23.1 (K); no longer D23.2 (A)
- net ROW2: now also D119.1 (K)
- net ROW3: now also D120.1 (K); no longer D113.1 (K), D114.1 (K)
- net ROW4: now also D121.1 (K)
- net ROW5: now also D122.1 (K); no longer D115.1 (K)
- net ENC1: now reaches D112.1 (K), SW1.S2
- net at MX23.2: now also D23.2 (A); no longer D23.1 (K)
- net ENC3: now reaches SW3.S2
- net ENC3: now also D114.1 (K); no longer D114.2 (A)
- net ENC2: now reaches D113.2 (A), SW2.S2
- net COM renamed RKJ-C
- net RKJ-C: now also SW4.6 (C); no longer SW4.7 (COM)
- net ENC_A: no longer names the net of U6.3 (PC14)
- net ENC_B: no longer names the net of U6.4 (PC15)
- net LED_DAT_5V renamed LED_MTRX_IN
- new net: MX110.1, MX111.1, MX18.1, MX19.1, MX38.1, MX39.1, MX58.1, MX59.1, MX77.1, MX78.1, MX96.1, MX97.1
- new net RKJ-A: D121.2 (A), SW4.1 (A)
- new net RKJ-B: D120.2 (A), SW4.4 (B)
- new net RKJ-D: D119.2 (A), SW4.9 (D_1)
- new net RKJ-P: D122.2 (A), SW4.2 (PUSH)
Other:
- note added: "NOTE: Place each 100uF capacitor at each row branch point"
- note added: "SK6803 Current Limiter"
- note removed: "LED Decoupling"
- note removed: "LED Level Shifter"
- note removed: "LED Power"
- note removed: "NOTE: Capacitor placed at branching points of LED PWR"
- note removed: "NOTE: When USB=500mA, select Rlim = 75k = 74.25k @ 1% = 319mA-401mA range"
- note removed: "RESET & BOOT"
- note removed: "SK6812 Current Limiter"
- note removed: "Takes 3v LED signal and upshifts to 5V"
- moved on the sheet: C10, C11, C12, C13, C14, C15, C16, C19, C26, C27, C28, C29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
