File: Overkill/STM32/STM32.kicad_sch (KiCad schematic)
At the start: 443 parts, among them J1 USB_C_Receptacle_USB2.0, Q1 AO3401A, Q2 AO3401A, Q3 2N7002, Q4 2N7002, Q6 MMUN2133LT1G, Q7 AO3401A, Q8 MMUN2233LT1G, SW1 RotaryEncoder_Switch, SW2 RKJXT1F42001, U1 TPS2553DBVR-1, U2 TPS2553DBVR-1, U3 LMV321, U4 AZC199-04S, U5 AZ1117H-3.3TRE1, U6 STM32G474RETx, U7 MB85RS64, U8 W25Q32JVSSIQ

Commit message: Update PCB traces
Parts:
- removed C10: 100u, reversible-kicad-footprints:CP_6032, symbol Device:CP
- removed C24: 100n, Capacitor_SMD:C_0603_1608Metric_Pad1.08x0.95mm_HandSolder, symbol Device:C
- removed LED112, LED113, LED114, LED115, LED116, LED117, LED118, LED84: MX_SK6803MINI-E, Keyboard:LED_MX_6028R, symbol Keyboard:MX_SK6803MINI-E
- removed LED65: MX_SK6803MINI-E, Keyboard:LED_MX_6028R-ROT, symbol Keyboard:MX_SK6803MINI-E
- removed MX73: MX_SW_HS, Keyboard:SW_MX_HS_1u, symbol PCM_marbastlib-mx:MX_SW_HS_CPG151101S11
- added BT1: Battery_Cell, Battery:BatteryHolder_Keystone_1060_1x2032, symbol Device:Battery_Cell
- added C30, C31, C32, C33: 100u, Capacitor_Tantalum_SMD:CP_EIA-6032-15_Kemet-U_Pad2.25x2.35mm_HandSolder, symbol Djinn-rescue:CP-Device
- added C8: 100n, Capacitor_SMD:C_0603_1608Metric_Pad1.08x0.95mm_HandSolder, symbol Device:C
- added D61: D, Keyboard:D_SOD-123F, symbol Device:D
- added JP1: SolderJumper_2_Open, Jumper:SolderJumper-2_P1.3mm_Open_TrianglePad1.0x1.5mm, symbol Jumper:SolderJumper_2_Open
- added LED64: MX_SK6803MINI-E, Keyboard:LED_MX_6028R, symbol Keyboard:MX_SK6803MINI-E
- added LED82: MX_SK6803MINI-E, Keyboard:LED_MX_6028R-ROT, symbol Keyboard:MX_SK6803MINI-E
- added MX61, MX74: MX_SW_HS, Keyboard:SW_MX_HS_1u, symbol PCM_marbastlib-mx:MX_SW_HS_CPG151101S11
- LED1, LED10, LED11, LED12, LED13, LED14, LED15, LED16, LED17, LED18, LED19, LED2, LED3, LED4, LED40, LED41, LED42, LED43, LED44, LED5, LED6, LED7, LED79, LED8, LED80, LED81, LED85, LED86, LED87, LED88, LED89, LED9, LED90, LED91, LED92, LED93, LED94, LED95: footprint Keyboard:LED_MX_6028R -> Keyboard:LED_MX_6028R-ROT
- LED100, LED101, LED102, LED103, LED104, LED105, LED106, LED107, LED20, LED21, LED22, LED23, LED24, LED60, LED61, LED62, LED63, LED66, LED67, LED68, LED69, LED70, LED71, LED72, LED73, LED74, LED75, LED76, LED77, LED78, LED98, LED99: footprint Keyboard:LED_MX_6028R-ROT -> Keyboard:LED_MX_6028R
- LED65: renamed from LED64; footprint Keyboard:LED_MX_6028R-ROT -> Keyboard:LED_MX_6028R
- LED83: renamed from LED82; footprint Keyboard:LED_MX_6028R -> Keyboard:LED_MX_6028R-ROT
- LED84: renamed from LED83; footprint Keyboard:LED_MX_6028R -> Keyboard:LED_MX_6028R-ROT
- MX41: footprint Keyboard:SW_MX_HS_2u_Vertical -> Keyboard:SW_MX_HS_1u
- R28: renamed from R1; footprint reversible-kicad-footprints:R-0805_2012Metric -> Resistor_SMD:R_0805_2012Metric
- RESET1: footprint reversible-kicad-footprints:PushButton_4.5mm -> Button_Switch_SMD:SW_SPST_SKQG_WithStem
- renumbered C21 to C1, C20 to C11, C29 to C12, C17 to C13, C18 to C14, C9 to C15, C11 to C16, C12 to C17, C7 to C18, C14 to C19, C22 to C2, C13 to C20, C15 to C21, C16 to C22, C8 to C23, C6 to C24, C1 to C25, C2 to C26, C3 to C27, C4 to C28, C5 to C29, C23 to C3, C25 to C4, C26 to C5, C27 to C6, C28 to C7, C19 to C9, D99 to D100, D100 to D101, D101 to D102, D102 to D103, D103 to D104, D104 to D105, D105 to D106, D106 to D107, D107 to D108, D108 to D109, D109 to D110, D110 to D111, D117 to D112, D111 to D113, D112 to D114, D113 to D115, D114 to D116, D115 to D117, D116 to D118, D118 to D119, D119 to D120, D61 to D62, D62 to D63, D63 to D64, D64 to D65, D65 to D66, D66 to D67, D67 to D68, D68 to D69, D69 to D70, D70 to D71, D71 to D72, D72 to D73, D73 to D74, D74 to D75, D75 to D76, D76 to D77, D77 to D78, D78 to D79, D79 to D80, D80 to D81, D81 to D82, D82 to D83, D83 to D84, D84 to D85, D85 to D86, D86 to D87, D87 to D88, D88 to D89, D89 to D90, D90 to D91, D91 to D92, D92 to D93, D93 to D94, D94 to D95, D95 to D96, D96 to D97, D97 to D98, D98 to D99, LED45 to LED25, LED46 to LED26, LED47 to LED27, LED48 to LED28, LED49 to LED29, LED50 to LED30, LED51 to LED31, LED52 to LED32, LED53 to LED33, LED54 to LED34, LED55 to LED35, LED56 to LED36, LED57 to LED37, LED58 to LED38, LED59 to LED39, LED25 to LED45, LED26 to LED46, LED27 to LED47, LED28 to LED48, LED29 to LED49, LED30 to LED50, LED31 to LED51, LED32 to LED52, LED33 to LED53, LED34 to LED54, LED35 to LED55, LED36 to LED56, LED37 to LED57, LED38 to LED58, LED39 to LED59, MX99 to MX100, MX100 to MX101, MX101 to MX102, MX102 to MX103, MX103 to MX104, MX104 to MX105, MX105 to MX106, MX106 to MX107, MX107 to MX108, MX108 to MX109, MX109 to MX110, MX110 to MX111, MX61 to MX62, MX62 to MX63, MX63 to MX64, MX64 to MX65, MX65 to MX66, MX66 to MX67, MX67 to MX68, MX68 to MX69, MX69 to MX70, MX70 to MX71, MX71 to MX72, MX72 to MX73, MX74 to MX75, MX75 to MX76, MX76 to MX77, MX77 to MX78, MX78 to MX79, MX79 to MX80, MX80 to MX81, MX81 to MX82, MX82 to MX83, MX83 to MX84, MX84 to MX85, MX85 to MX86, MX86 to MX87, MX87 to MX88, MX88 to MX89, MX89 to MX90, MX90 to MX91, MX91 to MX92, MX92 to MX93, MX93 to MX94, MX94 to MX95, MX95 to MX96, MX96 to MX97, MX97 to MX98, MX98 to MX99, Q6 to Q3, Q3 to Q4, Q4 to Q6, R26 to R1, R20 to R10, R22 to R11, R19 to R12, R24 to R13, R21 to R14, R25 to R16, R2 to R18, R3 to R19, R27 to R2, R5 to R20, R11 to R21, R14 to R22, R6 to R23, R7 to R24, R8 to R25, R12 to R26, R16 to R27, R28 to R3, R10 to R5, R13 to R6, R18 to R7, R23 to R8, SW2 to SW1, SW1 to SW2, U4 to U1, U8 to U2, U7 to U4, U2 to U7, U1 to U8
Connections:
- net +3V3: now also JP1.1 (A); no longer Q7.2 (S), U6.1 (VBAT)
- net +5V: no longer C16.2, U5.3 (VI)
- net BOARD_NFAULT: no longer U6.41 (PC9)
- net COL0: now also U6.30 (PB10), MX61.1; no longer U6.8 (PC0)
- net COL1: now also MX100.1, U6.26 (PB2); no longer U6.9 (PC1)
- net COL2: now also MX101.1, MX25.1, MX45.1, MX5.1, MX65.1, MX84.1, U6.25 (PB1); no longer MX100.1, SW1.7 (COM), U6.10 (PC2)
- net COL3: now also MX103.1, MX27.1, MX47.1, MX67.1, MX7.1; no longer MX101.1, MX25.1, MX45.1, MX5.1, MX65.1, MX84.1, U6.11 (PC3)
- net COL4: now also MX29.1, MX49.1, MX69.1, MX9.1; no longer MX103.1, MX27.1, MX47.1, MX67.1, MX7.1, U6.38 (PC6)
- net COL5: now also MX11.1, MX31.1, MX51.1, MX71.1; no longer MX29.1, MX49.1, MX69.1, MX9.1, U6.39 (PC7)
- net COL6: now also MX13.1, MX33.1, MX53.1, MX73.1; no longer MX11.1, MX31.1, MX51.1, MX71.1, U6.40 (PC8)
- net COL7: now also MX15.1, MX35.1, MX55.1, MX75.1, MX74.1; no longer MX13.1, MX33.1, MX53.1, MX73.1, U6.2 (PC13)
- net COL8: now also MX108.1, MX109.1, MX17.1, MX37.1, MX57.1, MX95.1; no longer MX15.1, MX35.1, MX55.1, MX75.1, U6.3 (PC14)
- net COL9: now also MX110.1, MX111.1, MX18.1, MX19.1, MX38.1, MX39.1, MX58.1, MX59.1, MX77.1, MX78.1, MX96.1, MX97.1; no longer U6.4 (PC15)
- net CURR_1500mA_OK: now also U6.39 (PC7); no longer U6.23 (PC5)
- net CURR_3000mA_OK: now also U6.38 (PC6); no longer U6.22 (PC4)
- net ENC1_A: now also U6.4 (PC15); no longer U6.36 (PB14)
- net ENC1_B: now also U6.3 (PC14); no longer U6.37 (PB15)
- net ENC2_A: now also U6.35 (PB13); no longer U6.33 (PB11)
- net ENC2_B: now also U6.36 (PB14); no longer U6.35 (PB13)
- net GND: now also LED25.4 (VSS), LED26.4 (VSS), LED27.4 (VSS), LED28.4 (VSS), LED29.4 (VSS), LED30.4 (VSS), LED31.4 (VSS), LED32.4 (VSS), LED33.4 (VSS), LED34.4 (VSS), LED35.4 (VSS), LED36.4 (VSS), LED37.4 (VSS), LED38.4 (VSS), LED39.4 (VSS), LED40.4 (VSS), LED41.4 (VSS), LED42.4 (VSS), LED43.4 (VSS), LED44.4 (VSS), LED60.4 (VSS), LED61.4 (VSS), LED62.4 (VSS), LED63.4 (VSS), LED65.4 (VSS), LED66.4 (VSS), LED67.4 (VSS), LED68.4 (VSS), LED69.4 (VSS), LED70.4 (VSS), LED71.4 (VSS), LED72.4 (VSS), LED73.4 (VSS), LED74.4 (VSS), LED75.4 (VSS), LED76.4 (VSS), LED77.4 (VSS), LED78.4 (VSS), LED79.4 (VSS), LED80.4 (VSS), LED81.4 (VSS), LED83.4 (VSS), LED84.4 (VSS), LED85.4 (VSS), LED86.4 (VSS), LED87.4 (VSS), LED88.4 (VSS), LED89.4 (VSS), LED90.4 (VSS), LED91.4 (VSS), LED92.4 (VSS), LED93.4 (VSS), LED94.4 (VSS), LED95.4 (VSS), BT1.2 (-), C30.2, C31.2, C32.2, C33.2, C8.2, LED64.4 (VSS), LED82.4 (VSS); no longer LED25.1 (VDD), LED26.1 (VDD), LED27.1 (VDD), LED28.1 (VDD), LED29.1 (VDD), LED30.1 (VDD), LED31.1 (VDD), LED32.1 (VDD), LED33.1 (VDD), LED34.1 (VDD), LED35.1 (VDD), LED36.1 (VDD), LED37.1 (VDD), LED38.1 (VDD), LED39.1 (VDD), LED40.1 (VDD), LED41.1 (VDD), LED42.1 (VDD), LED43.1 (VDD), LED44.1 (VDD), LED60.1 (VDD), LED61.1 (VDD), LED62.1 (VDD), LED63.1 (VDD), LED65.1 (VDD), LED66.1 (VDD), LED67.1 (VDD), LED68.1 (VDD), LED69.1 (VDD), LED70.1 (VDD), LED71.1 (VDD), LED72.1 (VDD), LED73.1 (VDD), LED74.1 (VDD), LED75.1 (VDD), LED76.1 (VDD), LED77.1 (VDD), LED78.1 (VDD), LED79.1 (VDD), LED80.1 (VDD), LED81.1 (VDD), LED83.1 (VDD), LED84.1 (VDD), LED85.1 (VDD), LED86.1 (VDD), LED87.1 (VDD), LED88.1 (VDD), LED89.1 (VDD), LED90.1 (VDD), LED91.1 (VDD), LED92.1 (VDD), LED93.1 (VDD), LED94.1 (VDD), LED95.1 (VDD)
- net LCD_BL_PWM: now also U6.10 (PC2); no longer U6.21 (PA7)
- net LCD_CS: now also U6.9 (PC1); no longer U6.55 (PD2)
- net LCD_DC: now also U6.8 (PC0); no longer U6.51 (PA15)
- net LCD_EN: now also U6.62 (PB9); no longer U6.20 (PA6)
- net LCD_RST: now also U6.2 (PC13); no longer U6.56 (PB3)
- net LED_EN: now also U6.41 (PC9); no longer U6.24 (PB0)
- net LED_MTRX_IN: now also LED4.3 (DIN), R28.2, U6.37 (PB15); no longer LED1.3 (DIN)
- net LED_NFAULT: now also U6.40 (PC8); no longer U6.25 (PB1)
- net LED_PWR: now also LED25.1 (VDD), LED26.1 (VDD), LED27.1 (VDD), LED28.1 (VDD), LED29.1 (VDD), LED30.1 (VDD), LED31.1 (VDD), LED32.1 (VDD), LED33.1 (VDD), LED34.1 (VDD), LED35.1 (VDD), LED36.1 (VDD), LED37.1 (VDD), LED38.1 (VDD), LED39.1 (VDD), LED40.1 (VDD), LED41.1 (VDD), LED42.1 (VDD), LED43.1 (VDD), LED44.1 (VDD), LED60.1 (VDD), LED61.1 (VDD), LED62.1 (VDD), LED63.1 (VDD), LED65.1 (VDD), LED66.1 (VDD), LED67.1 (VDD), LED68.1 (VDD), LED69.1 (VDD), LED70.1 (VDD), LED71.1 (VDD), LED72.1 (VDD), LED73.1 (VDD), LED74.1 (VDD), LED75.1 (VDD), LED76.1 (VDD), LED77.1 (VDD), LED78.1 (VDD), LED79.1 (VDD), LED80.1 (VDD), LED81.1 (VDD), LED83.1 (VDD), LED84.1 (VDD), LED85.1 (VDD), LED86.1 (VDD), LED87.1 (VDD), LED88.1 (VDD), LED89.1 (VDD), LED90.1 (VDD), LED91.1 (VDD), LED92.1 (VDD), LED93.1 (VDD), LED94.1 (VDD), LED95.1 (VDD), C30.1, C31.1, C32.1, C33.1, LED64.1 (VDD), LED82.1 (VDD); no longer LED25.4 (VSS), LED26.4 (VSS), LED27.4 (VSS), LED28.4 (VSS), LED29.4 (VSS), LED30.4 (VSS), LED31.4 (VSS), LED32.4 (VSS), LED33.4 (VSS), LED34.4 (VSS), LED35.4 (VSS), LED36.4 (VSS), LED37.4 (VSS), LED38.4 (VSS), LED39.4 (VSS), LED40.4 (VSS), LED41.4 (VSS), LED42.4 (VSS), LED43.4 (VSS), LED44.4 (VSS), LED60.4 (VSS), LED61.4 (VSS), LED62.4 (VSS), LED63.4 (VSS), LED65.4 (VSS), LED66.4 (VSS), LED67.4 (VSS), LED68.4 (VSS), LED69.4 (VSS), LED70.4 (VSS), LED71.4 (VSS), LED72.4 (VSS), LED73.4 (VSS), LED74.4 (VSS), LED75.4 (VSS), LED76.4 (VSS), LED77.4 (VSS), LED78.4 (VSS), LED79.4 (VSS), LED80.4 (VSS), LED81.4 (VSS), LED83.4 (VSS), LED84.4 (VSS), LED85.4 (VSS), LED86.4 (VSS), LED87.4 (VSS), LED88.4 (VSS), LED89.4 (VSS), LED90.4 (VSS), LED91.4 (VSS), LED92.4 (VSS), LED93.4 (VSS), LED94.4 (VSS), LED95.4 (VSS)
- net RKJ-B: now also D114.2 (A); no longer D115.2 (A)
- net RKJ-C: now also D113.2 (A); no longer D114.2 (A)
- net RKJ-D: now also D117.2 (A); no longer D113.2 (A)
- net RKJ-P: now also D115.2 (A); no longer D117.2 (A)
- net ROW0: now also D19.1 (K), U6.33 (PB11); no longer U6.12 (PA0)
- net ROW1: now also U6.24 (PB0); no longer U6.13 (PA1)
- net ROW2: now also U6.23 (PC5); no longer U6.14 (PA2)
- net ROW3: now also D65.1 (K), D66.2 (A), D67.1 (K), D68.2 (A), D69.1 (K), D70.2 (A), D71.1 (K), D72.2 (A), D73.1 (K), D74.2 (A), D75.1 (K), D76.2 (A), U6.22 (PC4), D61.1 (K); no longer D65.2 (A), D66.1 (K), D67.2 (A), D68.1 (K), D69.2 (A), D70.1 (K), D71.2 (A), D72.1 (K), D73.2 (A), D74.1 (K), D75.2 (A), D76.1 (K), U6.17 (PA3)
- net ROW4: now also D84.1 (K), U6.21 (PA7); no longer D80.1 (K), D84.2 (A), U6.18 (PA4)
- net ROW5: now also D104.1 (K), D105.1 (K), D106.1 (K), D107.1 (K), D80.1 (K), D80.2 (A), MX80.2, U6.20 (PA6); no longer D104.2 (A), D105.2 (A), D106.2 (A), D107.2 (A), U6.19 (PA5)
- net VDD: now also C16.2, Q7.2 (S), U5.3 (VI)
- net at LED43.3 (DIN): now also LED44.2 (DOUT); no longer LED42.2 (DOUT)
- net at LED42.3 (DIN): now also LED43.2 (DOUT); no longer LED41.2 (DOUT)
- net at LED97.2 (DOUT): now also LED95.3 (DIN); no longer LED98.2 (DOUT)
- net at LED96.3 (DIN): now also LED111.2 (DOUT); no longer LED97.3 (DIN)
- net at LED59.3 (DIN): now also LED78.2 (DOUT); no longer LED19.2 (DOUT)
- net at LED19.3 (DIN): now also LED39.2 (DOUT); no longer LED18.2 (DOUT)
- net at LED38.2 (DOUT): now also LED39.3 (DIN)
- net at LED38.3 (DIN): now also LED37.2 (DOUT)
- net at MX76.2: now also D76.1 (K); no longer D76.2 (A)
- net at LED65.3 (DIN): now also LED84.2 (DOUT)
- net at LED66.2 (DOUT): now also LED67.3 (DIN)
- net at LED94.2 (DOUT): now also LED93.3 (DIN); no longer LED95.3 (DIN)
- net at LED93.2 (DOUT): now also LED92.3 (DIN); no longer LED94.3 (DIN)
- net at LED6.3 (DIN): now also LED7.2 (DOUT); no longer LED5.2 (DOUT)
- net at LED4.2 (DOUT): now also LED3.3 (DIN); no longer LED5.3 (DIN)
- net at MX107.2: now also D107.2 (A); no longer D107.1 (K)
- net at MX104.2: now also D104.2 (A); no longer D104.1 (K)
- net at LED105.3 (DIN): now also LED104.2 (DOUT); no longer LED106.2 (DOUT)
- net at LED106.3 (DIN): now also LED105.2 (DOUT); no longer LED107.2 (DOUT)
- net at LED74.2 (DOUT): now also LED75.3 (DIN); no longer LED73.3 (DIN)
- net at LED75.2 (DOUT): now also LED76.3 (DIN); no longer LED74.3 (DIN)
- net at LED6.2 (DOUT): now also LED5.3 (DIN); no longer LED7.3 (DIN)
- net at LED88.2 (DOUT): now also LED87.3 (DIN); no longer LED89.3 (DIN)
- net at LED87.2 (DOUT): now also LED86.3 (DIN); no longer LED88.3 (DIN)
- net at MX72.2: now also D72.1 (K); no longer D72.2 (A)
- net at LED72.3 (DIN): now also LED71.2 (DOUT); no longer LED73.2 (DOUT)
- net at MX65.2: now also D65.2 (A); no longer D65.1 (K)
- net at LED99.3 (DIN): now also LED98.2 (DOUT); no longer LED100.2 (DOUT)
- net at LED101.2 (DOUT): now also LED102.3 (DIN); no longer LED100.3 (DIN)
- net at LED9.3 (DIN): now also LED10.2 (DOUT); no longer LED8.2 (DOUT)
- net at LED8.3 (DIN): now also LED9.2 (DOUT); no longer LED7.2 (DOUT)
- net at LED90.3 (DIN): now also LED91.2 (DOUT); no longer LED89.2 (DOUT)
- net at LED95.2 (DOUT): now also LED94.3 (DIN); no longer LED107.3 (DIN)
- net at LED66.3 (DIN): now also LED65.2 (DOUT); no longer LED67.2 (DOUT)
- net at LED21.2 (DOUT): now also LED22.3 (DIN); no longer LED20.3 (DIN)
- net at LED21.3 (DIN): now also LED20.2 (DOUT); no longer LED22.2 (DOUT)
- net at LED77.3 (DIN): now also LED76.2 (DOUT); no longer LED78.2 (DOUT)
- net at LED78.3 (DIN): now also LED77.2 (DOUT); no longer LED39.2 (DOUT)
- net at MX19.2: now also D19.2 (A); no longer D19.1 (K)
- net at LED103.2 (DOUT): now also LED104.3 (DIN); no longer LED102.3 (DIN)
- net at LED103.3 (DIN): now also LED102.2 (DOUT); no longer LED104.2 (DOUT)
- net at MX71.2: now also D71.2 (A); no longer D71.1 (K)
- net at MX66.2: now also D66.1 (K); no longer D66.2 (A)
- net at MX69.2: now also D69.2 (A); no longer D69.1 (K)
- net at MX84.2: now also D84.2 (A); no longer D84.1 (K)
- net at LED25.3 (DIN): now also LED45.2 (DOUT); no longer LED44.2 (DOUT)
- net at LED44.3 (DIN): now also LED24.2 (DOUT); no longer LED43.2 (DOUT)
- net at LED98.3 (DIN): now also LED79.2 (DOUT); no longer LED99.2 (DOUT)
- net at LED40.2 (DOUT): now also LED60.3 (DIN); no longer LED41.3 (DIN)
- net at LED40.3 (DIN): now also LED41.2 (DOUT); no longer LED20.2 (DOUT)
- net at LED71.3 (DIN): now also LED70.2 (DOUT); no longer LED72.2 (DOUT)
- net at LED85.2 (DOUT): now also LED84.3 (DIN)
- net at LED85.3 (DIN): now also LED86.2 (DOUT)
- net at LED92.2 (DOUT): now also LED91.3 (DIN); no longer LED93.3 (DIN)
- net at LED3.2 (DOUT): now also LED2.3 (DIN); no longer LED4.3 (DIN)
- net at LED11.2 (DOUT): now also LED10.3 (DIN); no longer LED12.3 (DIN)
- net at LED11.3 (DIN): now also LED12.2 (DOUT); no longer LED10.2 (DOUT)
- net at LED17.2 (DOUT): now also LED16.3 (DIN); no longer LED18.3 (DIN)
- net at LED15.2 (DOUT): now also LED14.3 (DIN); no longer LED16.3 (DIN)
- net at LED15.3 (DIN): now also LED16.2 (DOUT); no longer LED14.2 (DOUT)
- net at LED2.2 (DOUT): now also LED1.3 (DIN); no longer LED3.3 (DIN)
- net at LED1.2 (DOUT): now also LED20.3 (DIN); no longer LED2.3 (DIN)
- net at LED80.2 (DOUT): now also LED79.3 (DIN); no longer LED81.3 (DIN)
- net at LED80.3 (DIN): now also LED81.2 (DOUT); no longer LED79.2 (DOUT)
- net at MX105.2: now also D105.2 (A); no longer D105.1 (K)
- net at MX106.2: now also D106.2 (A); no longer D106.1 (K)
- net at LED36.2 (DOUT): now also LED37.3 (DIN)
- net at LED36.3 (DIN): now also LED35.2 (DOUT)
- net at MX68.2: now also D68.1 (K); no longer D68.2 (A)
- net at LED69.3 (DIN): now also LED68.2 (DOUT); no longer LED70.2 (DOUT)
- net at LED70.3 (DIN): now also LED69.2 (DOUT); no longer LED71.2 (DOUT)
- net at LED83.2 (DOUT): now also LED82.3 (DIN); no longer LED84.3 (DIN)
- net at LED63.3 (DIN): now also LED62.2 (DOUT); no longer LED65.2 (DOUT)
- net at LED83.3 (DIN): now also LED64.2 (DOUT); no longer LED81.2 (DOUT)
- net at LED23.2 (DOUT): now also LED24.3 (DIN); no longer LED22.3 (DIN)
- net at MX75.2: now also D75.2 (A); no longer D75.1 (K)
- net at LED17.3 (DIN): now also LED18.2 (DOUT); no longer LED16.2 (DOUT)
- net at LED96.2 (DOUT): now also LED97.3 (DIN)
- net at LED13.3 (DIN): now also LED14.2 (DOUT); no longer LED12.2 (DOUT)
- net at LED27.2 (DOUT): now also LED28.3 (DIN)
- net at LED27.3 (DIN): now also LED26.2 (DOUT)
- net at LED61.3 (DIN): now also LED60.2 (DOUT); no longer LED62.2 (DOUT)
- net at LED62.3 (DIN): now also LED61.2 (DOUT); no longer LED63.2 (DOUT)
- net at MX73.2: now also D73.2 (A); no longer D73.1 (K)
- net at LED28.2 (DOUT): now also LED29.3 (DIN)
- net at LED101.3 (DIN): now also LED100.2 (DOUT); no longer LED102.2 (DOUT)
- net at LED23.3 (DIN): now also LED22.2 (DOUT); no longer LED24.2 (DOUT)
- net at LED31.2 (DOUT): now also LED32.3 (DIN)
- net at LED31.3 (DIN): now also LED30.2 (DOUT)
- net at LED34.2 (DOUT): now also LED35.3 (DIN)
- net at LED34.3 (DIN): now also LED33.2 (DOUT)
- net at MX67.2: now also D67.2 (A); no longer D67.1 (K)
- net at LED29.2 (DOUT): now also LED30.3 (DIN)
- net at LED68.3 (DIN): now also LED67.2 (DOUT); no longer LED69.2 (DOUT)
- net at LED90.2 (DOUT): now also LED89.3 (DIN)
- net at MX70.2: now also D70.1 (K); no longer D70.2 (A)
- net at LED33.3 (DIN): now also LED32.2 (DOUT)
- net at LED13.2 (DOUT): now also LED12.3 (DIN); no longer LED14.3 (DIN)
- removed net LED_PWM: LED108.3 (DIN), R28.2, U6.26 (PB2)
- new net: LED88.3 (DIN), LED89.2 (DOUT)
- new net: D74.1 (K), MX74.2
- new net: D61.2 (A), MX61.2
- new net: LED72.2 (DOUT), LED73.3 (DIN)
- new net: LED18.3 (DIN), LED19.2 (DOUT)
- new net: LED81.3 (DIN), LED82.2 (DOUT)
- new net: LED63.2 (DOUT), LED64.3 (DIN)
- new net: LED41.3 (DIN), LED42.2 (DOUT)
- new net: LED106.2 (DOUT), LED107.3 (DIN)
- new net: LED73.2 (DOUT), LED74.3 (DIN)
- new net: LED107.2 (DOUT), LED108.3 (DIN)
- new net: LED100.3 (DIN), LED99.2 (DOUT)
- new net: LED7.3 (DIN), LED8.2 (DOUT)
- new net COL10: SW1.7 (COM)
- new net VBAT: BT1.1 (+), C8.1, JP1.2 (B), U6.1 (VBAT)
Other:
- note removed: "RGB Underglow"
- moved on the sheet: C1, C2, C25, C26, C27, C28, C29, C3, C4, C5, C6, C7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

Commit message: Rotate mcu & wire nets
Connections:
- net BOARD_NFAULT: now also U6.30 (PB10)
- net COL0: no longer U6.30 (PB10)
- net COL1: no longer U6.26 (PB2)
- net COL2: now also U6.19 (PA5); no longer U6.25 (PB1)
- net COL3: now also U6.41 (PC9)
- net COL4: now also U6.40 (PC8)
- net COL5: now also U6.39 (PC7)
- net COL6: now also U6.38 (PC6)
- net COL7: now also U6.37 (PB15)
- net COL8: now also U6.36 (PB14)
- net COL9: now also U6.35 (PB13)
- net CURR_1500mA_OK: now also U6.25 (PB1); no longer U6.39 (PC7)
- net CURR_3000mA_OK: now also U6.24 (PB0); no longer U6.38 (PC6)
- net ENC1_A: no longer U6.4 (PC15)
- net ENC1_B: no longer U6.3 (PC14)
- net ENC2_A: now also U6.21 (PA7); no longer U6.35 (PB13)
- net ENC2_B: now also U6.22 (PC4); no longer U6.36 (PB14)
- net LCD_BL_PWM: now also U6.2 (PC13); no longer U6.10 (PC2)
- net LCD_CS: now also U6.62 (PB9); no longer U6.9 (PC1)
- net LCD_DC: now also U6.56 (PB3); no longer U6.8 (PC0)
- net LCD_EN: now also U6.51 (PA15); no longer U6.62 (PB9)
- net LCD_RST: now also U6.55 (PD2); no longer U6.2 (PC13)
- net LED_EN: now also U6.33 (PB11); no longer U6.41 (PC9)
- net LED_MTRX_IN: now also U6.23 (PC5); no longer U6.37 (PB15)
- net LED_NFAULT: now also U6.26 (PB2); no longer U6.40 (PC8)
- net ROW0: now also U6.20 (PA6); no longer U6.33 (PB11)
- net ROW1: no longer U6.24 (PB0)
- net ROW2: no longer U6.23 (PC5)
- net ROW3: no longer U6.22 (PC4)
- net ROW4: no longer U6.21 (PA7)
- net ROW5: no longer U6.20 (PA6)

Commit message: update
Parts:
- removed H1, H10, H2, H3, H4, H5, H6, H7, H8, H9: MountingHole, MountingHole:MountingHole_2.2mm_M2_DIN965_Pad, symbol Mechanical:MountingHole
- removed TP7: SWD, Keyboard:TestPoint, symbol Connector:TestPoint
- D1, D10, D100, D101, D102, D103, D104, D105, D106, D107, D108, D109, D11, D110, D111, D112, D113, D114, D115, D116, D117, D118, D119, D12, D120, D13, D14, D15, D16, D17, D18, D19, D2, D20, D21, D22, D23, D24, D25, D26, D27, D28, D29, D3, D30, D31, D32, D33, D34, D35, D36, D37, D38, D39, D4, D40, D41, D42, D43, D44, D45, D46, D47, D48, D49, D5, D50, D51, D52, D53, D54, D55, D56, D57, D58, D59, D6, D60, D61, D62, D63, D64, D65, D66, D67, D68, D69, D7, D70, D71, D72, D73, D74, D75, D76, D77, D78, D79, D8, D80, D81, D82, D83, D84, D85, D86, D87, D88, D89, D9, D90, D91, D92, D93, D94, D95, D96, D97, D98, D99: footprint Keyboard:D_SOD-123F -> Keyboard:D_SOD-123
- TP5: value RST -> NRST
- TP6: value SWC -> VBAT
Connections:
- net +5V is gone; now on net VDD: TP2.1
- net RESET is gone; now on net NRST: TP5.1
- net SWC is gone; now on net VBAT: TP6.1
- net COL0: now also U6.20 (PA6)
- net COL1: now also U6.19 (PA5)
- net COL10: now also U6.9 (PC1)
- net COL2: now also U6.17 (PA3); no longer U6.19 (PA5)
- net ENC1: now also D112.1 (K); no longer D112.2 (A)
- net ENC1_A: now also U6.55 (PD2)
- net ENC1_B: now also U6.56 (PB3)
- net GND: now also J1.S1 (SHIELD)
- net LCD_BL_PWM: now also U6.8 (PC0); no longer U6.2 (PC13)
- net LCD_CS: now also U6.4 (PC15); no longer U6.62 (PB9)
- net LCD_DC: now also U6.3 (PC14); no longer U6.56 (PB3)
- net LCD_RST: now also U6.2 (PC13); no longer U6.55 (PD2)
- net ROW0: now also D112.2 (A), U6.18 (PA4); no longer D112.1 (K), U6.20 (PA6)
- net ROW1: now also U6.14 (PA2)
- net ROW2: now also U6.13 (PA1)
- net ROW3: now also U6.12 (PA0)
- net ROW4: now also U6.11 (PC3)
- net ROW5: now also U6.10 (PC2); no longer D80.2 (A), MX80.2
- net SHIELD: no longer J1.S1 (SHIELD)
- net VBUS: no longer TP1.1
- net V_USB: now also TP1.1
- new net: D80.2 (A), MX80.2
Other:
- note removed: "M2 Mounting Holes"
- moved on the sheet: C15, C16, C17, C18, C19, C20, C21, C22, C23, C24, D112, D113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

Commit message: update
Parts:
- removed C33: 100u, Capacitor_Tantalum_SMD:CP_EIA-6032-15_Kemet-U_Pad2.25x2.35mm_HandSolder, symbol Djinn-rescue:CP-Device
- removed U5: AZ1117H-3.3TRE1, Package_TO_SOT_SMD:SOT-23-3, symbol Regulator_Linear:XC6206PxxxMR
- added D65, D66: D, Keyboard:D_SOD-123, symbol Device:D
- added LED67, LED68: MX_SK6803MINI-E, Keyboard:LED_MX_6028R, symbol Keyboard:MX_SK6803MINI-E
- added MX65, MX66: MX_SW_HS, Keyboard:SW_MX_HS_1u, symbol PCM_marbastlib-mx:MX_SW_HS_CPG151101S11
- added U5: AP2127K-3.3, Package_TO_SOT_SMD:SOT-23-5_HandSoldering, symbol Regulator_Linear:AP2127K-3.3
- C16, C17: value 1u -> 4.7u
- renumbered D98 to D100, D99 to D101, D100 to D102, D101 to D103, D102 to D104, D103 to D105, D104 to D106, D105 to D107, D106 to D108, D107 to D109, D108 to D110, D109 to D111, D110 to D112, D111 to D113, D113 to D114, D114 to D115, D115 to D116, D116 to D117, D117 to D118, D112 to D119, D119 to D120, D120 to D121, D118 to D122, D65 to D67, D66 to D68, D67 to D69, D68 to D70, D69 to D71, D70 to D72, D71 to D73, D72 to D74, D73 to D75, D74 to D76, D75 to D77, D76 to D78, D77 to D79, D78 to D80, D79 to D81, D80 to D82, D81 to D83, D82 to D84, D83 to D85, D84 to D86, D85 to D87, D86 to D88, D87 to D89, D88 to D90, D89 to D91, D90 to D92, D91 to D93, D92 to D94, D93 to D95, D94 to D96, D95 to D97, D97 to D98, D96 to D99, LED98 to LED100, LED99 to LED101, LED100 to LED102, LED101 to LED103, LED102 to LED104, LED103 to LED105, LED104 to LED106, LED105 to LED107, LED106 to LED108, LED107 to LED109, LED108 to LED110, LED109 to LED111, LED110 to LED112, LED111 to LED113, LED77 to LED65, LED78 to LED66, LED65 to LED69, LED66 to LED70, LED67 to LED71, LED68 to LED72, LED69 to LED73, LED70 to LED74, LED71 to LED75, LED72 to LED76, LED73 to LED77, LED74 to LED78, LED75 to LED79, LED76 to LED80, LED79 to LED81, LED80 to LED82, LED81 to LED83, LED82 to LED84, LED83 to LED85, LED84 to LED86, LED85 to LED87, LED86 to LED88, LED87 to LED89, LED88 to LED90, LED89 to LED91, LED90 to LED92, LED91 to LED93, LED92 to LED94, LED93 to LED95, LED94 to LED96, LED95 to LED97, LED96 to LED98, LED97 to LED99, MX98 to MX100, MX99 to MX101, MX100 to MX102, MX101 to MX103, MX102 to MX104, MX103 to MX105, MX104 to MX106, MX105 to MX107, MX106 to MX108, MX107 to MX109, MX108 to MX110, MX109 to MX111, MX110 to MX112, MX111 to MX113, MX65 to MX67, MX66 to MX68, MX67 to MX69, MX68 to MX70, MX69 to MX71, MX70 to MX72, MX71 to MX73, MX72 to MX74, MX73 to MX75, MX74 to MX76, MX75 to MX77, MX76 to MX78, MX77 to MX79, MX78 to MX80, MX79 to MX81, MX80 to MX82, MX81 to MX83, MX82 to MX84, MX83 to MX85, MX84 to MX86, MX85 to MX87, MX86 to MX88, MX87 to MX89, MX88 to MX90, MX89 to MX91, MX90 to MX92, MX91 to MX93, MX92 to MX94, MX93 to MX95, MX94 to MX96, MX95 to MX97, MX97 to MX98, MX96 to MX99
Connections:
- net +3V3: now also U5.5 (VOUT)
- net COL0: now also U6.19 (PA5); no longer U6.20 (PA6)
- net COL1: now also U6.18 (PA4); no longer U6.19 (PA5)
- net COL3: now also U6.40 (PC8); no longer U6.41 (PC9)
- net COL4: now also U6.39 (PC7); no longer U6.40 (PC8)
- net COL5: now also U6.38 (PC6); no longer U6.39 (PC7)
- net COL6: now also U6.37 (PB15); no longer U6.38 (PC6)
- net COL7: now also U6.36 (PB14); no longer U6.37 (PB15)
- net COL8: now also U6.35 (PB13); no longer U6.36 (PB14)
- net COL9: now also U6.34 (PB12); no longer U6.35 (PB13)
- net ENC2_A: now also U6.20 (PA6); no longer U6.21 (PA7)
- net ENC2_B: now also U6.21 (PA7); no longer U6.22 (PC4)
- net GND: now also LED67.4 (VSS), LED68.4 (VSS), U5.2 (GND)
- net LED_PWR: now also LED67.1 (VDD), LED68.1 (VDD)
- net PLUG_DETECT: no longer U6.34 (PB12)
- net RKJ-A: now also D118.2 (A); no longer D117.2 (A)
- net RKJ-B: now also D116.2 (A); no longer D115.2 (A)
- net RKJ-D: now also D115.2 (A); no longer D118.2 (A)
- net RKJ-P: now also D117.2 (A); no longer D116.2 (A)
- net ROW0: now also U6.22 (PC4); no longer U6.18 (PA4)
- net ROW2: now also D116.1 (K); no longer D115.1 (K)
- net ROW3: now also D115.1 (K), D65.2 (A), D66.2 (A); no longer D116.1 (K)
- net VDD: now also U5.1 (VIN), U5.3 (EN)
- net at LED66.2 (DOUT): now also LED67.3 (DIN); no longer LED59.3 (DIN)
- net at LED86.2 (DOUT): now also LED65.3 (DIN); no longer LED69.3 (DIN)
- net at LED80.2 (DOUT): now also LED59.3 (DIN); no longer LED65.3 (DIN)
- new net: D66.1 (K), MX66.2
- new net: LED67.2 (DOUT), LED68.3 (DIN)
- new net: D65.1 (K), MX65.2
Other:
- moved on the sheet: C16, C17, D111, D112, D113, D43, D82, D99, LED65, LED66, LED69, LED70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
